File: Storage_and_memory.sch (KiCad schematic (older format))
At the start: 10 parts

Commit message: v0.1
Parts:
- gave numbers to parts that had none: 10
Changed lines of the file:
@@
 $Descr A4 11693 8268
 encoding utf-8
-Sheet 6 9
-Title "QuadSPI Flash and SD Card storage"
-Date "2021-05-08"
-Rev "0.1"
-Comp "SVIELCOM"
-Comment1 ""
+Sheet 5 9
+Title "ШВУ"
+Date "2021-03-25"
+Rev "V0.1"
+Comp "ЦВЕТМЕТНАЛАДКА"
+Comment1 "Шустов В.И."
 Comment2 ""
 Comment3 ""
@@
 $EndDescr
 $Comp
-L Схема-и-печатная-плата-rescue:W25Q256JVFIQ-Memory_Flash U?
+L Схема-и-печатная-плата-rescue:W25Q256JVFIQ-Memory_Flash U15
 U 1 1 60D8B67A
 P 4270 4710
-F 0 "U?" H 4820 4975 50  0000 C CNN
+F 0 "U15" H 4820 4975 50  0000 C CNN
 F 1 "W25Q256JVFIQ" H 4820 4884 50  0000 C CNN
 F 2 "Package_SO:SOIC-16W_7.5x10.3mm_P1.27mm" H 4270 5110 50  0001 L CNN
@@
 $EndComp
 $Comp
-L Connector:Micro_SD_Card_Det J?
+L Connector:Micro_SD_Card_Det J4
 U 1 1 60912CF3
 P 6840 1990
-F 0 "J?" H 6790 2807 50  0000 C CNN
+F 0 "J4" H 6790 2807 50  0000 C CNN
 F 1 "Micro_SD_Card_Det" H 6790 2716 50  0000 C CNN
 F 2 "" H 8890 2690 50  0001 C CNN
@@
 	5870 2090 5870 2790
 $Comp
-L SVIELCOM_Library:TXS0206-29YFPRB U?
+L SVIELCOM_Library:TXS0206-29YFPRB U14
 U 1 1 6095792B
 P 3800 1590
-F 0 "U?" H 4600 1877 60  0000 C CNN
+F 0 "U14" H 4600 1877 60  0000 C CNN
 F 1 "TXS0206-29YFPRB" H 4600 1771 60  0000 C CNN
 F 2 "SVIELCOM:TXS0206-29YFPRB" H 4600 190 60  0001 C CNN
@@
 AR Path="/6098D661" Ref="#PWR?"  Part="1"
 AR Path="/60A03F8A/6098D661" Ref="#PWR?"  Part="1"
-AR Path="/60D8A641/6098D661" Ref="#PWR?"  Part="1"
-F 0 "#PWR?" H 5300 2660 50  0001 C CNN
+AR Path="/60D8A641/6098D661" Ref="#PWR060"  Part="1"
+F 0 "#PWR060" H 5300 2660 50  0001 C CNN
 F 1 "GNDREF" V 5305 2782 50  0001 R CNN
 F 2 "" H 5300 2910 50  0001 C CNN
@@
 AR Path="/6099014F" Ref="C?"  Part="1"
 AR Path="/60A03F8A/6099014F" Ref="C?"  Part="1"
-AR Path="/60D8A641/6099014F" Ref="C?"  Part="1"
-F 0 "C?" H 5450 2500 50  0000 L CNN
+AR Path="/60D8A641/6099014F" Ref="C51"  Part="1"
+F 0 "C51" H 5450 2500 50  0000 L CNN
 F 1 "1µF" H 5370 2360 50  0000 L CNN
 F 2 "Capacitor_SMD:C_0603_1608Metric_Pad1.08x0.95mm_HandSolder" H 5468 2460 50  0001 C CNN
@@
 AR Path="/60990581" Ref="C?"  Part="1"
 AR Path="/60A03F8A/60990581" Ref="C?"  Part="1"
-AR Path="/60D8A641/60990581" Ref="C?"  Part="1"
-F 0 "C?" H 5710 2500 50  0000 L CNN
+AR Path="/60D8A641/60990581" Ref="C52"  Part="1"
+F 0 "C52" H 5710 2500 50  0000 L CNN
 F 1 "1µF" H 5680 2360 50  0000 L CNN
 F 2 "Capacitor_SMD:C_0603_1608Metric_Pad1.08x0.95mm_HandSolder" H 5718 2460 50  0001 C CNN
@@
 AR Path="/60996784" Ref="C?"  Part="1"
 AR Path="/60A03F8A/60996784" Ref="C?"  Part="1"
-AR Path="/60D8A641/60996784" Ref="C?"  Part="1"
-F 0 "C?" H 3050 1530 50  0000 L CNN
+AR Path="/60D8A641/60996784" Ref="C50"  Part="1"
+F 0 "C50" H 3050 1530 50  0000 L CNN
 F 1 "1µF" H 3080 1340 50  0000 L CNN
 F 2 "Capacitor_SMD:C_0603_1608Metric_Pad1.08x0.95mm_HandSolder" H 3288 1290 50  0001 C CNN
@@
 AR Path="/60997B3F" Ref="#PWR?"  Part="1"
 AR Path="/60A03F8A/60997B3F" Ref="#PWR?"  Part="1"
-AR Path="/60D8A641/60997B3F" Ref="#PWR?"  Part="1"
-F 0 "#PWR?" H 3250 1340 50  0001 C CNN
+AR Path="/60D8A641/60997B3F" Ref="#PWR058"  Part="1"
+F 0 "#PWR058" H 3250 1340 50  0001 C CNN
 F 1 "GNDREF" V 3255 1462 50  0001 R CNN
 F 2 "" H 3250 1590 50  0001 C CNN
@@
 AR Path="/60998CBA" Ref="#PWR?"  Part="1"
 AR Path="/60A03F8A/60998CBA" Ref="#PWR?"  Part="1"
-AR Path="/60D8A641/60998CBA" Ref="#PWR?"  Part="1"
-F 0 "#PWR?" H 3860 2660 50  0001 C CNN
+AR Path="/60D8A641/60998CBA" Ref="#PWR059"  Part="1"
+F 0 "#PWR059" H 3860 2660 50  0001 C CNN
 F 1 "GNDREF" V 3865 2782 50  0001 R CNN
 F 2 "" H 3860 2910 50  0001 C CNN
@@
 AR Path="/609998AA" Ref="#PWR?"  Part="1"
 AR Path="/60A03F8A/609998AA" Ref="#PWR?"  Part="1"
-AR Path="/60D8A641/609998AA" Ref="#PWR?"  Part="1"
-F 0 "#PWR?" H 7640 2660 50  0001 C CNN
+AR Path="/60D8A641/609998AA" Ref="#PWR061"  Part="1"
+F 0 "#PWR061" H 7640 2660 50  0001 C CNN
 F 1 "GNDREF" V 7645 2782 50  0001 R CNN
 F 2 "" H 7640 2910 50  0001 C CNN
@@
 	7640 2490 7640 2910
 $Comp
-L SVIELCOM_Library:+2.9V_SD #PWR?
+L SVIELCOM_Library:+2.9V_SD #PWR057
 U 1 1 6099AF71
 P 5430 1060
-F 0 "#PWR?" H 5430 910 50  0001 C CNN
+F 0 "#PWR057" H 5430 910 50  0001 C CNN
 F 1 "+2.9V_SD" H 5445 1233 50  0000 C CNN
 F 2 "" H 5430 1060 50  0001 C CNN
@@
 PB8
 $Comp
-L SVIELCOM_Library:VDD_MCU #PWR?
+L SVIELCOM_Library:VDD_MCU #PWR056
 U 1 1 60A156B1
 P 3480 1060
-F 0 "#PWR?" H 3480 910 50  0001 C CNN
+F 0 "#PWR056" H 3480 910 50  0001 C CNN
 F 1 "VDD_MCU" H 3495 1233 50  0000 C CNN
 F 2 "" H 3480 1060 50  0001 C CNN
@@
 $EndComp
 $Comp
-L SVIELCOM_Library:VDD_MCU #PWR?
+L SVIELCOM_Library:VDD_MCU #PWR062
 U 1 1 60A15E6C
 P 4030 4590
-F 0 "#PWR?" H 4030 4440 50  0001 C CNN
+F 0 "#PWR062" H 4030 4440 50  0001 C CNN
 F 1 "VDD_MCU" H 4045 4763 50  0000 C CNN
 F 2 "" H 4030 4590 50  0001 C CNN
@@
 AR Path="/60A17165" Ref="#PWR?"  Part="1"
 AR Path="/60A03F8A/60A17165" Ref="#PWR?"  Part="1"
-AR Path="/60D8A641/60A17165" Ref="#PWR?"  Part="1"
-F 0 "#PWR?" H 5500 5220 50  0001 C CNN
+AR Path="/60D8A641/60A17165" Ref="#PWR063"  Part="1"
+F 0 "#PWR063" H 5500 5220 50  0001 C CNN
 F 1 "GNDREF" V 5505 5342 50  0001 R CNN
 F 2 "" H 5500 5470 50  0001 C CNN
@@
 AR Path="/60A1C3E5" Ref="R?"  Part="1"
 AR Path="/60A03F8A/60A1C3E5" Ref="R?"  Part="1"
-AR Path="/60D8A641/60A1C3E5" Ref="R?"  Part="1"
-F 0 "R?" V 5740 4530 50  0000 C CNN
+AR Path="/60D8A641/60A1C3E5" Ref="R17"  Part="1"
+F 0 "R17" V 5740 4530 50  0000 C CNN
 F 1 "33" V 5750 4910 50  0000 C CNN
 F 2 "Resistor_SMD:R_0805_2012Metric_Pad1.20x1.40mm_HandSolder" V 5720 4710 50  0001 C CNN
@@
 AR Path="/60A1DE64" Ref="R?"  Part="1"
 AR Path="/60A03F8A/60A1DE64" Ref="R?"  Part="1"
-AR Path="/60D8A641/60A1DE64" Ref="R?"  Part="1"
-F 0 "R?" V 5750 4630 50  0000 C CNN
+AR Path="/60D8A641/60A1DE64" Ref="R18"  Part="1"
+F 0 "R18" V 5750 4630 50  0000 C CNN
 F 1 "33" V 5750 5010 50  0000 C CNN
 F 2 "Resistor_SMD:R_0805_2012Metric_Pad1.20x1.40mm_HandSolder" V 5720 4810 50  0001 C CNN
@@
 AR Path="/60A1EB77" Ref="R?"  Part="1"
 AR Path="/60A03F8A/60A1EB77" Ref="R?"  Part="1"
-AR Path="/60D8A641/60A1EB77" Ref="R?"  Part="1"
-F 0 "R?" V 5700 4930 50  0000 C CNN
+AR Path="/60D8A641/60A1EB77" Ref="R19"  Part="1"
+F 0 "R19" V 5700 4930 50  0000 C CNN
 F 1 "33" V 5700 5070 50  0000 C CNN
 F 2 "Resistor_SMD:R_0805_2012Metric_Pad1.20x1.40mm_HandSolder" V 5720 5010 50  0001 C CNN
@@
 AR Path="/60A1F94D" Ref="R?"  Part="1"
 AR Path="/60A03F8A/60A1F94D" Ref="R?"  Part="1"
-AR Path="/60D8A641/60A1F94D" Ref="R?"  Part="1"
-F 0 "R?" V 5880 5030 50  0000 C CNN
+AR Path="/60D8A641/60A1F94D" Ref="R20"  Part="1"
+F 0 "R20" V 5880 5030 50  0000 C CNN
 F 1 "33" V 5880 5170 50  0000 C CNN
 F 2 "Resistor_SMD:R_0805_2012Metric_Pad1.20x1.40mm_HandSolder" V 5720 5110 50  0001 C CNN

Commit message: v0.3 changed sd_card holder
Parts:
- removed J4: Micro_SD_Card_Det, symbol Connector:Micro_SD_Card_Det
- added J?: DM3AT-SF-PEJM5, SVIELCOM:HRS_DM3AT-SF-PEJM5, symbol SVIELCOM_Library:DM3AT-SF-PEJM5
- renumbered C50 to C45, C51 to C46, C52 to C47
Connections:
- wire segments 52 -> 53
- no-connect marks 3 -> 2
Changed lines of the file:
@@
-	1    0    0    -1
-$EndComp
-$Comp
-L Connector:Micro_SD_Card_Det J4
-U 1 1 60912CF3
-P 6840 1990
-F 0 "J4" H 6790 2807 50  0000 C CNN
-F 1 "Micro_SD_Card_Det" H 6790 2716 50  0000 C CNN
-F 2 "" H 8890 2690 50  0001 C CNN
-F 3 "https://www.hirose.com/product/en/download_file/key_name/DM3/category/Catalog/doc_file_id/49662/?file_category_id=4&item_id=195&is_series=1" H 6840 2090 50  0001 C CNN
-	1    6840 1990
 	1    0    0    -1
 $EndComp
@@
 Wire Wire Line
 	5300 1890 5430 1890
-NoConn ~ 5940 2390
 $Comp
 L power:GNDREF #PWR?
@@
 AR Path="/6099014F" Ref="C?"  Part="1"
 AR Path="/60A03F8A/6099014F" Ref="C?"  Part="1"
-AR Path="/60D8A641/6099014F" Ref="C51"  Part="1"
-F 0 "C51" H 5450 2500 50  0000 L CNN
+AR Path="/60D8A641/6099014F" Ref="C46"  Part="1"
+F 0 "C46" H 5450 2500 50  0000 L CNN
 F 1 "1µF" H 5370 2360 50  0000 L CNN
 F 2 "Capacitor_SMD:C_0603_1608Metric_Pad1.08x0.95mm_HandSolder" H 5468 2460 50  0001 C CNN
@@
 AR Path="/60990581" Ref="C?"  Part="1"
 AR Path="/60A03F8A/60990581" Ref="C?"  Part="1"
-AR Path="/60D8A641/60990581" Ref="C52"  Part="1"
-F 0 "C52" H 5710 2500 50  0000 L CNN
+AR Path="/60D8A641/60990581" Ref="C47"  Part="1"
+F 0 "C47" H 5710 2500 50  0000 L CNN
 F 1 "1µF" H 5680 2360 50  0000 L CNN
 F 2 "Capacitor_SMD:C_0603_1608Metric_Pad1.08x0.95mm_HandSolder" H 5718 2460 50  0001 C CNN
@@
 AR Path="/60996784" Ref="C?"  Part="1"
 AR Path="/60A03F8A/60996784" Ref="C?"  Part="1"
-AR Path="/60D8A641/60996784" Ref="C50"  Part="1"
-F 0 "C50" H 3050 1530 50  0000 L CNN
+AR Path="/60D8A641/60996784" Ref="C45"  Part="1"
+F 0 "C45" H 3050 1530 50  0000 L CNN
 F 1 "1µF" H 3080 1340 50  0000 L CNN
 F 2 "Capacitor_SMD:C_0603_1608Metric_Pad1.08x0.95mm_HandSolder" H 3288 1290 50  0001 C CNN
@@
 L power:GNDREF #PWR?
 U 1 1 609998AA
-P 7640 2910
+P 6940 2910
 AR Path="/609998AA" Ref="#PWR?"  Part="1"
 AR Path="/60A03F8A/609998AA" Ref="#PWR?"  Part="1"
 AR Path="/60D8A641/609998AA" Ref="#PWR061"  Part="1"
-F 0 "#PWR061" H 7640 2660 50  0001 C CNN
-F 1 "GNDREF" V 7645 2782 50  0001 R CNN
-F 2 "" H 7640 2910 50  0001 C CNN
-F 3 "" H 7640 2910 50  0001 C CNN
-	1    7640 2910
-	1    0    0    -1
-$EndComp
-Wire Wire Line
-	7640 2490 7640 2910
+F 0 "#PWR061" H 6940 2660 50  0001 C CNN
+F 1 "GNDREF" V 6945 2782 50  0001 R CNN
+F 2 "" H 6940 2910 50  0001 C CNN
+F 3 "" H 6940 2910 50  0001 C CNN
+	1    6940 2910
+	1    0    0    -1
+$EndComp
+Wire Wire Line
+	6940 2490 6940 2910
 $Comp
 L SVIELCOM_Library:+2.9V_SD #PWR057
@@
 Text Label 3770 5110 0    50   ~ 0
 PB6
+$Comp
+L SVIELCOM_Library:DM3AT-SF-PEJM5 J?
+U 1 1 61644FF6
+P 6440 2190
+F 0 "J?" H 6480 3100 50  0000 C CNN
+F 1 "DM3AT-SF-PEJM5" H 6480 3000 50  0000 C CNN
+F 2 "SVIELCOM:HRS_DM3AT-SF-PEJM5" H 6740 2840 50  0001 L BNN
+F 3 "https://www.terraelectronica.ru/pdf/show?pdf_file=%252Fds%252Fpdf%252FD%252FDM3AT-SF-PEJM5.pdf" H 6440 2190 50  0001 L BNN
+F 4 "DM3 RA SMT microSD memory card push/push" H 6740 2740 50  0001 L BNN "DESCRIPTION"
+F 5 "DM3AT-SF-PEJM5" H 6740 2640 50  0001 L BNN "MP"
+	1    6440 2190
+	1    0    0    -1
+$EndComp
+$Comp
+L power:GNDREF #PWR?
+U 1 1 6164845D
+P 5940 2810
+AR Path="/6164845D" Ref="#PWR?"  Part="1"
+AR Path="/60A03F8A/6164845D" Ref="#PWR?"  Part="1"
+AR Path="/60D8A641/6164845D" Ref="#PWR?"  Part="1"
+F 0 "#PWR?" H 5940 2560 50  0001 C CNN
+F 1 "GNDREF" V 5945 2682 50  0001 R CNN
+F 2 "" H 5940 2810 50  0001 C CNN
+F 3 "" H 5940 2810 50  0001 C CNN
+	1    5940 2810
+	1    0    0    -1
+$EndComp
+Wire Wire Line
+	5940 2390 5940 2810
 $EndSCHEMATC

Commit message: footprints associations is done
Parts:
- gave numbers to parts that had none: 1
- renumbered R17 to R19, R18 to R20, R19 to R21, R20 to R22
Changed lines of the file:
@@
 Title "ШВУ"
 Date "2021-03-25"
-Rev "V0.1"
+Rev "V0.3"
 Comp "ЦВЕТМЕТНАЛАДКА"
 Comment1 "Шустов В.И."
@@
 AR Path="/6098D661" Ref="#PWR?"  Part="1"
 AR Path="/60A03F8A/6098D661" Ref="#PWR?"  Part="1"
-AR Path="/60D8A641/6098D661" Ref="#PWR060"  Part="1"
-F 0 "#PWR060" H 5300 2660 50  0001 C CNN
+AR Path="/60D8A641/6098D661" Ref="#PWR061"  Part="1"
+F 0 "#PWR061" H 5300 2660 50  0001 C CNN
 F 1 "GNDREF" V 5305 2782 50  0001 R CNN
 F 2 "" H 5300 2910 50  0001 C CNN
@@
 AR Path="/60998CBA" Ref="#PWR?"  Part="1"
 AR Path="/60A03F8A/60998CBA" Ref="#PWR?"  Part="1"
-AR Path="/60D8A641/60998CBA" Ref="#PWR059"  Part="1"
-F 0 "#PWR059" H 3860 2660 50  0001 C CNN
+AR Path="/60D8A641/60998CBA" Ref="#PWR060"  Part="1"
+F 0 "#PWR060" H 3860 2660 50  0001 C CNN
 F 1 "GNDREF" V 3865 2782 50  0001 R CNN
 F 2 "" H 3860 2910 50  0001 C CNN
@@
 AR Path="/609998AA" Ref="#PWR?"  Part="1"
 AR Path="/60A03F8A/609998AA" Ref="#PWR?"  Part="1"
-AR Path="/60D8A641/609998AA" Ref="#PWR061"  Part="1"
-F 0 "#PWR061" H 6940 2660 50  0001 C CNN
+AR Path="/60D8A641/609998AA" Ref="#PWR062"  Part="1"
+F 0 "#PWR062" H 6940 2660 50  0001 C CNN
 F 1 "GNDREF" V 6945 2782 50  0001 R CNN
 F 2 "" H 6940 2910 50  0001 C CNN
@@
 $EndComp
 $Comp
-L SVIELCOM_Library:VDD_MCU #PWR062
+L SVIELCOM_Library:VDD_MCU #PWR063
 U 1 1 60A15E6C
 P 4030 4590
-F 0 "#PWR062" H 4030 4440 50  0001 C CNN
+F 0 "#PWR063" H 4030 4440 50  0001 C CNN
 F 1 "VDD_MCU" H 4045 4763 50  0000 C CNN
 F 2 "" H 4030 4590 50  0001 C CNN
@@
 AR Path="/60A17165" Ref="#PWR?"  Part="1"
 AR Path="/60A03F8A/60A17165" Ref="#PWR?"  Part="1"
-AR Path="/60D8A641/60A17165" Ref="#PWR063"  Part="1"
-F 0 "#PWR063" H 5500 5220 50  0001 C CNN
+AR Path="/60D8A641/60A17165" Ref="#PWR064"  Part="1"
+F 0 "#PWR064" H 5500 5220 50  0001 C CNN
 F 1 "GNDREF" V 5505 5342 50  0001 R CNN
 F 2 "" H 5500 5470 50  0001 C CNN
@@
 AR Path="/60A1C3E5" Ref="R?"  Part="1"
 AR Path="/60A03F8A/60A1C3E5" Ref="R?"  Part="1"
-AR Path="/60D8A641/60A1C3E5" Ref="R17"  Part="1"
-F 0 "R17" V 5740 4530 50  0000 C CNN
+AR Path="/60D8A641/60A1C3E5" Ref="R19"  Part="1"
+F 0 "R19" V 5740 4530 50  0000 C CNN
 F 1 "33" V 5750 4910 50  0000 C CNN
 F 2 "Resistor_SMD:R_0805_2012Metric_Pad1.20x1.40mm_HandSolder" V 5720 4710 50  0001 C CNN
@@
 AR Path="/60A1DE64" Ref="R?"  Part="1"
 AR Path="/60A03F8A/60A1DE64" Ref="R?"  Part="1"
-AR Path="/60D8A641/60A1DE64" Ref="R18"  Part="1"
-F 0 "R18" V 5750 4630 50  0000 C CNN
+AR Path="/60D8A641/60A1DE64" Ref="R20"  Part="1"
+F 0 "R20" V 5750 4630 50  0000 C CNN
 F 1 "33" V 5750 5010 50  0000 C CNN
 F 2 "Resistor_SMD:R_0805_2012Metric_Pad1.20x1.40mm_HandSolder" V 5720 4810 50  0001 C CNN
@@
 AR Path="/60A1EB77" Ref="R?"  Part="1"
 AR Path="/60A03F8A/60A1EB77" Ref="R?"  Part="1"
-AR Path="/60D8A641/60A1EB77" Ref="R19"  Part="1"
-F 0 "R19" V 5700 4930 50  0000 C CNN
+AR Path="/60D8A641/60A1EB77" Ref="R21"  Part="1"
+F 0 "R21" V 5700 4930 50  0000 C CNN
 F 1 "33" V 5700 5070 50  0000 C CNN
 F 2 "Resistor_SMD:R_0805_2012Metric_Pad1.20x1.40mm_HandSolder" V 5720 5010 50  0001 C CNN
@@
 AR Path="/60A1F94D" Ref="R?"  Part="1"
 AR Path="/60A03F8A/60A1F94D" Ref="R?"  Part="1"
-AR Path="/60D8A641/60A1F94D" Ref="R20"  Part="1"
-F 0 "R20" V 5880 5030 50  0000 C CNN
+AR Path="/60D8A641/60A1F94D" Ref="R22"  Part="1"
+F 0 "R22" V 5880 5030 50  0000 C CNN
 F 1 "33" V 5880 5170 50  0000 C CNN
 F 2 "Resistor_SMD:R_0805_2012Metric_Pad1.20x1.40mm_HandSolder" V 5720 5110 50  0001 C CNN
@@
 PB6
 $Comp
-L SVIELCOM_Library:DM3AT-SF-PEJM5 J?
+L SVIELCOM_Library:DM3AT-SF-PEJM5 J4
 U 1 1 61644FF6
 P 6440 2190
-F 0 "J?" H 6480 3100 50  0000 C CNN
+F 0 "J4" H 6480 3100 50  0000 C CNN
 F 1 "DM3AT-SF-PEJM5" H 6480 3000 50  0000 C CNN
 F 2 "SVIELCOM:HRS_DM3AT-SF-PEJM5" H 6740 2840 50  0001 L BNN
@@
 AR Path="/6164845D" Ref="#PWR?"  Part="1"
 AR Path="/60A03F8A/6164845D" Ref="#PWR?"  Part="1"
-AR Path="/60D8A641/6164845D" Ref="#PWR?"  Part="1"
-F 0 "#PWR?" H 5940 2560 50  0001 C CNN
+AR Path="/60D8A641/6164845D" Ref="#PWR059"  Part="1"
+F 0 "#PWR059" H 5940 2560 50  0001 C CNN
 F 1 "GNDREF" V 5945 2682 50  0001 R CNN
 F 2 "" H 5940 2810 50  0001 C CNN

Commit message: corrected few footprints, correct all resistors and capacitors type for ordering
Parts:
- R19, R20, R21, R22: Type (none) -> RC0805FR-0733RL
Changed lines of the file:
@@
 F 2 "Resistor_SMD:R_0805_2012Metric_Pad1.20x1.40mm_HandSolder" V 5720 4710 50  0001 C CNN
 F 3 "~" H 5790 4710 50  0001 C CNN
+F 4 "RC0805FR-0733RL" V 5790 4710 50  0001 C CNN "Type"
 	1    5790 4710
 	0    1    1    0
@@
 F 2 "Resistor_SMD:R_0805_2012Metric_Pad1.20x1.40mm_HandSolder" V 5720 4810 50  0001 C CNN
 F 3 "~" H 5790 4810 50  0001 C CNN
+F 4 "RC0805FR-0733RL" V 5790 4810 50  0001 C CNN "Type"
 	1    5790 4810
 	0    1    1    0
@@
 F 2 "Resistor_SMD:R_0805_2012Metric_Pad1.20x1.40mm_HandSolder" V 5720 5010 50  0001 C CNN
 F 3 "~" H 5790 5010 50  0001 C CNN
+F 4 "RC0805FR-0733RL" V 5790 5010 50  0001 C CNN "Type"
 	1    5790 5010
 	0    1    1    0
@@
 F 2 "Resistor_SMD:R_0805_2012Metric_Pad1.20x1.40mm_HandSolder" V 5720 5110 50  0001 C CNN
 F 3 "~" H 5790 5110 50  0001 C CNN
+F 4 "RC0805FR-0733RL" V 5790 5110 50  0001 C CNN "Type"
 	1    5790 5110
 	0    1    1    0
