File: Schema_and_PCB.sch (KiCad schematic (older format))
At the start: 8 parts, among them SW1 PST-11A, U6 STM32H743ZIT6

Commit message: Indication edit
Changed lines of the file:
@@
 $EndSheet
 $Sheet
-S 1200 8020 1010 840
+S 890  8000 1010 840
 U 60D8A641
 F0 "Storage_and_memory" 50

Commit message: start create Analog IO
Parts:
- removed PS1: TMH2415S, Converter_DCDC:Converter_DCDC_XP_POWER-IAxxxxS_THT, symbol Converter_DCDC:IA2415S
Changed lines of the file:
@@
 F1 "Analog_and_digital_IO.sch" 50
 $EndSheet
-$Comp
-L Converter_DCDC:IA2415S PS1
-U 1 1 6062DF49
-P 9430 2970
-F 0 "PS1" H 9430 3337 50  0000 C CNN
-F 1 "TMH2415S" H 9430 3246 50  0000 C CNN
-F 2 "Converter_DCDC:Converter_DCDC_XP_POWER-IAxxxxS_THT" H 8380 2720 50  0001 L CNN
-F 3 "https://www.terraelectronica.ru/pdf/show?pdf_file=%252Fds%252Fpdf%252FT%252FTMH.pdf" H 10480 2670 50  0001 L CNN
-	1    9430 2970
-	1    0    0    -1
-$EndComp
 $EndSCHEMATC

Commit message: Analog Input edited
Other:
- moved on the sheet: C1, C2, C3, C4, C5, SW1A
Changed lines of the file:
@@
 L Device:C C4
 U 1 1 606157F0
-P 5010 1920
-F 0 "C4" H 5125 1966 50  0000 L CNN
-F 1 "1µF" H 5125 1875 50  0000 L CNN
-F 2 "Capacitor_SMD:C_0603_1608Metric_Pad1.08x0.95mm_HandSolder" H 5048 1770 50  0001 C CNN
-F 3 "http://www.farnell.com/datasheets/2710676.pdf" H 5010 1920 50  0001 C CNN
-F 4 "CL10B105KA8NNNC" H 5010 1920 50  0001 C CNN "Type"
-	1    5010 1920
+P 5090 -1500
+F 0 "C4" H 5205 -1454 50  0000 L CNN
+F 1 "1µF" H 5205 -1545 50  0000 L CNN
+F 2 "Capacitor_SMD:C_0603_1608Metric_Pad1.08x0.95mm_HandSolder" H 5128 -1650 50  0001 C CNN
+F 3 "http://www.farnell.com/datasheets/2710676.pdf" H 5090 -1500 50  0001 C CNN
+F 4 "CL10B105KA8NNNC" H 5090 -1500 50  0001 C CNN "Type"
+	1    5090 -1500
 	1    0    0    -1
 $EndComp
@@
 L Device:CP C3
 U 1 1 6061539B
-P 5270 1540
-F 0 "C3" H 5388 1586 50  0000 L CNN
-F 1 "10µF" H 5388 1495 50  0000 L CNN
-F 2 "Capacitor_Tantalum_SMD:CP_EIA-3216-10_Kemet-I" H 5308 1390 50  0001 C CNN
-F 3 "http://www.mouser.com/ds/2/427/593d-239975.pdf" H 5270 1540 50  0001 C CNN
-F 4 "593D106X9016A2TE3" H 5270 1540 50  0001 C CNN "Type"
-	1    5270 1540
+P 5350 -1880
+F 0 "C3" H 5468 -1834 50  0000 L CNN
+F 1 "10µF" H 5468 -1925 50  0000 L CNN
+F 2 "Capacitor_Tantalum_SMD:CP_EIA-3216-10_Kemet-I" H 5388 -2030 50  0001 C CNN
+F 3 "http://www.mouser.com/ds/2/427/593d-239975.pdf" H 5350 -1880 50  0001 C CNN
+F 4 "593D106X9016A2TE3" H 5350 -1880 50  0001 C CNN "Type"
+	1    5350 -1880
 	1    0    0    -1
 $EndComp
@@
 L Device:CP C2
 U 1 1 6061A793
-P 5830 1510
-F 0 "C2" H 5948 1556 50  0000 L CNN
-F 1 "47µFx25" H 5948 1465 50  0000 L CNN
-F 2 "Capacitor_Tantalum_SMD:CP_EIA-6032-28_Kemet-C_Pad2.25x2.35mm_HandSolder" H 5868 1360 50  0001 C CNN
-F 3 "https://www.farnell.com/datasheets/1878216.pdf" H 5830 1510 50  0001 C CNN
-F 4 "TR3D476K025C0150" H 5830 1510 50  0001 C CNN "Type"
-	1    5830 1510
+P 5910 -1910
+F 0 "C2" H 6028 -1864 50  0000 L CNN
+F 1 "47µFx25" H 6028 -1955 50  0000 L CNN
+F 2 "Capacitor_Tantalum_SMD:CP_EIA-6032-28_Kemet-C_Pad2.25x2.35mm_HandSolder" H 5948 -2060 50  0001 C CNN
+F 3 "https://www.farnell.com/datasheets/1878216.pdf" H 5910 -1910 50  0001 C CNN
+F 4 "TR3D476K025C0150" H 5910 -1910 50  0001 C CNN "Type"
+	1    5910 -1910
 	1    0    0    -1
 $EndComp
@@
 L Device:C C1
 U 1 1 60633F0C
-P 4280 970
-F 0 "C1" H 4395 1016 50  0000 L CNN
-F 1 "1µF" H 4395 925 50  0000 L CNN
-F 2 "Capacitor_SMD:C_0603_1608Metric_Pad1.08x0.95mm_HandSolder" H 4318 820 50  0001 C CNN
-F 3 "https://www.farnell.com/datasheets/2048520.pdf" H 4280 970 50  0001 C CNN
-F 4 "GRM188R7YA105KA12D" H 4280 970 50  0001 C CNN "Type"
-	1    4280 970
+P 4360 -2450
+F 0 "C1" H 4475 -2404 50  0000 L CNN
+F 1 "1µF" H 4475 -2495 50  0000 L CNN
+F 2 "Capacitor_SMD:C_0603_1608Metric_Pad1.08x0.95mm_HandSolder" H 4398 -2600 50  0001 C CNN
+F 3 "https://www.farnell.com/datasheets/2048520.pdf" H 4360 -2450 50  0001 C CNN
+F 4 "GRM188R7YA105KA12D" H 4360 -2450 50  0001 C CNN "Type"
+	1    4360 -2450
 	1    0    0    -1
 $EndComp
@@
 L Device:CP C5
 U 1 1 60634752
-P 6400 1940
-F 0 "C5" H 6518 1986 50  0000 L CNN
-F 1 "47µFx16" H 6518 1895 50  0000 L CNN
-F 2 "Capacitor_Tantalum_SMD:CP_EIA-7343-31_Kemet-D_Pad2.25x2.55mm_HandSolder" H 6438 1790 50  0001 C CNN
-F 3 "https://www.farnell.com/datasheets/1995953.pdf" H 6400 1940 50  0001 C CNN
-F 4 "593D476X9016D2TE3" H 6400 1940 50  0001 C CNN "Type"
-	1    6400 1940
+P 6480 -1480
+F 0 "C5" H 6598 -1434 50  0000 L CNN
+F 1 "47µFx16" H 6598 -1525 50  0000 L CNN
+F 2 "Capacitor_Tantalum_SMD:CP_EIA-7343-31_Kemet-D_Pad2.25x2.55mm_HandSolder" H 6518 -1630 50  0001 C CNN
+F 3 "https://www.farnell.com/datasheets/1995953.pdf" H 6480 -1480 50  0001 C CNN
+F 4 "593D476X9016D2TE3" H 6480 -1480 50  0001 C CNN "Type"
+	1    6480 -1480
 	1    0    0    -1
 $EndComp
@@
 L Switch:SW_DPDT_x2 SW1
 U 1 1 6063E7A3
-P 8850 1360
-F 0 "SW1" H 8850 1645 50  0000 C CNN
-F 1 "PST-11A" H 8850 1554 50  0000 C CNN
-F 2 "" H 8850 1360 50  0001 C CNN
-F 3 "https://www.terraelectronica.ru/product/45953" H 8850 1360 50  0001 C CNN
-	1    8850 1360
+P 8930 -2060
+F 0 "SW1" H 8930 -1775 50  0000 C CNN
+F 1 "PST-11A" H 8930 -1866 50  0000 C CNN
+F 2 "" H 8930 -2060 50  0001 C CNN
+F 3 "https://www.terraelectronica.ru/product/45953" H 8930 -2060 50  0001 C CNN
+	1    8930 -2060
 	1    0    0    -1
 $EndComp
