File: Analog_and_digital_IO.sch (KiCad schematic (older format))
At the start: 4 parts

Commit message: start create Analog IO
Parts:
- added PS?: TMH2415S, Converter_DCDC:Converter_DCDC_XP_POWER-IAxxxxS_THT, symbol Converter_DCDC:IA2415S
- added U?: LT1129CST-5#PBF, Package_TO_SOT_SMD:SOT-223-3_TabPin2, symbol SVIELCOM_Library:LT1129CST-5#PBF
- added U?: REF1933AIDDCT, Package_TO_SOT_SMD:SOT-23-5_HandSoldering, symbol SVIELCOM_Library:REF1933AIDDCT
Other:
- moved on the sheet: U?
Changed lines of the file:
@@
 L Схема-и-печатная-плата-rescue:ISO224ADWVR-Isolator U?
 U 1 1 60D90026
-P 4300 3670
+P 2610 3180
 AR Path="/60D90026" Ref="U?"  Part="1"
 AR Path="/60D8C564/60D90026" Ref="U?"  Part="1"
-F 0 "U?" H 4950 3935 50  0000 C CNN
-F 1 "ISO224ADWVR" H 4950 3844 50  0000 C CNN
-F 2 "Texas_Instruments-DWV0008A-0-0-*" H 4300 4070 50  0001 L CNN
-F 3 "https://www.ti.com/lit/ds/symlink/iso224.pdf" H 4300 4170 50  0001 L CNN
-F 4 "+125°C" H 4300 4270 50  0001 L CNN "ambient temperature range high"
-F 5 "-55°C" H 4300 4370 50  0001 L CNN "ambient temperature range low"
-F 6 "No" H 4300 4470 50  0001 L CNN "automotive"
-F 7 "IC" H 4300 4570 50  0001 L CNN "category"
-F 8 "Integrated Circuits (ICs)" H 4300 4670 50  0001 L CNN "device class L1"
-F 9 "Linear ICs" H 4300 4770 50  0001 L CNN "device class L2"
-F 10 "unset" H 4300 4870 50  0001 L CNN "device class L3"
-F 11 "IC ISOLATED 8SOIC" H 4300 4970 50  0001 L CNN "digikey description"
-F 12 "296-52315-1-ND" H 4300 5070 50  0001 L CNN "digikey part number"
-F 13 "185kHz" H 4300 5170 50  0001 L CNN "gain bandwidth"
-F 14 "2.8mm" H 4300 5270 50  0001 L CNN "height"
-F 15 "0.015uA" H 4300 5370 50  0001 L CNN "input bias current"
-F 16 "1mV" H 4300 5470 50  0001 L CNN "input offset voltage"
-F 17 "Yes" H 4300 5570 50  0001 L CNN "lead free"
-F 18 "f96fe3b55d649421" H 4300 5670 50  0001 L CNN "library id"
-F 19 "Texas Instruments" H 4300 5770 50  0001 L CNN "manufacturer"
-F 20 "+150°C" H 4300 5870 50  0001 L CNN "max junction temp"
-F 21 "18V" H 4300 5970 50  0001 L CNN "max supply voltage"
-F 22 "4.5V" H 4300 6070 50  0001 L CNN "min supply voltage"
-F 23 "Reinforced isolated amplifier for voltage sensing with ±12-V input 8-SOIC -55 to 125" H 4300 6170 50  0001 L CNN "mouser description"
-F 24 "595-ISO224ADWVR" H 4300 6270 50  0001 L CNN "mouser part number"
-F 25 "1" H 4300 6370 50  0001 L CNN "number of channels"
-F 26 "18mA" H 4300 6470 50  0001 L CNN "output current per channel"
-F 27 "SOICW8" H 4300 6570 50  0001 L CNN "package"
-F 28 "250us" H 4300 6670 50  0001 L CNN "response time"
-F 29 "Yes" H 4300 6770 50  0001 L CNN "rohs"
-F 30 "0.36mm" H 4300 6870 50  0001 L CNN "standoff height"
-F 31 "+125°C" H 4300 6970 50  0001 L CNN "temperature range high"
-F 32 "-55°C" H 4300 7070 50  0001 L CNN "temperature range low"
-F 33 "0.001/3V/mV" H 4300 7170 50  0001 L CNN "voltage gain"
-	1    4300 3670
+F 0 "U?" H 3260 3445 50  0000 C CNN
+F 1 "ISO224ADWVR" H 3260 3354 50  0000 C CNN
+F 2 "Texas_Instruments-DWV0008A-0-0-*" H 2610 3580 50  0001 L CNN
+F 3 "https://www.ti.com/lit/ds/symlink/iso224.pdf" H 2610 3680 50  0001 L CNN
+F 4 "+125°C" H 2610 3780 50  0001 L CNN "ambient temperature range high"
+F 5 "-55°C" H 2610 3880 50  0001 L CNN "ambient temperature range low"
+F 6 "No" H 2610 3980 50  0001 L CNN "automotive"
+F 7 "IC" H 2610 4080 50  0001 L CNN "category"
+F 8 "Integrated Circuits (ICs)" H 2610 4180 50  0001 L CNN "device class L1"
+F 9 "Linear ICs" H 2610 4280 50  0001 L CNN "device class L2"
+F 10 "unset" H 2610 4380 50  0001 L CNN "device class L3"
+F 11 "IC ISOLATED 8SOIC" H 2610 4480 50  0001 L CNN "digikey description"
+F 12 "296-52315-1-ND" H 2610 4580 50  0001 L CNN "digikey part number"
+F 13 "185kHz" H 2610 4680 50  0001 L CNN "gain bandwidth"
+F 14 "2.8mm" H 2610 4780 50  0001 L CNN "height"
+F 15 "0.015uA" H 2610 4880 50  0001 L CNN "input bias current"
+F 16 "1mV" H 2610 4980 50  0001 L CNN "input offset voltage"
+F 17 "Yes" H 2610 5080 50  0001 L CNN "lead free"
+F 18 "f96fe3b55d649421" H 2610 5180 50  0001 L CNN "library id"
+F 19 "Texas Instruments" H 2610 5280 50  0001 L CNN "manufacturer"
+F 20 "+150°C" H 2610 5380 50  0001 L CNN "max junction temp"
+F 21 "18V" H 2610 5480 50  0001 L CNN "max supply voltage"
+F 22 "4.5V" H 2610 5580 50  0001 L CNN "min supply voltage"
+F 23 "Reinforced isolated amplifier for voltage sensing with ±12-V input 8-SOIC -55 to 125" H 2610 5680 50  0001 L CNN "mouser description"
+F 24 "595-ISO224ADWVR" H 2610 5780 50  0001 L CNN "mouser part number"
+F 25 "1" H 2610 5880 50  0001 L CNN "number of channels"
+F 26 "18mA" H 2610 5980 50  0001 L CNN "output current per channel"
+F 27 "SOICW8" H 2610 6080 50  0001 L CNN "package"
+F 28 "250us" H 2610 6180 50  0001 L CNN "response time"
+F 29 "Yes" H 2610 6280 50  0001 L CNN "rohs"
+F 30 "0.36mm" H 2610 6380 50  0001 L CNN "standoff height"
+F 31 "+125°C" H 2610 6480 50  0001 L CNN "temperature range high"
+F 32 "-55°C" H 2610 6580 50  0001 L CNN "temperature range low"
+F 33 "0.001/3V/mV" H 2610 6680 50  0001 L CNN "voltage gain"
+	1    2610 3180
 	1    0    0    -1
 $EndComp
@@
 	1    0    0    -1
 $EndComp
+$Comp
+L Converter_DCDC:IA2415S PS?
+U 1 1 609B5185
+P 2580 1890
+F 0 "PS?" H 2580 2257 50  0000 C CNN
+F 1 "TMH2415S" H 2580 2166 50  0000 C CNN
+F 2 "Converter_DCDC:Converter_DCDC_XP_POWER-IAxxxxS_THT" H 1530 1640 50  0001 L CNN
+F 3 "https://www.terraelectronica.ru/pdf/show?pdf_file=%252Fds%252Fpdf%252FT%252FTMH.pdf" H 3630 1590 50  0001 L CNN
+	1    2580 1890
+	1    0    0    -1
+$EndComp
+$Comp
+L SVIELCOM_Library:LT1129CST-5#PBF U?
+U 1 1 609E8AE5
+P 6840 1330
+F 0 "U?" H 6840 1817 60  0000 C CNN
+F 1 "LT1129CST-5#PBF" H 6840 1711 60  0000 C CNN
+F 2 "Package_TO_SOT_SMD:SOT-223-3_TabPin2" H 6790 930 60  0001 C CNN
+F 3 "https://www.farnell.com/datasheets/1576439.pdf" H 6740 1630 60  0001 C CNN
+	1    6840 1330
+	1    0    0    -1
+$EndComp
+$Comp
+L SVIELCOM_Library:REF1933AIDDCT U?
+U 1 1 609E97C9
+P 4550 2050
+F 0 "U?" H 4550 2537 60  0000 C CNN
+F 1 "REF1933AIDDCT" H 4550 2431 60  0000 C CNN
+F 2 "Package_TO_SOT_SMD:SOT-23-5_HandSoldering" H 4600 1650 60  0001 C CNN
+F 3 "https://www.ti.com/lit/ds/symlink/ref1933.pdf?ts=1620800334381&ref_url=https%253A%252F%252Fwww.ti.com%252Fproduct%252FREF1933%253FkeyMatch%253DREF1933%2526tisearch%253Dsearch-everything%2526usecase%253DGPN" H 4900 2050 60  0001 C CNN
+	1    4550 2050
+	1    0    0    -1
+$EndComp

Commit message: Analog Input edited
Parts:
- removed U?: LT1129CST-5#PBF, Package_TO_SOT_SMD:SOT-223-3_TabPin2, symbol SVIELCOM_Library:LT1129CST-5#PBF
- removed U?: REF1933AIDDCT, Package_TO_SOT_SMD:SOT-23-5_HandSoldering, symbol SVIELCOM_Library:REF1933AIDDCT
- added C? (x3): 0,22µF, Capacitor_SMD:C_0603_1608Metric_Pad1.08x0.95mm_HandSolder, symbol Device:C
- added C? (x3): 0,1µF, Capacitor_SMD:C_0603_1608Metric_Pad1.08x0.95mm_HandSolder, symbol Device:C
- added C? (x4): 10µFx35, symbol Device:CP
- added C? (x11): 1µF, Capacitor_SMD:C_0603_1608Metric_Pad1.08x0.95mm_HandSolder, symbol Device:C
- added C?: 10µFx16, symbol Device:CP
- added C? (x3): 330pF, Capacitor_SMD:C_0603_1608Metric_Pad1.08x0.95mm_HandSolder, symbol Device:C
- added D? (x6): 1N4743A, Diode_THT:D_DO-41_SOD81_P10.16mm_Horizontal, symbol Diode:1N47xxA
- added J? (x3): 22-23-2021, digikey-footprints:PinHeader_1x2_P2.54mm_Drill1.02mm, symbol dk_Rectangular-Connectors-Headers-Male-Pins:22-23-2021
- added L? (x2): B82790C0225N265, Inductor_SMD:L_Wuerth_WE-DD-Typ-L-Typ-XL-Typ-XXL, symbol Device:L_Core_Ferrite_Coupled
- added PS? (x2): TMH2415S, Converter_DCDC:Converter_DCDC_XP_POWER-IAxxxxS_THT, symbol Converter_DCDC:IA2415S
- added R? (x12): 1K, Resistor_SMD:R_0805_2012Metric_Pad1.20x1.40mm_HandSolder, symbol Device:R
- added R? (x12): 10K, Resistor_SMD:R_0805_2012Metric_Pad1.20x1.40mm_HandSolder, symbol Device:R
- added R? (x3): 2K, Resistor_SMD:R_0805_2012Metric_Pad1.20x1.40mm_HandSolder, symbol Device:R
- added R? (x6): 4,125K, Resistor_SMD:R_0805_2012Metric_Pad1.20x1.40mm_HandSolder, symbol Device:R
- added R? (x3): 1,1K, Resistor_SMD:R_0805_2012Metric_Pad1.20x1.40mm_HandSolder, symbol Device:R
- added TP? (x12): TestPoint, symbol Connector:TestPoint
- added U?: LT1129CST-5#PBF, Package_TO_SOT_SMD:SOT-223-3_TabPin2, symbol SVIELCOM_Library:LT1129CST-5#PBF
- added U?: REF1933AIDDCT, Package_TO_SOT_SMD:SOT-23-5_HandSoldering, symbol SVIELCOM_Library:REF1933AIDDCT
- added U? (x5): TLV9001IDBVR, Package_TO_SOT_SMD:SOT-23-5_HandSoldering, symbol Amplifier_Operational:TLV9001IDCK
- added U? (x2): ISO224ADWVR, Texas_Instruments-DWV0008A-0-0-*, symbol Схема-и-печатная-плата-rescue:ISO224ADWVR-Isolator
- L?: value L_Core_Ferrite_Coupled -> B82790C0225N265
Connections:
- net +24V: now reaches PS?.1 (+Vin)
- net +24V: now also C?.1, C?.1, C?.1, C?.1, PS?.1 (+Vin), PS?.1 (+Vin), U?.1 (VIN)
- net GNDREF: now reaches PS?.2 (-Vin)
- net GNDREF: now also U?.2 (V-), U?.5 (GND2), C?.1, C?.1, C?.1, C?.2, C?.2, C?.2, C?.2, C?.2, C?.2, C?.2, C?.2, C?.2, C?.2, PS?.2 (-Vin), PS?.2 (-Vin), R?.1, R?.1, R?.1, R?.1, R?.1, R?.1, U?.2 (GND), U?.2 (GND), U?.2 (V-), U?.2 (V-), U?.2 (V-), U?.2 (V-), U?.2 (V-), U?.5 (GND2), U?.5 (GND2)
- net at PS?.4 (-Vout): now also L?.4, U?.4 (GND1), C?.2, C?.2, C?.2, C?.2, D?.2 (A), TP?.1
- net at PS?.6 (+Vout): now also U?.3 (VDD1), C?.1, C?.1, TP?.1
- net at L?.1: now also J?.1
- net at L?.2: now also R?.2
- net at L?.3: now also J?.2
- net at U?.1 (VCAP): now also C?.1
- net at U?.2 (IN): now also C?.1, D?.2 (A), R?.1, TP?.1
- net at U?.6 (OUTN): now also R?.2
- net at U?.7 (OUTP): now also R?.2
- net +5V_Analog: now reaches U?.8 (VDD2)
- net +5V_Analog: now also U?.5 (V+), C?.1, C?.1, C?.2, C?.2, C?.2, R?.2, R?.2, R?.2, U?.3 (EN), U?.3 (OUTPUT), U?.4 (VIN), U?.5 (V+), U?.5 (V+), U?.5 (V+), U?.5 (V+), U?.5 (V+), U?.8 (VDD2), U?.8 (VDD2)
- net at U?.1 (+): now also R?.1, R?.2
- net at U?.3 (-): now also R?.1, R?.1
- net at U?.4: now also R?.1
- new net: D?.1 (K), D?.1 (K) (x3)
- new net: R?.1, R?.1, R?.2, U?.1 (+) (x3)
- new net: R?.1, R?.1, R?.2, U?.3 (-) (x3)
- new net: R?.1, R?.2, U?.4 (x3)
- new net: J?.1, L?.1 (x2)
- new net: L?.2, R?.2 (x2)
- new net: J?.2, L?.3 (x2)
- new net: C?.2, C?.2, C?.2, C?.2, D?.2 (A), L?.4, PS?.4 (-Vout), TP?.1, U?.4 (GND1) (x2)
- new net: C?.1, U?.1 (VCAP) (x2)
- new net: C?.1, D?.2 (A), R?.1, TP?.1, U?.2 (IN) (x2)
- new net: C?.1, C?.1, PS?.6 (+Vout), TP?.1, U?.3 (VDD1) (x2)
- new net: R?.2, U?.6 (OUTN) (x2)
- new net: R?.2, U?.7 (OUTP) (x2)
- new net: R?.1, R?.2, U?.1 (+) (x2)
- new net: R?.1, R?.1, U?.3 (-) (x2)
- new net: R?.1, U?.4 (x2)
- new net ADC1_P: C?.1, R?.2, TP?.1
- new net ADC2_P: C?.1, R?.2, TP?.1
- new net ADC3_P: C?.1, R?.2, TP?.1
- new net A_CH1_FAULT: R?.2, R?.2
- new net A_CH2_FAULT: R?.2, R?.2
- new net A_CH3_FAULT: R?.2, R?.2
- new net Ref_1,65V: C?.1, R?.2, R?.2, R?.2, U?.1 (VBIAS)
- no-connect marks 0 -> 4
Other:
- moved on the sheet: L?, PS?, U?

Commit message: ISO1211
Parts:
- added C?: 0,1µF, Capacitor_SMD:C_0603_1608Metric_Pad1.08x0.95mm_HandSolder, symbol Device:C
- added D?: BZV85-C56.113, Diode_THT:D_DO-41_SOD81_P10.16mm_Horizontal, symbol Diode:1N47xxA
- added D?: 2W10G-E4/51, Diode_THT:Diode_Bridge_Round_D9.8mm, symbol SVIELCOM_Library:2W10G
- added R?: 82K, Resistor_SMD:R_0805_2012Metric_Pad1.20x1.40mm_HandSolder, symbol Device:R
- added R?: 560, Resistor_SMD:R_0805_2012Metric_Pad1.20x1.40mm_HandSolder, symbol Device:R
- added R?: 15K, Resistor_SMD:R_0805_2012Metric_Pad1.20x1.40mm_HandSolder, symbol Device:R
Connections:
- net GNDREF: now also U?.4 (GND1)
- net VDD_PER: now reaches U?.1 (VCC1)
- net VDD_PER: now also U?.2 (EN)
- net at U?.6 (FGND): now also C?.2, D?.2 (A), D?.4 (-), R?.2
- net at U?.7 (IN): now also R?.2
- net at U?.8 (SENSE): now also C?.1, D?.1 (K), D?.2 (+), R?.1, R?.1
- new net: D?.3, R?.2
- no-connect marks 4 -> 5
Changed lines of the file:
@@
 L Isolator:ISO1211 U?
 U 1 1 60D8FFFC
-P 13900 3710
+P 13900 3700
 AR Path="/60D8FFFC" Ref="U?"  Part="1"
 AR Path="/60D8C564/60D8FFFC" Ref="U?"  Part="1"
-F 0 "U?" H 13900 4191 50  0000 C CNN
-F 1 "ISO1211DR" H 13900 4100 50  0000 C CNN
-F 2 "Package_SO:SOIC-8_3.9x4.9mm_P1.27mm" H 13900 2960 50  0001 C CNN
-F 3 "http://www.ti.com/lit/ds/symlink/iso1211.pdf" H 13850 3760 50  0001 C CNN
-	1    13900 3710
+F 0 "U?" H 13550 4050 50  0000 C CNN
+F 1 "ISO1211DR" H 13670 3970 50  0000 C CNN
+F 2 "Package_SO:SOIC-8_3.9x4.9mm_P1.27mm" H 13900 2950 50  0001 C CNN
+F 3 "http://www.ti.com/lit/ds/symlink/iso1211.pdf" H 13850 3750 50  0001 C CNN
+	1    13900 3700
 	1    0    0    -1
 $EndComp
@@
 	1    0    0    -1
 $EndComp
+Wire Wire Line
+	12200 4000 11180 4000
+Wire Wire Line
+	11180 3200 11580 3200
+$Comp
+L Device:R R?
+U 1 1 60B676E2
+P 13250 3700
+AR Path="/60B676E2" Ref="R?"  Part="1"
+AR Path="/60A03F8A/60B676E2" Ref="R?"  Part="1"
+AR Path="/60D8C564/60B676E2" Ref="R?"  Part="1"
+F 0 "R?" V 13470 3720 50  0000 C CNN
+F 1 "560" V 13390 3720 50  0000 C CNN
+F 2 "Resistor_SMD:R_0805_2012Metric_Pad1.20x1.40mm_HandSolder" V 13180 3700 50  0001 C CNN
+F 3 "~" H 13250 3700 50  0001 C CNN
+	1    13250 3700
+	0    -1   -1   0
+$EndComp
+Wire Wire Line
+	12600 3600 12640 3600
+Wire Wire Line
+	13100 3700 13010 3700
+Wire Wire Line
+	13010 3700 13010 3600
+Connection ~ 13010 3600
+Wire Wire Line
+	13010 3600 13400 3600
+Wire Wire Line
+	13400 4100 13400 3900
+NoConn ~ 13400 3800
+$Comp
+L Device:C C?
+U 1 1 60BE1F29
+P 13010 3900
+AR Path="/60BE1F29" Ref="C?"  Part="1"
+AR Path="/60A03F8A/60BE1F29" Ref="C?"  Part="1"
+AR Path="/60D8C564/60BE1F29" Ref="C?"  Part="1"
+F 0 "C?" H 13190 3870 50  0000 L CNN
+F 1 "0,1µF" H 13110 3790 50  0000 L CNN
+F 2 "Capacitor_SMD:C_0603_1608Metric_Pad1.08x0.95mm_HandSolder" H 13048 3750 50  0001 C CNN
+F 3 "http://www.farnell.com/datasheets/2710676.pdf" H 13010 3900 50  0001 C CNN
+F 4 "CL10B105KA8NNNC" H 13010 3900 50  0001 C CNN "Type"
+	1    13010 3900
+	1    0    0    -1
+$EndComp
+Wire Wire Line
+	13010 4050 13010 4100
+Connection ~ 13010 4100
+Wire Wire Line
+	13010 4100 13400 4100
+Wire Wire Line
+	13010 3750 13010 3700
+Connection ~ 13010 3700
+$Comp
+L Device:R R?
+U 1 1 60B0A699
+P 11730 3200
+AR Path="/60B0A699" Ref="R?"  Part="1"
+AR Path="/60A03F8A/60B0A699" Ref="R?"  Part="1"
+AR Path="/60D8C564/60B0A699" Ref="R?"  Part="1"
+F 0 "R?" V 11890 3210 50  0000 C CNN
+F 1 "82K" V 11820 3200 50  0000 C CNN
+F 2 "Resistor_SMD:R_0805_2012Metric_Pad1.20x1.40mm_HandSolder" V 11660 3200 50  0001 C CNN
+F 3 "~" H 11730 3200 50  0001 C CNN
+	1    11730 3200
+	0    -1   -1   0
+$EndComp
+$Comp
+L Device:R R?
+U 1 1 60C2A5C4
+P 12640 3860
+AR Path="/60C2A5C4" Ref="R?"  Part="1"
+AR Path="/60A03F8A/60C2A5C4" Ref="R?"  Part="1"
+AR Path="/60D8C564/60C2A5C4" Ref="R?"  Part="1"
+F 0 "R?" H 12450 3890 50  0000 C CNN
+F 1 "15K" H 12470 3820 50  0000 C CNN
+F 2 "Resistor_SMD:R_0805_2012Metric_Pad1.20x1.40mm_HandSolder" V 12570 3860 50  0001 C CNN
+F 3 "~" H 12640 3860 50  0001 C CNN
+	1    12640 3860
+	1    0    0    -1
+$EndComp
+Wire Wire Line
+	12640 3710 12640 3600
+Connection ~ 12640 3600
+Wire Wire Line
+	12640 3600 12810 3600
+Wire Wire Line
+	12640 4010 12640 4100
+Connection ~ 12640 4100
+Wire Wire Line
+	12640 4100 12810 4100
+$Comp
+L Diode:1N47xxA D?
+U 1 1 60C5B600
+P 12810 3870
+F 0 "D?" V 13110 3830 50  0000 L CNN
+F 1 "BZV85-C56.113" V 13190 3550 50  0000 L CNN
+F 2 "Diode_THT:D_DO-41_SOD81_P10.16mm_Horizontal" H 12810 3695 50  0001 C CNN
+F 3 "https://www.vishay.com/docs/85816/1n4728a.pdf" H 12810 3870 50  0001 C CNN
+	1    12810 3870
+	0    1    1    0
+$EndComp
+Wire Wire Line
+	12810 3720 12810 3600
+Connection ~ 12810 3600
+Wire Wire Line
+	12810 3600 13010 3600
+Wire Wire Line
+	12810 4020 12810 4100
+Connection ~ 12810 4100
+Wire Wire Line
+	12810 4100 13010 4100
+Wire Wire Line
+	11880 3200 12200 3200
+Wire Wire Line
+	11800 3600 11800 4100
+Wire Wire Line
+	11800 4100 12640 4100
+$Comp
+L SVIELCOM_Library:2W10G D?
+U 1 1 60DE8FAC
+P 12200 3600
+F 0 "D?" H 12260 3940 50  0000 L CNN
+F 1 "2W10G-E4/51" H 12250 3870 50  0000 L CNN
+F 2 "Diode_THT:Diode_Bridge_Round_D9.8mm" H 12400 3800 60  0001 L CNN
+F 3 "http://www.farnell.com/datasheets/2047189.pdf" H 12400 3900 60  0001 L CNN
+F 4 "Diodes - Bridge Rectifiers" H 12400 4300 60  0001 L CNN "Family"
+F 5 "BRIDGE RECT 1P 1000V" H 12400 4600 60  0001 L CNN "Description"
+	1    12200 3600
+	1    0    0    -1
+$EndComp
+$Comp
+L power:GNDREF #PWR?
+U 1 1 60DEFE4B
+P 14000 4100
+AR Path="/60DEFE4B" Ref="#PWR?"  Part="1"
+AR Path="/60A03F8A/60DEFE4B" Ref="#PWR?"  Part="1"
+AR Path="/60D8C564/60DEFE4B" Ref="#PWR?"  Part="1"
+F 0 "#PWR?" H 14000 3850 50  0001 C CNN
+F 1 "GNDREF" V 14005 3972 50  0001 R CNN
+F 2 "" H 14000 4100 50  0001 C CNN
+F 3 "" H 14000 4100 50  0001 C CNN
+	1    14000 4100
+	1    0    0    -1
+$EndComp
+$Comp
+L SVIELCOM_Library:VDD_PER #PWR?
+U 1 1 60DF50DD
+P 14000 3320
+F 0 "#PWR?" H 14000 3170 50  0001 C CNN
+F 1 "VDD_PER" H 14015 3493 50  0000 C CNN
+F 2 "" H 14000 3320 50  0001 C CNN
+F 3 "" H 14000 3320 50  0001 C CNN
+	1    14000 3320
+	1    0    0    -1
+$EndComp
+Wire Wire Line
+	14000 3400 14000 3360
+Wire Wire Line
+	14000 3360 14540 3360
+Wire Wire Line
+	14540 3360 14540 3900
+Wire Wire Line
+	14540 3900 14400 3900
+Connection ~ 14000 3360
+Wire Wire Line
+	14000 3360 14000 3320
 $EndSCHEMATC

Commit message: Digital IO ended
Parts:
- added D?: D, symbol Device:D
- added LS?: HCM1203X, symbol Device:Speaker_Crystal
- added Q? (x2): BC817-25LT1G, digikey-footprints:SOT-23-3, symbol dk_Transistors-Bipolar-BJT-Single:BC817-25LT1G
- added R? (x2): 5,1K, Resistor_SMD:R_0805_2012Metric_Pad1.20x1.40mm_HandSolder, symbol Device:R
- added RL?: G2RL-1-E-DC5, Relay_THT:Relay_DPDT_Omron_G2RL, symbol SVIELCOM_Library:G2RL-1-E-DC5
Connections:
- net GNDREF: now also Q?.2 (E), Q?.2 (E)
- net VDD_PER: now also LS?.1
- net 220V_Phase: now reaches R?.1
- net LEVEL_SWITCH: now reaches U?.3 (OUT)
- net LEVEL_SWITCH_AC: now reaches D?.1
- new net: Q?.1 (B), R?.1 (x2)
- new net: D?.2 (A), Q?.3 (C), RL?.8
- new net: LS?.2, Q?.3 (C)
- new net +5V: D?.1 (K), RL?.1
- new net SKIP_N_UNLOADED_REL: R?.2
- new net SKIP_N_UNLOADED_SOUD: R?.2
- new net SKIP_N_UNL_REL_NC: RL?.2, RL?.7
- new net SKIP_N_UNL_REL_NO: RL?.4, RL?.5
- new net SKIP_N_UNL_REL_SW: RL?.3, RL?.6
Other:
- moved on the sheet: C?, D?, R?, U?
