File: Indicator.sch (KiCad schematic (older format))
At the start: 6 parts, among them U10 BC56-12SURKWA, U11 SC56-11SRWA, U12 MAX7219EWG+T, U8 CC56-12SURKWA, U9 MAX7219EWG+T

Commit message: Indication edit
Parts:
- added U? (x2): CC56-12SURKWA, Display_7Segment:CA56-12SURKWA, symbol SVIELCOM_Library:CC56-12SURKWA
- U10: footprint Display_7Segment:CA56-12SURKWA -> SVIELCOM:BC56-11SURKWA
Connections:
- net CC5: now reaches U12.10 (DIG_5)
- net CC1: now reaches U12.11 (DIG_1)
- net A2: now reaches U12.14 (SEG_A)
- net A2: now also U10.16 (a3), U10.21 (a2), U10.25 (a1), U11.7 (A), U?.11 (a)
- net F2: now reaches U12.15 (SEG_F)
- net B2: now reaches U12.16 (SEG_B)
- net G2: now reaches U12.17 (SEG_G)
- net CC0: now reaches U12.2 (DIG_0)
- net C2: now reaches U12.20 (SEG_C)
- net E2: now reaches U12.21 (SEG_E)
- net DP2: now reaches U12.22 (SEG_DP)
- net D2: now reaches U12.23 (SEG_D)
- net CC4: now reaches U12.3 (DIG_4)
- net CC6: now reaches U12.5 (DIG_6)
- net CC2: now reaches U12.6 (DIG_2)
- net CC3: now reaches U12.7 (DIG_3)
- net CC7: now reaches U12.8 (DIG_7)
- net at U11.3 (CC): now also U11.8 (CC)
- net at U10.1 (e1): now also U10.10 (e3), U10.6 (e2)
- net at U10.11 (d3): now also U10.2 (d1), U10.7 (d2)
- net at U10.12 (g3): now also U10.22 (g2), U10.28 (g1)
- net at U10.13 (c3): now also U10.4 (c1), U10.8 (c2)
- net at U10.14 (DP3): now also U10.5 (DP1), U10.9 (DP2)
- net at U10.15 (b3): now also U10.20 (b2), U10.24 (b1)
- net at U10.17 (f3): now also U10.23 (f2), U10.27 (f1)
- net at U10.26 (CC1): now also U10.3 (CC1)
Other:
- note added: ""No Смены""
- note added: ""No Цикла""
- note added: ""Вес""
- note added: ""Время""
- note added: ""Дата""
- moved on the sheet: D2, U10, U11, U12, U8, U9

Commit message: Indication edit end
Parts:
- added D?: L-1154ID, LED_THT:LED_D3.0mm, symbol Device:LED
- added Q? (x2): BC817-25LT1G, digikey-footprints:SOT-23-3, symbol dk_Transistors-Bipolar-BJT-Single:BC817-25LT1G
- added R? (x2): 17,1K, Resistor_SMD:R_0805_2012Metric_Pad1.20x1.40mm_HandSolder, symbol Device:R
- added R? (x2): 100, Resistor_SMD:R_0805_2012Metric_Pad1.20x1.40mm_HandSolder, symbol Device:R
- added R? (x2): 5,1K, Resistor_SMD:R_0805_2012Metric_Pad1.20x1.40mm_HandSolder, symbol Device:R
Connections:
- net CC0 is gone; now on net 2C0: U12.2 (DIG_0)
- net CC1 is gone; now on net 2C1: U12.11 (DIG_1)
- net CC2 is gone; now on net 2C2: U12.6 (DIG_2)
- net CC3 is gone; now on net 2C3: U12.7 (DIG_3)
- net CC4 is gone; now on net 2C4: U12.3 (DIG_4)
- net CC5 is gone; now on net 2C5: U12.10 (DIG_5)
- net CC6 is gone; now on net 2C6: U12.5 (DIG_6)
- net CC7 is gone; now on net 2C7: U12.8 (DIG_7)
- net B2: now also U10.15 (b3), U10.20 (b2), U10.24 (b1), U11.6 (B), U?.7 (b)
- net C2: now also U10.13 (c3), U10.4 (c1), U10.8 (c2), U11.4 (C), U?.4 (c)
- net D2: now also U10.11 (d3), U10.2 (d1), U10.7 (d2), U11.2 (D), U?.2 (d)
- net DP2: now also U10.14 (DP3), U10.5 (DP1), U10.9 (DP2), U11.5 (DP), U?.3 (DPX)
- net E2: now also U10.1 (e1), U10.10 (e3), U10.6 (e2), U11.1 (E), U?.1 (e)
- net F2: now also U10.17 (f3), U10.23 (f2), U10.27 (f1), U11.9 (F), U?.10 (f)
- net G2: now also U10.12 (g3), U10.22 (g2), U10.28 (g1), U11.10 (G), U?.5 (g)
- net SPI6_MOSI: now reaches U9.1 (DIN)
- net 1C5: now reaches U9.10 (DIG_5)
- net 1C5: now also U8.8 (CC3)
- net 1C1: now reaches U9.11 (DIG_1)
- net 1C1: now also U?.8 (CC3)
- net SPI6_CS: now reaches U9.12 (LOAD)
- net SPI6_CS: now also U12.12 (LOAD)
- net SPI6_SCK: now reaches U9.13 (CLK)
- net SPI6_SCK: now also U12.13 (CLK)
- net A1: now reaches U9.14 (SEG_A)
- net A1: now also U8.11 (a), U?.11 (a)
- net F1: now reaches U9.15 (SEG_F)
- net F1: now also U8.10 (f), U?.10 (f)
- net B1: now reaches U9.16 (SEG_B)
- net B1: now also U8.7 (b), U?.7 (b)
- net G1: now reaches U9.17 (SEG_G)
- net G1: now also U8.5 (g), U?.5 (g)
- net at U9.18 (ISET): now also R?.2
- net +5V: now reaches U9.19 (V+)
- net +5V: now also U12.19 (V+), R?.1, R?.1, R?.1, R?.1
- net 1C0: now reaches U9.2 (DIG_0)
- net 1C0: now also U?.6 (CC4)
- net C1: now reaches U9.20 (SEG_C)
- net C1: now also U8.4 (c), U?.4 (c)
- net E1: now reaches U9.21 (SEG_E)
- net E1: now also U8.1 (e), U?.1 (e)
- net DP1: now reaches U9.22 (SEG_DP)
- net DP1: now also U8.3 (DPX), U?.3 (DPX)
- net D1: now reaches U9.23 (SEG_D)
- net D1: now also U8.2 (d), U?.2 (d)
- net at U9.24 (DOUT): now also U12.1 (DIN)
- net 1C4: now reaches U9.3 (DIG_4)
- net 1C4: now also U8.6 (CC4)
- net GNDREF: now reaches U9.4 (GND), U9.9 (GND)
- net GNDREF: now also U12.4 (GND), U12.9 (GND), Q?.2 (E), Q?.2 (E)
- net 1C6: now reaches U9.5 (DIG_6)
- net 1C6: now also U8.9 (CC2)
- net 1C2: now reaches U9.6 (DIG_2)
- net 1C2: now also U?.9 (CC2)
- net 1C3: now reaches U9.7 (DIG_3)
- net 1C3: now also U?.12 (CC1)
- net 1C7: now reaches U9.8 (DIG_7)
- net 1C7: now also U8.12 (CC1)
- net at U12.18 (ISET): now also R?.2
- net 2C3: now reaches U11.3 (CC), U11.8 (CC)
- net 2C0: now reaches U10.18 (CC3)
- net 2C1: now reaches U10.19 (CC2)
- net 2C2: now reaches U10.26 (CC1), U10.3 (CC1)
- net at D2.1 (K): now also Q?.3 (C)
- net at D2.2 (A): now also R?.2
- net 2C7: now reaches U?.12 (CC1)
- net 2C4: now reaches U?.6 (CC4)
- net 2C5: now reaches U?.8 (CC3)
- net 2C6: now reaches U?.9 (CC2)
- new net: D?.1 (K), Q?.3 (C)
- new net: D?.2 (A), R?.2
- new net: Q?.1 (B), R?.1 (x2)
- new net EAST_SKIP_LED: R?.2
- new net WEST_SKIP_LED: R?.2
- no-connect marks 0 -> 1
Other:
- moved on the sheet: D2

Commit message: Digital IO ended
Other:
- note added: ""EAST""
- note added: ""WEST""
- moved on the sheet: D2, D?, Q?, R?
