File: Schema_and_PCB.kicad_pcb (KiCad board)
At the start: 4 copper layers, 291.6 x 143.3 mm, 321 parts, among them J1 USB4085-GF-A_REVA, J10 22-23-2021, J11 Pulse_JXD6-0001NL, J12 OSTTC020162, J13 640456-2, J14 640456-3, J15 640456-3, J16 0022232041, J17 0022232041, J2 OSTTC020162, J3 OSTTC020162, J4 DM3AT-SF-PEJM5, J5 OSTTC020162, J6 22-23-2021, J7 OSTTC030162, J8 22-23-2021, J9 0022232031, Q1 BC817-25LT1G, Q2 BC817-25LT1G, Q3 BC817-25LT1G, Q4 BC817-25LT1G, SW1 SW_PUSHBUTTON, SW2 SW_PUSHBUTTON, SW3 SW_PUSHBUTTON, SW4 SW_PUSHBUTTON, SW5 SW_PUSHBUTTON, SW6 SW_PUSHBUTTON, U1 CC56-12SURKWA, U10 TLV75529PDBV, U11 STM32H743ZIT6, U12 LD1117S33CTR, U13 LD1117S33CTR, U14 SN74AVCA406DGGR, U15 W25Q256JVFIQ, U16 LT1129CST-5#PBF, U17 ISO1211DR, U18 ISO224ADWVR, U19 TLV9001IDBVR, U2 CC56-12SURKWA, U20 TLV9001IDBVR, U21 ISO224ADWVR, U22 TLV9001IDBVR, U23 TLV9001IDBVR, U24 ISO1211DR, U25 REF1933AIDDCT, U26 ISO1211DR, U27 ISO224ADWVR, U28 TLV9001IDBVR, U29 TLV9001IDBVR, U3 MAX7219EWG+T, U30 LAN8742A-CZ-TR, U4 BC56-12SURKWA, U5 SC56-11SRWA, U6 MAX7219EWG+T, U7 CC56-12SURKWA, U8 ADUM4160, U9 ST1L05APU33R, Y1 NX5032GA-8MHz, Y2 NX3215SA-32.768K-STD-MUA-14, Y3 NX2016SA-25MHz

Commit message: main PCB changes
Parts:
- removed C51, C60, C72: 10µFx35, Capacitor_Tantalum_SMD:CP_EIA-7343-30_AVX-N_Pad2.25x2.55mm_HandSolder
- removed C52, C58, C59, C62, C67, C68, C70, C71, C73: 1µF, Capacitor_SMD:C_0603_1608Metric_Pad1.08x0.95mm_HandSolder
- removed C53: 10µFx16, Capacitor_Tantalum_SMD:CP_EIA-3216-10_Kemet-I
- removed C55, C63, C76: 0.1µF, Capacitor_SMD:C_0603_1608Metric_Pad1.08x0.95mm_HandSolder
- removed C56, C64, C77: 0.22µF, Capacitor_SMD:C_0603_1608Metric_Pad1.08x0.95mm_HandSolder
- removed C57, C65, C78: 330pF, Capacitor_SMD:C_0603_1608Metric_Pad1.08x0.95mm_HandSolder
- removed D10, D13, D14, D6, D7, D9: 1N4743A, Diode_THT:D_DO-41_SOD81_P10.16mm_Horizontal
- removed J10, J6, J8: 22-23-2021, digikey-footprints:PinHeader_1x2_P2.54mm_Drill1.02mm
- removed L3, L4, L5: B82790C0225N265, SVIELCOM:B82790C0225N265
- removed PS1, PS2, PS3: TMH2415S, Converter_DCDC:Converter_DCDC_XP_POWER-IAxxxxS_THT
- removed R24, R35, R41, R51, R58, R69: 3.3K, Resistor_SMD:R_0603_1608Metric_Pad0.98x0.95mm_HandSolder
- removed R25, R32, R42, R48, R59, R66: 825, Resistor_SMD:R_0603_1608Metric_Pad0.98x0.95mm_HandSolder
- removed R28, R44, R62: 1K, Resistor_THT:R_Axial_DIN0207_L6.3mm_D2.5mm_P10.16mm_Horizontal
- removed R29, R31, R33, R34, R45, R47, R49, R50, R63, R65, R67, R68: 10K, Resistor_SMD:R_0805_2012Metric_Pad1.20x1.40mm_HandSolder
- removed R30, R46, R64: 1.1K, Resistor_SMD:R_0805_2012Metric_Pad1.20x1.40mm_HandSolder
- removed R36, R52, R70: 2K, Resistor_SMD:R_0805_2012Metric_Pad1.20x1.40mm_HandSolder
- removed R37, R38, R39, R53, R54, R55, R71, R72, R73: 1K, Resistor_SMD:R_0805_2012Metric_Pad1.20x1.40mm_HandSolder
- removed TP10, TP11, TP12, TP13, TP14, TP15, TP17, TP18, TP20, TP21, TP22, TP5, TP6, TP8, TP9: TestPoint, TestPoint:TestPoint_Pad_D1.5mm
- removed U16: LT1129CST-5#PBF, Package_TO_SOT_SMD:SOT-223-3_TabPin2
- removed U18, U21, U27: ISO224ADWVR, SVIELCOM:Texas_Instruments-DWV0008A-0-0-IPC_A
- removed U19, U20, U22, U23, U28, U29: TLV9001IDBVR, Package_TO_SOT_SMD:SOT-23-5_HandSoldering
- removed U25: REF1933AIDDCT, Package_TO_SOT_SMD:SOT-23-5_HandSoldering
- C48, C50: value 1µF -> 330pF
- C49: value 10µFx35 -> 330pF; footprint Capacitor_Tantalum_SMD:CP_EIA-7343-30_AVX-N_Pad2.25x2.55mm_HandSolder -> Capacitor_SMD:C_0603_1608Metric_Pad1.08x0.95mm_HandSolder
- C61, D8, Q4, R43: moved to B.Cu
- J3: value OSTTC020162 -> 302-S101; footprint digikey-footprints:Term_Block_1x2_P5mm -> digikey-footprints:PinHeader_2x5_P2.54mm_Drill1.2mm
- moved C13 205.2 mm to (86.2, 104.4), turned to 180 degrees
- moved J3 172.2 mm to (105.7, 75.2)
- moved C39 148.2 mm to (151.5, 129.8)
- moved C49 144.0 mm to (116.1, 156.4)
- moved C50 142.8 mm to (116.3, 159.3)
- moved R16 141.0 mm to (150.6, 96.5)
- moved C34 138.2 mm to (104.1, 103.9)
- moved R18 136.8 mm to (100.3, 100.1), turned to 180 degrees
- moved JP5 136.7 mm to (104.6, 100.1)
- moved C48 126.1 mm to (116.0, 153.2)
- moved D11 121.9 mm to (327.9, 97.3), turned to 180 degrees
- moved R43 121.3 mm to (212.9, 94.5), turned to 90 degrees
- moved LS1 120.6 mm to (221.0, 86.9), turned to 270 degrees
- moved Q4 116.9 mm to (216.7, 94.5)
- moved R57 112.0 mm to (313.4, 97.0), turned to 90 degrees
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Connections:
- net /Analog_and_digital_IO/220V_Phase renamed /Digital_IO_analog_Inputs/220V_Phase
- net /Analog_and_digital_IO/ENCODER_A renamed /Digital_IO_analog_Inputs/ENCODER_A
- net /Analog_and_digital_IO/ENCODER_B renamed /Digital_IO_analog_Inputs/ENCODER_B
- net /Analog_and_digital_IO/LEVEL_SWITCH renamed /Digital_IO_analog_Inputs/LEVEL_SWITCH
- net /Analog_and_digital_IO/LEVEL_SWITCH_AC renamed /Digital_IO_analog_Inputs/LEVEL_SWITCH_AC
- net /Analog_and_digital_IO/SKIP_N_UNLOADED_BEEPER renamed /Digital_IO_analog_Inputs/SKIP_N_UNLOADED_BEEPER
- net /Analog_and_digital_IO/SKIP_N_UNLOADED_REL renamed /Digital_IO_analog_Inputs/SKIP_N_UNLOADED_REL
- C48 pad 1: +24V -> /Digital_IO_analog_Inputs/ADC1_P
- C49 pad 1: +24V -> /Digital_IO_analog_Inputs/ADC2_P
- C50 pad 1: Net-(C50-Pad1) -> /Digital_IO_analog_Inputs/ADC3_P
- C50 pad 2: Net-(C50-Pad2) -> GNDREF
- J3 pad 2: +24V -> /Digital_IO_analog_Inputs/ADC1_P
- U11 pad 14: /Analog_and_digital_IO/A_CH3_FAULT -> /Digital_IO_analog_Inputs/A_CH3_FAULT
- U11 pad 15: /Analog_and_digital_IO/ADC3_P -> /Digital_IO_analog_Inputs/ADC3_P
- U11 pad 49: /Analog_and_digital_IO/A_CH1_FAULT -> /Digital_IO_analog_Inputs/ADC3_P
- U11 pad 50: /Analog_and_digital_IO/ADC1_P -> /Digital_IO_analog_Inputs/ADC1_P
- U11 pad 53: /Analog_and_digital_IO/ADC2_P -> /Digital_IO_analog_Inputs/ADC2_P
- U11 pad 54: /Analog_and_digital_IO/A_CH2_FAULT -> /Digital_IO_analog_Inputs/A_CH2_FAULT
Other:
- board size 291.6 x 143.3 mm -> 293.6 x 143.3 mm
