File: Schema_and_PCB.kicad_pcb (KiCad board)
At the start: 4 copper layers, 293.6 x 143.3 mm, 217 parts, among them J1 USB4085-GF-A_REVA, J11 Pulse_JXD6-0001NL, J12 Ground, J13 640456-2, J14 640456-3, J15 640456-3, J16 0022232041, J17 0022232041, J2 OSTTC020162, J3 302-S101, J4 DM3AT-SF-PEJM5, J5 OSTTC020162, J7 OSTTC030162, J9 0022232031, Q1 BC817-25LT1G, Q2 BC817-25LT1G, Q3 BC817-25LT1G, Q4 BC817-25LT1G, SW1 SW_PUSHBUTTON, SW2 SW_PUSHBUTTON, SW3 SW_PUSHBUTTON, SW4 SW_PUSHBUTTON, SW5 SW_PUSHBUTTON, SW6 SW_PUSHBUTTON, U1 CC56-12SURKWA, U10 TLV75529PDBV, U11 STM32H743ZIT6, U12 LD1117S33CTR, U13 LD1117S33CTR, U14 SN74AVCA406DGGR, U15 W25Q256JVFIQ, U17 ISO1211DR, U2 CC56-12SURKWA, U24 ISO1211DR, U26 ISO1211DR, U3 MAX7219EWG+T, U30 LAN8742A-CZ-TR, U4 BC56-12SURKWA, U5 SC56-11SRWA, U6 MAX7219EWG+T, U7 CC56-12SURKWA, U8 ADUM4160, U9 ST1L05APU33R, Y1 NX5032GA-8MHz, Y2 NX3215SA-32.768K-STD-MUA-14, Y3 NX2016SA-25MHz

Commit message: Indicators layout finished
Parts:
- added C43: 1µF, Capacitor_SMD:C_0603_1608Metric_Pad1.08x0.95mm_HandSolder, F.Cu at (221.1, 153.1)
- added C44: 1µF, Capacitor_SMD:C_0603_1608Metric_Pad1.08x0.95mm_HandSolder, F.Cu at (219.5, 121.7)
- Q4, R43: moved to F.Cu
- R3, R6, R7, R8: moved to B.Cu
- moved J13 41.7 mm to (134.3, 62.6)
- moved J15 38.6 mm to (174.3, 49.2)
- moved J14 38.3 mm to (106.6, 53.8)
- moved J16 34.9 mm to (152.7, 56.0)
- moved J17 29.4 mm to (146.7, 53.6)
- moved C28 26.8 mm to (151.7, 118.4)
- moved R17 25.7 mm to (151.3, 124.9)
- moved JP4 25.7 mm to (151.7, 121.6)
- moved R79 23.5 mm to (118.2, 185.1)
- moved R75 20.2 mm to (111.4, 189.3)
- moved R78 20.2 mm to (118.4, 188.9)
- moved R76 20.2 mm to (112.2, 180.5)
- moved R77 20.2 mm to (112.2, 185.1)
- moved R21 19.2 mm to (131.9, 113.6), turned to 90 degrees
- moved L3 14.1 mm to (133.7, 184.9)
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Connections:
- U11 pad 117: /Microcontroller/SD_CARD_CS -> /Microcontroller/SD_CARD_INS
- U11 pad 118: /Microcontroller/SD_CARD_INS -> /Microcontroller/SD_CARD_CS
Routing:
- net +5V: track 205.3 -> 574.7 mm, vias 0 -> 7
- net /Indicator/B2: track 0.00 -> 197.3 mm, vias 0 -> 4
- net /Indicator/A2: track 0.00 -> 166.7 mm, vias 0 -> 4
- net /Indicator/DP2: track 0.00 -> 166.2 mm, vias 0 -> 1
- net /Indicator/D2: track 0.00 -> 165.8 mm, vias 0 -> 2
- net /Indicator/G2: track 0.00 -> 162.7 mm, vias 0 -> 3
- net Net-(BT1-Pad1): track 0.00 -> 162.3 mm, vias 0 -> 2
- net /Indicator/F2: track 0.00 -> 153.2 mm, vias 0 -> 3
- net /Indicator/C2: track 0.00 -> 151.1 mm, vias 0 -> 4
- net /MCU_Power_supply_clocking/BOOT0: track 0.00 -> 135.2 mm, vias 0 -> 2
- net /Indicator/E2: track 0.00 -> 129.4 mm
- net /Buttons/Button_Plus: track 0.00 -> 120.7 mm
- net /Indicator/DP1: track 0.00 -> 118.1 mm, vias 0 -> 2
- net /Indicator/D1: track 0.00 -> 110.5 mm, vias 0 -> 3
- net /Indicator/C1: track 0.00 -> 108.7 mm, vias 0 -> 2
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- added copper zone on F.Cu, net Net-(U17-Pad5)
Other:
- net class Indicators added: clearance 0.2, trace_width 0.2, via_dia 0.6, via_drill 0.3

Commit message: Draft PCB done
Parts:
- R74, R75, R76, R77, R78, R79: moved to B.Cu
- moved BT1 156.9 mm to (97.6, 104.3)
- moved J15 145.2 mm to (124.1, 185.4), turned to 270 degrees
- moved J14 134.6 mm to (148.2, 181.8), turned to 180 degrees
- moved J16 130.4 mm to (136.2, 185.4), turned to 270 degrees
- moved J3 118.8 mm to (96.5, 195.9), turned to 180 degrees
- moved R76 69.3 mm to (181.3, 176.4), turned to 90 degrees
- moved R77 66.6 mm to (178.2, 176.4), turned to 90 degrees
- moved R75 59.1 mm to (169.1, 176.4), turned to 90 degrees
- moved R78 58.1 mm to (175.2, 176.4), turned to 90 degrees
- moved R79 54.6 mm to (172.1, 176.4), turned to 90 degrees
- moved R74 48.9 mm to (166.0, 176.4), turned to 90 degrees
- moved L3 26.7 mm to (160.2, 188.5)
- moved J17 23.3 mm to (145.9, 76.9)
- moved J13 14.3 mm to (132.4, 76.8)
- moved R1 10.3 mm to (201.5, 189.3)
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Connections:
- U11 pad 110: Net-(U11-Pad110) -> /Digital_IO_analog_Inputs/LEVEL_SWITCH
- U11 pad 14: /Digital_IO_analog_Inputs/A_CH3_FAULT -> Net-(U11-Pad14)
- U11 pad 141: Net-(U11-Pad141) -> /Digital_IO_analog_Inputs/SKIP_N_UNLOADED_REL
- U11 pad 142: Net-(U11-Pad142) -> /Digital_IO_analog_Inputs/SKIP_N_UNLOADED_BEEPER
- U11 pad 49: /Digital_IO_analog_Inputs/A_CH1_FAULT -> Net-(U11-Pad49)
- U11 pad 54: /Digital_IO_analog_Inputs/A_CH2_FAULT -> Net-(U11-Pad54)
- U11 pad 75: Net-(U11-Pad75) -> /Digital_IO_analog_Inputs/A_CH2_FAULT
- U11 pad 76: Net-(U11-Pad76) -> /Digital_IO_analog_Inputs/A_CH3_FAULT
- U11 pad 77: Net-(U11-Pad77) -> /Digital_IO_analog_Inputs/A_CH1_FAULT
- U11 pad 78: /Digital_IO_analog_Inputs/LEVEL_SWITCH -> Net-(U11-Pad78)
- U11 pad 79: /Digital_IO_analog_Inputs/SKIP_N_UNLOADED_REL -> Net-(U11-Pad79)
- U11 pad 85: /Digital_IO_analog_Inputs/SKIP_N_UNLOADED_BEEPER -> Net-(U11-Pad85)
- U11 pad 89: /Buttons/Button_Emh -> /Buttons/Button_Func
- U11 pad 90: /Buttons/Button_Clock -> /Buttons/Button_pH
- U11 pad 91: /Buttons/Button_pH -> /Buttons/Button_Clock
- U11 pad 92: /Buttons/Button_Func -> /Buttons/Button_Emh
Routing:
- net /Digital_IO_analog_Inputs/SKIP_N_UNLOADED_REL: track 0.00 -> 200.6 mm, vias 0 -> 2
- net /Digital_IO_analog_Inputs/ENCODER_B: track 7.20 -> 201.1 mm, vias 0 -> 2
- net /Digital_IO_analog_Inputs/LEVEL_SWITCH: track 7.18 -> 200.3 mm
- net Net-(C51-Pad1): track 108.1 -> 291.2 mm, vias 0 -> 3
- net /Digital_IO_analog_Inputs/ENCODER_A: track 7.51 -> 189.5 mm, vias 0 -> 2
- net /Digital_IO_analog_Inputs/SKIP_N_UNLOADED_BEEPER: track 0.00 -> 112.9 mm, vias 0 -> 2
- net /Indicator/WEST_SKIP_LED: track 1.57 -> 97.5 mm, vias 1 -> 2
- net /Buttons/Button_Plus: track 120.7 -> 210.4 mm, vias 0 -> 3
- net /Buttons/Button_Minus: track 99.5 -> 187.9 mm, vias 0 -> 3
- net /Indicator/SPI6_MOSI: track 4.76 -> 91.9 mm, vias 0 -> 2
- net /Digital_IO_analog_Inputs/ADC3_P: track 3.75 -> 81.4 mm
- net /Buttons/Button_Emh: track 89.9 -> 161.4 mm, vias 0 -> 3
- net /Digital_IO_analog_Inputs/ADC1_P: track 4.06 -> 75.1 mm, vias 0 -> 1
- net /Digital_IO_analog_Inputs/ADC2_P: track 4.29 -> 75.1 mm, vias 0 -> 1
- net /Digital_IO_analog_Inputs/A_CH2_FAULT: track 0.00 -> 69.1 mm, vias 0 -> 1
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
Commit message: PCB minor changes
Parts:
- C66, C74, R56, R60: moved to B.Cu
- J13: value 640456-2 -> I2C
- JP3: value Jumper_3_Bridged12 -> BOOT0
- moved C74 5.75 mm to (310.8, 79.4)
- moved JP3 2.68 mm to (87.0, 84.4)
- turned C66 to 90 degrees
Connections:
- net Net-(C74-Pad1) renamed /Digital_IO_analog_Inputs/ENCODER_IN_B
Routing:
- net /Digital_IO_analog_Inputs/ENCODER_IN_B: track 47.8 -> 40.2 mm, vias 0 -> 1
- net /Storage_and_memory/QUADPSI_BK1_IO0: track 22.6 -> 27.1 mm
- net /Digital_IO_analog_Inputs/ENCODER_IN_A: track 54.9 -> 58.9 mm, vias 0 -> 1
- net /Indicator/B2: track 197.3 -> 200.1 mm
- net GNDREF: track 299.3 -> 302.0 mm, vias 105 -> 147
- net Net-(JP3-Pad2): track 9.84 -> 7.65 mm
- net VDD_MCU: track 169.7 -> 171.9 mm, vias 37 -> 38
- net /Digital_IO_analog_Inputs/COM_ENCODER: track 31.7 -> 33.5 mm
- net Net-(J11-Pad9): track 11.9 -> 13.6 mm
- net NRST: track 107.9 -> 108.4 mm
- net /Indicator/D2: track 165.8 -> 166.3 mm
- net Net-(R56-Pad2): track 5.05 -> 5.08 mm, vias 0 -> 1
- net Net-(R60-Pad2): vias 0 -> 1
- added copper zone on F.Cu, net GNDREF
- removed copper zone on F.Cu, net Net-(U10-Pad4)
- removed copper zone on F.Cu, net VDD_PER
Other:
- net class Default: clearance 0.2 -> 0.125
- net class Indicators: clearance 0.2 -> 0.125
- net class Power: clearance 0.2 -> 0.125
- net class Thin: clearance 0.2 -> 0.125
- rule trace_clearance: 0.2 -> 0.125
- board text added: "+5V"
- board text added: "1"
- board text added: "ADC1_P"
- board text added: "ADC2_P"
- board text added: "ADC3_P"
- board text added: "A_CH1_FAULT"
- board text added: "A_CH2_FAULT"
- board text added: "A_CH3_FAULT"
- board text added: "BOOT0_RX"
- board text added: "BOOT0_TX"
- board text added: "COM"
- board text added: "ENCODER_IN"
- board text added: "GND"
- board text added: "IN_A"
- board text added: "IN_B"
- board text added: "LAN"
- board text added: "MISO"
- board text added: "MOSI"
- board text added: "Micro SD CARD"
- board text added: "NSS"
- board text added: "PERIPH SUPPLY"
- board text added: "Power"
- board text added: "RX"
- board text added: "SCK"
- board text added: "SPI"
- board text added: "SWDIO"
- board text added: "SWO"
- board text added: "SWSLK"
- board text added: "TX"
- board text added: "UART2"
- board text added: "USB"
- board text added: "VDD"
- board text added: "ШВУ 2.0"

Commit message: PCB before Gerber creating
Parts:
- removed S1: KS-01Q-01_Obsolete, digikey-footprints:PushButton_Round_D12mm_THT_KS-01Q-01
- added SW7: RESET, Button_Switch_THT:SW_PUSH_6mm, F.Cu at (78.3, 105.8)
- J13: value I2C -> 640456-3; footprint Connector_PinHeader_2.54mm:PinHeader_1x02_P2.54mm_Vertical -> Connector_PinHeader_2.54mm:PinHeader_1x03_P2.54mm_Vertical
- moved Q1 6.21 mm to (200.7, 179.7), turned to 0 degrees
- moved R1 3.49 mm to (199.0, 191.8)
- moved D1 1.41 mm to (199.0, 184.5)
- moved D2 1.41 mm to (157.9, 184.5)
- moved J13 0.06 mm to (132.5, 76.9)
- turned C14 to 0 degrees
Routing:
- net NRST: track 108.4 -> 103.0 mm
- net /Indicator/2C5: track 77.8 -> 72.8 mm
- net Net-(D1-Pad2): track 5.90 -> 7.88 mm
- net +5V: track 573.8 -> 571.9 mm
- net /Digital_IO_analog_Inputs/ADC1_P: track 75.1 -> 76.9 mm
- net /Indicator/G1: track 100.5 -> 102.2 mm
- net /Microcontroller/QUADSPI_CLK: track 43.0 -> 41.5 mm
- net Net-(D2-Pad2): track 4.51 -> 5.92 mm
- net /Digital_IO_analog_Inputs/ADC3_P: track 81.4 -> 80.0 mm
- net Net-(D1-Pad1): track 4.79 -> 5.96 mm
- net Net-(R21-Pad2): track 19.2 -> 18.2 mm
- net /Storage_and_memory/QUADPSI_BK1_IO1: track 24.3 -> 23.4 mm
- net GNDREF: track 302.0 -> 301.2 mm, vias 147 -> 170
- net /Indicator/E1: track 97.8 -> 98.5 mm
- net Net-(D2-Pad1): track 4.86 -> 5.45 mm
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- added copper zone on B.Cu, net GNDREF
Other:
- net class Default: clearance 0.125 -> 0.15
- net class Indicators: clearance 0.125 -> 0.2
- net class Power: clearance 0.125 -> 0.2
- net class Thin: clearance 0.125 -> 0.2
- rule trace_clearance: 0.125 -> 0.15
- board text added: "B_"
- board text added: "B_CLOCK"
- board text added: "B_Emh"
- board text added: "B_FUNC"
- board text added: "B_pH"
- board text added: "I2C"
- board text added: "PCB ver. 0.1 (02.06.2021)"
- board text added: "SCL"
- board text added: "SDA"
- board text added: "SWD"
- board text added: "Schema and PCB designed by SVIELCOM"
- board text added: "k"

Commit message: main PCB done. Gerbers sent to manufacturer
Routing:
- net VDD_MCU: track 171.9 -> 176.0 mm
- net GNDREF: track 301.2 -> 298.0 mm, vias 170 -> 168
- net /LAN/RMII_RXD1: track 28.0 -> 27.5 mm

Commit message: All vias changed
Parts:
- U9: value ST1L05APU33R -> DFN_5APU33R_STM
- moved C90 1.44 mm to (80.3, 148.2)
Routing:
- net /Buttons/Button_Emh: track 161.4 -> 16.2 mm, vias 3 -> 1
- net /Buttons/Button_Clock: track 139.6 -> 98.7 mm, vias 3 -> 2
- net /Buttons/Button_pH: track 118.7 -> 78.6 mm, vias 3 -> 2
- net /Buttons/Button_Func: track 96.7 -> 62.2 mm, vias 3 -> 2
- net /Buttons/Button_Minus: track 187.9 -> 155.8 mm, vias 3 -> 2
- net GNDREF: track 298.0 -> 311.1 mm
- net Net-(J4-Pad2): track 24.3 -> 20.5 mm
- net /Buttons/Button_Plus: track 210.4 -> 208.4 mm, vias 3 -> 2
- net Net-(J11-Pad10): track 26.0 -> 28.0 mm
- net /LAN/RD_P: track 18.0 -> 19.5 mm
- net VDD_MCU: track 176.0 -> 174.7 mm
- net /Microcontroller/SD_CARD_CS: track 67.8 -> 68.8 mm
- net /LAN/LAN_PWR: track 54.7 -> 55.6 mm
- net /Microcontroller/SDMMC1_CK: track 48.9 -> 49.4 mm
Other:
- net class Default: clearance 0.15 -> 0.2
- rule pad_to_mask_clearance: 0 -> 0.051
- rule trace_clearance: 0.15 -> 0.2

Commit message: All mounting holes changed
Parts:
- added REF**: MountingHole_3.7mm, MountingHole:MountingHole_3.7mm, F.Cu at (70.2, 187.1)
- added REF**: MountingHole_3.7mm, MountingHole:MountingHole_3.7mm, F.Cu at (70.2, 92.1)
- added REF**: MountingHole_3.7mm, MountingHole:MountingHole_3.7mm, F.Cu at (346.2, 92.9)
- added REF**: MountingHole_3.7mm, MountingHole:MountingHole_3.7mm, F.Cu at (346.2, 187.9)
- added REF**: MountingHole_3.7mm, MountingHole:MountingHole_3.7mm, F.Cu at (217.1, 161.5)
Routing:
- net /Buttons/Button_Emh: track 16.2 -> 161.5 mm, vias 1 -> 3
- net /Buttons/Button_Clock: track 98.7 -> 140.4 mm, vias 2 -> 3
- net /Buttons/Button_pH: track 78.6 -> 119.5 mm, vias 2 -> 3
- net /Buttons/Button_Func: track 62.2 -> 97.7 mm, vias 2 -> 3
- net /Buttons/Button_Minus: track 155.8 -> 189.1 mm, vias 2 -> 3
- net /Indicator/C2: track 151.1 -> 167.1 mm
- net /Indicator/D2: track 166.3 -> 151.8 mm, vias 2 -> 3
- net GNDREF: track 311.1 -> 300.4 mm, vias 168 -> 165
- net /Buttons/Button_Plus: track 208.4 -> 212.6 mm, vias 2 -> 3
- net /Microcontroller/BOOT0_TX: track 25.1 -> 28.4 mm
- net /MCU_Power_supply_clocking/BOOT0: track 139.6 -> 136.5 mm
- net /Microcontroller/BOOT0_RX: track 22.2 -> 25.4 mm
- net /Microcontroller/SWO: track 55.9 -> 58.5 mm
- net /Microcontroller/SWDIO: track 35.8 -> 38.4 mm
- net /Indicator/E2: track 129.4 -> 131.0 mm
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- added copper zone on F.Cu, net /USB/USB_GND
Other:
- outline, holes or cut-outs redrawn
- net class Default: clearance 0.2 -> 0.15; via_dia 0.6 -> 0.7
- net class Indicators: via_dia 0.6 -> 0.7
- net class Power: via_dia 0.6 -> 0.7
- net class Thin: via_dia 0.6 -> 0.7
- rule trace_clearance: 0.2 -> 0.15
- rule via_min_size: 0.6 -> 0.7
