File: Microcontroller.sch (KiCad schematic (older format))
At the start: 1 part

Commit message: begin MCU editing
Parts:
- added U? (x2): STM32H743ZIT6, QFP50P2200X2200X160-144N, symbol SVIELCOM_Library:STM32H743ZIT6
Connections:
- net BOOT0_TX: now reaches U?.101 (PA9)
- net BOOT0_RX: now reaches U?.102 (PA10)
- net USB_FS_DN: now reaches U?.103 (PA11)
- net USB_FS_DP: now reaches U?.104 (PA12)
- net SWDIO: now reaches U?.105 (PA13(JTMS-SWDIO))
- net SWCLK: now reaches U?.109 (PA14(JTCK/SWCLK))
- net SWO: now reaches U?.133 (PB3(JTDO/TRACESWO))
- net QUADSPI_BK1_NCS: now reaches U?.136 (PB6)
- net SDMMC1_CKIN: now reaches U?.139 (PB8)
- net RMII_REF_CLK: now reaches U?.35 (PA1)
- net RMII_MDIO: now reaches U?.36 (PA2)
- net RMII_CRS_DV: now reaches U?.43 (PA7)
- net RMII_TX_EN: now reaches U?.70 (PB11)
- net RMII_TXD0: now reaches U?.73 (PB12)
- net RMII_TXD1: now reaches U?.74 (PB13)
- no-connect marks 0 -> 17
Other:
- moved on the sheet: U?B
Changed lines of the file:
@@
 $Descr A4 11693 8268
 encoding utf-8
-Sheet 8 10
+Sheet 8 9
 Title ""
 Date ""
@@
 L SVIELCOM_Library:STM32H743ZIT6 U?
 U 2 1 60CDFA10
-P 4970 4060
+P 2630 2710
 AR Path="/60CDFA10" Ref="U?"  Part="2"
 AR Path="/60CDB738/60CDFA10" Ref="U?"  Part="2"
-F 0 "U?" H 5020 5727 50  0000 C CNN
-F 1 "STM32H743ZIT6" H 5020 5636 50  0000 C CNN
-F 2 "QFP50P2200X2200X160-144N" H 5020 5660 50  0001 L BNN
-F 3 "" H 5020 6060 50  0001 L BNN
-F 4 "STMicroelectronics" H 5020 5760 50  0001 L BNN "MANUFACTURER"
-F 5 "7" H 5020 6060 50  0001 L BNN "PARTREV"
-F 6 "1.6 mm" H 5020 5960 50  0001 L BNN "MAXIMUM_PACKAGE_HEIGHT"
-F 7 "IPC-7351B" H 5020 5860 50  0001 L BNN "STANDARD"
-	2    4970 4060
+F 0 "U?" H 2680 4377 50  0000 C CNN
+F 1 "STM32H743ZIT6" H 2680 4286 50  0000 C CNN
+F 2 "QFP50P2200X2200X160-144N" H 2680 4310 50  0001 L BNN
+F 3 "" H 2680 4710 50  0001 L BNN
+F 4 "STMicroelectronics" H 2680 4410 50  0001 L BNN "MANUFACTURER"
+F 5 "7" H 2680 4710 50  0001 L BNN "PARTREV"
+F 6 "1.6 mm" H 2680 4610 50  0001 L BNN "MAXIMUM_PACKAGE_HEIGHT"
+F 7 "IPC-7351B" H 2680 4510 50  0001 L BNN "STANDARD"
+	2    2630 2710
 	1    0    0    -1
 $EndComp
+$Comp
+L SVIELCOM_Library:STM32H743ZIT6 U?
+U 3 1 60FFD5D4
+P 7540 2710
+F 0 "U?" H 7540 4377 50  0000 C CNN
+F 1 "STM32H743ZIT6" H 7540 4286 50  0000 C CNN
+F 2 "QFP50P2200X2200X160-144N" H 7590 4310 50  0001 L BNN
+F 3 "" H 7590 4710 50  0001 L BNN
+F 4 "STMicroelectronics" H 7590 4410 50  0001 L BNN "MANUFACTURER"
+F 5 "7" H 7590 4710 50  0001 L BNN "PARTREV"
+F 6 "1.6 mm" H 7590 4610 50  0001 L BNN "MAXIMUM_PACKAGE_HEIGHT"
+F 7 "IPC-7351B" H 7590 4510 50  0001 L BNN "STANDARD"
+	3    7540 2710
+	1    0    0    -1
+$EndComp
+$Comp
+L SVIELCOM_Library:STM32H743ZIT6 U?
+U 4 1 6100866D
+P 7540 5640
+F 0 "U?" H 7540 7307 50  0000 C CNN
+F 1 "STM32H743ZIT6" H 7540 7216 50  0000 C CNN
+F 2 "QFP50P2200X2200X160-144N" H 7590 7240 50  0001 L BNN
+F 3 "" H 7590 7640 50  0001 L BNN
+F 4 "STMicroelectronics" H 7590 7340 50  0001 L BNN "MANUFACTURER"
+F 5 "7" H 7590 7640 50  0001 L BNN "PARTREV"
+F 6 "1.6 mm" H 7590 7540 50  0001 L BNN "MAXIMUM_PACKAGE_HEIGHT"
+F 7 "IPC-7351B" H 7590 7440 50  0001 L BNN "STANDARD"
+	4    7540 5640
+	1    0    0    -1
+$EndComp
+NoConn ~ 1780 1310
+Text HLabel 1780 1410 0    50   BiDi ~ 0
+RMII_REF_CLK
+Text HLabel 1780 1510 0    50   BiDi ~ 0
+RMII_MDIO
+NoConn ~ 1780 1610
+NoConn ~ 1780 1710
+NoConn ~ 1780 1810
+NoConn ~ 1780 1910
+Text HLabel 1780 2010 0    50   BiDi ~ 0
+RMII_CRS_DV
+NoConn ~ 1780 2110
+Wire Wire Line
+	1270 2210 1780 2210
+Wire Wire Line
+	1270 2310 1780 2310
+Text Label 1270 2210 0    50   ~ 0
+BOOT0_TX
+Text Label 1270 2310 0    50   ~ 0
+BOOT0_RX
+Text HLabel 1780 2410 0    50   BiDi ~ 0
+USB_FS_DN
+Text HLabel 1780 2510 0    50   BiDi ~ 0
+USB_FS_DP
+Wire Wire Line
+	1270 2610 1780 2610
+Text Label 1270 2610 0    50   ~ 0
+SWDIO
+Wire Wire Line
+	1270 2710 1780 2710
+Text Label 1270 2710 0    50   ~ 0
+SWCLK
+NoConn ~ 1780 2810
+NoConn ~ 1780 3010
+NoConn ~ 1780 3110
+NoConn ~ 1780 3210
+Wire Wire Line
+	1270 3310 1780 3310
+Text Label 1270 3310 0    50   ~ 0
+SWO
+NoConn ~ 1780 3410
+NoConn ~ 1780 3510
+Text HLabel 1780 3610 0    50   BiDi ~ 0
+QUADSPI_BK1_NCS
+NoConn ~ 1780 3710
+Text HLabel 1780 3810 0    50   BiDi ~ 0
+SDMMC1_CKIN
+NoConn ~ 1780 3910
+NoConn ~ 1780 4010
+Text HLabel 1780 4110 0    50   BiDi ~ 0
+RMII_TX_EN
+Text HLabel 1780 4210 0    50   BiDi ~ 0
+RMII_TXD0
+Text HLabel 1780 4310 0    50   BiDi ~ 0
+RMII_TXD1
+NoConn ~ 1780 4410
+NoConn ~ 1780 4510
 $EndSCHEMATC

Commit message: Probably pre-alpha version is done
Connections:
- net SDMMC1_D2: now reaches U?.111 (PC10)
- net SDMMC1_D3: now reaches U?.112 (PC11)
- net SDMMC1_CK: now reaches U?.113 (PC12)
- net RMII_MDC: now reaches U?.27 (PC1)
- net RMII_RXD0: now reaches U?.44 (PC4)
- net RMII_RXD1: now reaches U?.45 (PC5)
- net SDMMC1_D0: now reaches U?.98 (PC8)
- net SDMMC1_D1: now reaches U?.99 (PC9)
- net SPI4_SCK: now reaches U?.1 (PE2)
- net SDMMC1_CMD: now reaches U?.116 (PD2)
- net USART2_TX: now reaches U?.119 (PD5)
- net USART2_RX: now reaches U?.122 (PD6)
- net SPI4_NSS: now reaches U?.3 (PE4)
- net SPI4_MISO: now reaches U?.4 (PE5)
- net SPI4_MOSI: now reaches U?.5 (PE6)
- net LEVEL_SWITCH: now reaches U?.78 (PD9)
- net SKIP_N_UNLOADED_REL: now reaches U?.79 (PD10)
- net SKIP_N_UNLOADED_BEEPER: now reaches U?.85 (PD14)
- net I2C2_SDA: now reaches U?.10 (PF0)
- net I2C2_SCL: now reaches U?.11 (PF1)
- net EAST_SKIP_LED: now reaches U?.12 (PF2)
- net SPI6_CS: now reaches U?.127 (PG12)
- net SPI6_SCK: now reaches U?.128 (PG13)
- net SPI6_MOSI: now reaches U?.129 (PG14)
- net WEST_SKIP_LED: now reaches U?.13 (PF3)
- net A_CH3_FAULT: now reaches U?.14 (PF4)
- net ADC3_P: now reaches U?.15 (PF5)
- net QUADSPI_BK1_IO3: now reaches U?.18 (PF6)
- net QUADSPI_BK1_IO2: now reaches U?.19 (PF7)
- net QUADSPI_BK1_IO0: now reaches U?.20 (PF8)
- net QUADSPI_BK1_IO1: now reaches U?.21 (PF9)
- net QUADSPI_CLK: now reaches U?.22 (PF10)
- net A_CH1_FAULT: now reaches U?.49 (PF11)
- net ADC1_P: now reaches U?.50 (PF12)
- net ADC2_P: now reaches U?.53 (PF13)
- net A_CH2_FAULT: now reaches U?.54 (PF14)
- net Button_Plus: now reaches U?.87 (PG2)
- net Button_Minus: now reaches U?.88 (PG3)
- net Button_Emh: now reaches U?.89 (PG4)
- net Button_Clock: now reaches U?.90 (PG5)
- net Button_pH: now reaches U?.91 (PG6)
- net Button_Func: now reaches U?.92 (PG7)
- no-connect marks 17 -> 53

Commit message: v0.1
Parts:
- added J12: 640456-2, digikey-footprints:PinHeader_1x2_P2.54mm_Drill1.02mm, symbol dk_Rectangular-Connectors-Headers-Male-Pins:640456-2
- added J13, J14: 640456-3, digikey-footprints:PinHeader_1x3_P2.54_Drill1.1mm, symbol dk_Rectangular-Connectors-Headers-Male-Pins:640456-3
- added J15, J16: 0022232041, digikey-footprints:PinHeader_1x4_P2.54mm_Drill1.02mm, symbol dk_Rectangular-Connectors-Headers-Male-Pins:0022232041
- gave numbers to parts that had none: 1
Connections:
- net BOOT0_RX: now also J13.3
- net BOOT0_TX: now also J13.2
- net I2C2_SCL: now also J12.2
- net I2C2_SDA: now also J12.1
- net SPI4_MISO: now also J16.3
- net SPI4_MOSI: now also J16.4
- net SPI4_NSS: now also J16.2
- net SPI4_SCK: now also J16.1
- net SWCLK: now also J15.2
- net SWDIO: now also J15.3
- net SWO: now also J15.4
- net USART2_RX: now also J14.3
- net USART2_TX: now also J14.2
- new net GNDREF: J13.1, J14.1, J15.1
Changed lines of the file:
@@
 $Descr A4 11693 8268
 encoding utf-8
-Sheet 8 9
-Title ""
-Date ""
-Rev ""
-Comp ""
-Comment1 ""
+Sheet 9 9
+Title "ШВУ"
+Date "2021-03-25"
+Rev "V0.1"
+Comp "ЦВЕТМЕТНАЛАДКА"
+Comment1 "Шустов В.И."
 Comment2 ""
 Comment3 ""
@@
 P 2630 2710
 AR Path="/60CDFA10" Ref="U?"  Part="2"
-AR Path="/60CDB738/60CDFA10" Ref="U?"  Part="2"
-F 0 "U?" H 2680 4377 50  0000 C CNN
+AR Path="/60CDB738/60CDFA10" Ref="U11"  Part="2"
+F 0 "U11" H 2680 4377 50  0000 C CNN
 F 1 "STM32H743ZIT6" H 2680 4286 50  0000 C CNN
 F 2 "QFP50P2200X2200X160-144N" H 2680 4310 50  0001 L BNN
@@
 $EndComp
 $Comp
-L SVIELCOM_Library:STM32H743ZIT6 U?
+L SVIELCOM_Library:STM32H743ZIT6 U11
 U 3 1 60FFD5D4
 P 7540 2710
-F 0 "U?" H 7540 4377 50  0000 C CNN
+F 0 "U11" H 7540 4377 50  0000 C CNN
 F 1 "STM32H743ZIT6" H 7540 4286 50  0000 C CNN
 F 2 "QFP50P2200X2200X160-144N" H 7590 4310 50  0001 L BNN
@@
 $EndComp
 $Comp
-L SVIELCOM_Library:STM32H743ZIT6 U?
+L SVIELCOM_Library:STM32H743ZIT6 U11
 U 4 1 6100866D
 P 7540 5640
-F 0 "U?" H 7540 7307 50  0000 C CNN
+F 0 "U11" H 7540 7307 50  0000 C CNN
 F 1 "STM32H743ZIT6" H 7540 7216 50  0000 C CNN
 F 2 "QFP50P2200X2200X160-144N" H 7590 7240 50  0001 L BNN
@@
 NoConn ~ 8440 5040
 NoConn ~ 8440 5740
+Wire Wire Line
+	1350 6660 1980 6660
+Wire Wire Line
+	1350 6760 1980 6760
+Wire Wire Line
+	1350 6560 1980 6560
+$Comp
+L power:GNDREF #PWR?
+U 1 1 6129E864
+P 1490 7010
+AR Path="/6129E864" Ref="#PWR?"  Part="1"
+AR Path="/60A03F8A/6129E864" Ref="#PWR?"  Part="1"
+AR Path="/60D8C564/6129E864" Ref="#PWR?"  Part="1"
+AR Path="/60CDB738/6129E864" Ref="#PWR0118"  Part="1"
+F 0 "#PWR0118" H 1490 6760 50  0001 C CNN
+F 1 "GNDREF" V 1495 6882 50  0001 R CNN
+F 2 "" H 1490 7010 50  0001 C CNN
+F 3 "" H 1490 7010 50  0001 C CNN
+	1    1490 7010
+	1    0    0    -1
+$EndComp
+Text Label 1980 6560 2    50   ~ 0
+SWO
+Text Label 1980 6760 2    50   ~ 0
+SWCLK
+Text Label 1980 6660 2    50   ~ 0
+SWDIO
+$Comp
+L dk_Rectangular-Connectors-Headers-Male-Pins:640456-3 J13
+U 1 1 612A6373
+P 1250 5920
+F 0 "J13" V 1560 5880 50  0000 C CNN
+F 1 "640456-3" V 1120 5910 50  0000 C CNN
+F 2 "digikey-footprints:PinHeader_1x3_P2.54_Drill1.1mm" H 1450 6120 60  0001 L CNN
+F 3 "https://www.te.com/commerce/DocumentDelivery/DDEController?Action=srchrtrv&DocNm=640456&DocType=Customer+Drawing&DocLang=English" H 1450 6220 60  0001 L CNN
+F 4 "A19470-ND" H 1450 6320 60  0001 L CNN "Digi-Key_PN"
+F 5 "640456-3" H 1450 6420 60  0001 L CNN "MPN"
+F 6 "Connectors, Interconnects" H 1450 6520 60  0001 L CNN "Category"
+F 7 "Rectangular Connectors - Headers, Male Pins" H 1450 6620 60  0001 L CNN "Family"
+F 8 "https://www.te.com/commerce/DocumentDelivery/DDEController?Action=srchrtrv&DocNm=640456&DocType=Customer+Drawing&DocLang=English" H 1450 6720 60  0001 L CNN "DK_Datasheet_Link"
+F 9 "/product-detail/en/te-connectivity-amp-connectors/640456-3/A19470-ND/259010" H 1450 6820 60  0001 L CNN "DK_Detail_Page"
+F 10 "CONN HEADER VERT 3POS 2.54MM" H 1450 6920 60  0001 L CNN "Description"
+F 11 "TE Connectivity AMP Connectors" H 1450 7020 60  0001 L CNN "Manufacturer"
+F 12 "Active" H 1450 7120 60  0001 L CNN "Status"
+	1    1250 5920
+	0    1    -1   0
+$EndComp
+$Comp
+L dk_Rectangular-Connectors-Headers-Male-Pins:0022232041 J15
+U 1 1 612AA072
+P 1250 6860
+F 0 "J15" V 1650 6820 50  0000 C CNN
+F 1 "0022232041" V 1140 6820 50  0000 C CNN
+F 2 "digikey-footprints:PinHeader_1x4_P2.54mm_Drill1.02mm" H 1450 7060 60  0001 L CNN
+F 3 "https://www.molex.com/pdm_docs/sd/022232041_sd.pdf" H 1450 7160 60  0001 L CNN
+F 4 "WM4202-ND" H 1450 7260 60  0001 L CNN "Digi-Key_PN"
+F 5 "0022232041" H 1450 7360 60  0001 L CNN "MPN"
+F 6 "Connectors, Interconnects" H 1450 7460 60  0001 L CNN "Category"
+F 7 "Rectangular Connectors - Headers, Male Pins" H 1450 7560 60  0001 L CNN "Family"
+F 8 "https://www.molex.com/pdm_docs/sd/022232041_sd.pdf" H 1450 7660 60  0001 L CNN "DK_Datasheet_Link"
+F 9 "/product-detail/en/molex/0022232041/WM4202-ND/26671" H 1450 7760 60  0001 L CNN "DK_Detail_Page"
+F 10 "CONN HEADER VERT 4POS 2.54MM" H 1450 7860 60  0001 L CNN "Description"
+F 11 "Molex" H 1450 7960 60  0001 L CNN "Manufacturer"
+F 12 "Active" H 1450 8060 60  0001 L CNN "Status"
+	1    1250 6860
+	0    1    -1   0
+$EndComp
+Wire Wire Line
+	1350 6860 1490 6860
+Wire Wire Line
+	1490 6860 1490 7010
+$Comp
+L power:GNDREF #PWR?
+U 1 1 612B668B
+P 1490 6070
+AR Path="/612B668B" Ref="#PWR?"  Part="1"
+AR Path="/60A03F8A/612B668B" Ref="#PWR?"  Part="1"
+AR Path="/60D8C564/612B668B" Ref="#PWR?"  Part="1"
+AR Path="/60CDB738/612B668B" Ref="#PWR0116"  Part="1"
+F 0 "#PWR0116" H 1490 5820 50  0001 C CNN
+F 1 "GNDREF" V 1495 5942 50  0001 R CNN
+F 2 "" H 1490 6070 50  0001 C CNN
+F 3 "" H 1490 6070 50  0001 C CNN
+	1    1490 6070
+	1    0    0    -1
+$EndComp
+Wire Wire Line
+	1350 5920 1490 5920
+Wire Wire Line
+	1490 5920 1490 6070
+Wire Wire Line
+	1350 5720 1980 5720
+Wire Wire Line
+	1350 5820 1980 5820
+Text Label 1980 5820 2    50   ~ 0
+BOOT0_TX
+Text Label 1980 5720 2    50   ~ 0
+BOOT0_RX
+$Comp
+L dk_Rectangular-Connectors-Headers-Male-Pins:640456-3 J14
+U 1 1 612C1C26
+P 2430 5920
+F 0 "J14" V 2740 5880 50  0000 C CNN
+F 1 "640456-3" V 2300 5910 50  0000 C CNN
+F 2 "digikey-footprints:PinHeader_1x3_P2.54_Drill1.1mm" H 2630 6120 60  0001 L CNN
+F 3 "https://www.te.com/commerce/DocumentDelivery/DDEController?Action=srchrtrv&DocNm=640456&DocType=Customer+Drawing&DocLang=English" H 2630 6220 60  0001 L CNN
+F 4 "A19470-ND" H 2630 6320 60  0001 L CNN "Digi-Key_PN"
+F 5 "640456-3" H 2630 6420 60  0001 L CNN "MPN"
+F 6 "Connectors, Interconnects" H 2630 6520 60  0001 L CNN "Category"
+F 7 "Rectangular Connectors - Headers, Male Pins" H 2630 6620 60  0001 L CNN "Family"
+F 8 "https://www.te.com/commerce/DocumentDelivery/DDEController?Action=srchrtrv&DocNm=640456&DocType=Customer+Drawing&DocLang=English" H 2630 6720 60  0001 L CNN "DK_Datasheet_Link"
+F 9 "/product-detail/en/te-connectivity-amp-connectors/640456-3/A19470-ND/259010" H 2630 6820 60  0001 L CNN "DK_Detail_Page"
+F 10 "CONN HEADER VERT 3POS 2.54MM" H 2630 6920 60  0001 L CNN "Description"
+F 11 "TE Connectivity AMP Connectors" H 2630 7020 60  0001 L CNN "Manufacturer"
+F 12 "Active" H 2630 7120 60  0001 L CNN "Status"
+	1    2430 5920
+	0    1    -1   0
+$EndComp
+$Comp
+L power:GNDREF #PWR?
+U 1 1 612C1C2C
+P 2670 6070
+AR Path="/612C1C2C" Ref="#PWR?"  Part="1"
+AR Path="/60A03F8A/612C1C2C" Ref="#PWR?"  Part="1"
+AR Path="/60D8C564/612C1C2C" Ref="#PWR?"  Part="1"
+AR Path="/60CDB738/612C1C2C" Ref="#PWR0117"  Part="1"
+F 0 "#PWR0117" H 2670 5820 50  0001 C CNN
+F 1 "GNDREF" V 2675 5942 50  0001 R CNN
+F 2 "" H 2670 6070 50  0001 C CNN
+F 3 "" H 2670 6070 50  0001 C CNN
+	1    2670 6070
+	1    0    0    -1
+$EndComp
+Wire Wire Line
+	2530 5920 2670 5920
+Wire Wire Line
+	2670 5920 2670 6070
+Wire Wire Line
+	2530 5720 3160 5720
+Wire Wire Line
+	2530 5820 3160 5820
+Text Label 3160 5820 2    50   ~ 0
+USART2_TX
+Text Label 3160 5720 2    50   ~ 0
+USART2_RX
+Wire Wire Line
+	2530 6660 3160 6660
+Wire Wire Line
+	2530 6760 3160 6760
+Wire Wire Line
+	2530 6560 3160 6560
+$Comp
+L dk_Rectangular-Connectors-Headers-Male-Pins:0022232041 J16
+U 1 1 612D50A7
+P 2430 6860
+F 0 "J16" V 2830 6820 50  0000 C CNN
+F 1 "0022232041" V 2280 6800 50  0000 C CNN
+F 2 "digikey-footprints:PinHeader_1x4_P2.54mm_Drill1.02mm" H 2630 7060 60  0001 L CNN
+F 3 "https://www.molex.com/pdm_docs/sd/022232041_sd.pdf" H 2630 7160 60  0001 L CNN
+F 4 "WM4202-ND" H 2630 7260 60  0001 L CNN "Digi-Key_PN"
+F 5 "0022232041" H 2630 7360 60  0001 L CNN "MPN"
+F 6 "Connectors, Interconnects" H 2630 7460 60  0001 L CNN "Category"
+F 7 "Rectangular Connectors - Headers, Male Pins" H 2630 7560 60  0001 L CNN "Family"
+F 8 "https://www.molex.com/pdm_docs/sd/022232041_sd.pdf" H 2630 7660 60  0001 L CNN "DK_Datasheet_Link"
+F 9 "/product-detail/en/molex/0022232041/WM4202-ND/26671" H 2630 7760 60  0001 L CNN "DK_Detail_Page"
+F 10 "CONN HEADER VERT 4POS 2.54MM" H 2630 7860 60  0001 L CNN "Description"
+F 11 "Molex" H 2630 7960 60  0001 L CNN "Manufacturer"
+F 12 "Active" H 2630 8060 60  0001 L CNN "Status"
+	1    2430 6860
+	0    1    -1   0
+$EndComp
+Wire Wire Line
+	2530 6860 3160 6860
+Text Label 3160 6860 2    50   ~ 0
+SPI4_SCK
+Text Label 3160 6760 2    50   ~ 0
+SPI4_NSS
+Text Label 3160 6660 2    50   ~ 0
+SPI4_MISO
+Text Label 3160 6560 2    50   ~ 0
+SPI4_MOSI
+$Comp
+L dk_Rectangular-Connectors-Headers-Male-Pins:640456-2 J12
+U 1 1 612E235D
+P 3580 5720
+F 0 "J12" V 3460 5660 50  0000 C CNN
+F 1 "640456-2" V 3900 5740 50  0000 C CNN
+F 2 "digikey-footprints:PinHeader_1x2_P2.54mm_Drill1.02mm" H 3780 5920 60  0001 L CNN
+F 3 "https://www.te.com/commerce/DocumentDelivery/DDEController?Action=srchrtrv&DocNm=640456&DocType=Customer+Drawing&DocLang=English" H 3780 6020 60  0001 L CNN
+F 4 "A1921-ND" H 3780 6120 60  0001 L CNN "Digi-Key_PN"
+F 5 "640456-2" H 3780 6220 60  0001 L CNN "MPN"
+F 6 "Connectors, Interconnects" H 3780 6320 60  0001 L CNN "Category"
+F 7 "Rectangular Connectors - Headers, Male Pins" H 3780 6420 60  0001 L CNN "Family"
+F 8 "https://www.te.com/commerce/DocumentDelivery/DDEController?Action=srchrtrv&DocNm=640456&DocType=Customer+Drawing&DocLang=English" H 3780 6520 60  0001 L CNN "DK_Datasheet_Link"
+F 9 "/product-detail/en/te-connectivity-amp-connectors/640456-2/A1921-ND/109003" H 3780 6620 60  0001 L CNN "DK_Detail_Page"
+F 10 "CONN HEADER VERT 2POS 2.54MM" H 3780 6720 60  0001 L CNN "Description"
+F 11 "TE Connectivity AMP Connectors" H 3780 6820 60  0001 L CNN "Manufacturer"
+F 12 "Active" H 3780 6920 60  0001 L CNN "Status"
+	1    3580 5720
+	0    1    1    0
+$EndComp
+Wire Wire Line
+	3680 5720 4310 5720
+Wire Wire Line
+	3680 5820 4310 5820
+Text Label 4310 5720 2    50   ~ 0
+I2C2_SDA
+Text Label 4310 5820 2    50   ~ 0
+I2C2_SCL
 $EndSCHEMATC

Commit message: v0.2 added ecoder inputs
Connections:
- net ENCODER_A: now reaches U11.96 (PC6)
- net ENCODER_B: now reaches U11.97 (PC7)
- no-connect marks 53 -> 51
Changed lines of the file:
@@
 Wire Wire Line
 	3580 1810 4090 1810
-NoConn ~ 3580 1910
-NoConn ~ 3580 2010
 Text HLabel 4090 1410 2    50   BiDi ~ 0
 RMII_MDC
@@
 Text Label 4310 5820 2    50   ~ 0
 I2C2_SCL
+Wire Wire Line
+	3580 1910 4090 1910
+Text HLabel 4090 1910 2    50   Input ~ 0
+ENCODER_A
+Wire Wire Line
+	3580 2010 4090 2010
+Text HLabel 4090 2010 2    50   Input ~ 0
+ENCODER_B
 $EndSCHEMATC

Commit message: v0.3 changed sd_card holder
Parts:
- renumbered J12 to J13, J13 to J14, J14 to J15, J15 to J16, J16 to J17
Changed lines of the file:
@@
 AR Path="/60A03F8A/6129E864" Ref="#PWR?"  Part="1"
 AR Path="/60D8C564/6129E864" Ref="#PWR?"  Part="1"
-AR Path="/60CDB738/6129E864" Ref="#PWR0118"  Part="1"
-F 0 "#PWR0118" H 1490 6760 50  0001 C CNN
+AR Path="/60CDB738/6129E864" Ref="#PWR0122"  Part="1"
+F 0 "#PWR0122" H 1490 6760 50  0001 C CNN
 F 1 "GNDREF" V 1495 6882 50  0001 R CNN
 F 2 "" H 1490 7010 50  0001 C CNN
@@
 SWDIO
 $Comp
-L dk_Rectangular-Connectors-Headers-Male-Pins:640456-3 J13
+L dk_Rectangular-Connectors-Headers-Male-Pins:640456-3 J14
 U 1 1 612A6373
 P 1250 5920
-F 0 "J13" V 1560 5880 50  0000 C CNN
+F 0 "J14" V 1560 5880 50  0000 C CNN
 F 1 "640456-3" V 1120 5910 50  0000 C CNN
 F 2 "digikey-footprints:PinHeader_1x3_P2.54_Drill1.1mm" H 1450 6120 60  0001 L CNN
@@
 $EndComp
 $Comp
-L dk_Rectangular-Connectors-Headers-Male-Pins:0022232041 J15
+L dk_Rectangular-Connectors-Headers-Male-Pins:0022232041 J16
 U 1 1 612AA072
 P 1250 6860
-F 0 "J15" V 1650 6820 50  0000 C CNN
+F 0 "J16" V 1650 6820 50  0000 C CNN
 F 1 "0022232041" V 1140 6820 50  0000 C CNN
 F 2 "digikey-footprints:PinHeader_1x4_P2.54mm_Drill1.02mm" H 1450 7060 60  0001 L CNN
@@
 AR Path="/60A03F8A/612B668B" Ref="#PWR?"  Part="1"
 AR Path="/60D8C564/612B668B" Ref="#PWR?"  Part="1"
-AR Path="/60CDB738/612B668B" Ref="#PWR0116"  Part="1"
-F 0 "#PWR0116" H 1490 5820 50  0001 C CNN
+AR Path="/60CDB738/612B668B" Ref="#PWR0120"  Part="1"
+F 0 "#PWR0120" H 1490 5820 50  0001 C CNN
 F 1 "GNDREF" V 1495 5942 50  0001 R CNN
 F 2 "" H 1490 6070 50  0001 C CNN
@@
 BOOT0_RX
 $Comp
-L dk_Rectangular-Connectors-Headers-Male-Pins:640456-3 J14
+L dk_Rectangular-Connectors-Headers-Male-Pins:640456-3 J15
 U 1 1 612C1C26
 P 2430 5920
-F 0 "J14" V 2740 5880 50  0000 C CNN
+F 0 "J15" V 2740 5880 50  0000 C CNN
 F 1 "640456-3" V 2300 5910 50  0000 C CNN
 F 2 "digikey-footprints:PinHeader_1x3_P2.54_Drill1.1mm" H 2630 6120 60  0001 L CNN
@@
 AR Path="/60A03F8A/612C1C2C" Ref="#PWR?"  Part="1"
 AR Path="/60D8C564/612C1C2C" Ref="#PWR?"  Part="1"
-AR Path="/60CDB738/612C1C2C" Ref="#PWR0117"  Part="1"
-F 0 "#PWR0117" H 2670 5820 50  0001 C CNN
+AR Path="/60CDB738/612C1C2C" Ref="#PWR0121"  Part="1"
+F 0 "#PWR0121" H 2670 5820 50  0001 C CNN
 F 1 "GNDREF" V 2675 5942 50  0001 R CNN
 F 2 "" H 2670 6070 50  0001 C CNN
@@
 	2530 6560 3160 6560
 $Comp
-L dk_Rectangular-Connectors-Headers-Male-Pins:0022232041 J16
+L dk_Rectangular-Connectors-Headers-Male-Pins:0022232041 J17
 U 1 1 612D50A7
 P 2430 6860
-F 0 "J16" V 2830 6820 50  0000 C CNN
+F 0 "J17" V 2830 6820 50  0000 C CNN
 F 1 "0022232041" V 2280 6800 50  0000 C CNN
 F 2 "digikey-footprints:PinHeader_1x4_P2.54mm_Drill1.02mm" H 2630 7060 60  0001 L CNN
@@
 SPI4_MOSI
 $Comp
-L dk_Rectangular-Connectors-Headers-Male-Pins:640456-2 J12
+L dk_Rectangular-Connectors-Headers-Male-Pins:640456-2 J13
 U 1 1 612E235D
 P 3580 5720
-F 0 "J12" V 3460 5660 50  0000 C CNN
+F 0 "J13" V 3460 5660 50  0000 C CNN
 F 1 "640456-2" V 3900 5740 50  0000 C CNN
 F 2 "digikey-footprints:PinHeader_1x2_P2.54mm_Drill1.02mm" H 3780 5920 60  0001 L CNN

Commit message: footprints associations is done
Parts:
- U11: footprint QFP50P2200X2200X160-144N -> SVIELCOM:QFP50P2200X2200X160-144N
Changed lines of the file:
@@
 Title "ШВУ"
 Date "2021-03-25"
-Rev "V0.1"
+Rev "V0.3"
 Comp "ЦВЕТМЕТНАЛАДКА"
 Comment1 "Шустов В.И."
@@
 F 0 "U11" H 2680 4377 50  0000 C CNN
 F 1 "STM32H743ZIT6" H 2680 4286 50  0000 C CNN
-F 2 "QFP50P2200X2200X160-144N" H 2680 4310 50  0001 L BNN
+F 2 "SVIELCOM:QFP50P2200X2200X160-144N" H 2680 4310 50  0001 L BNN
 F 3 "" H 2680 4710 50  0001 L BNN
 F 4 "STMicroelectronics" H 2680 4410 50  0001 L BNN "MANUFACTURER"
@@
 F 0 "U11" H 7540 4377 50  0000 C CNN
 F 1 "STM32H743ZIT6" H 7540 4286 50  0000 C CNN
-F 2 "QFP50P2200X2200X160-144N" H 7590 4310 50  0001 L BNN
+F 2 "SVIELCOM:QFP50P2200X2200X160-144N" H 7590 4310 50  0001 L BNN
 F 3 "" H 7590 4710 50  0001 L BNN
 F 4 "STMicroelectronics" H 7590 4410 50  0001 L BNN "MANUFACTURER"
@@
 F 0 "U11" H 7540 7307 50  0000 C CNN
 F 1 "STM32H743ZIT6" H 7540 7216 50  0000 C CNN
-F 2 "QFP50P2200X2200X160-144N" H 7590 7240 50  0001 L BNN
+F 2 "SVIELCOM:QFP50P2200X2200X160-144N" H 7590 7240 50  0001 L BNN
 F 3 "" H 7590 7640 50  0001 L BNN
 F 4 "STMicroelectronics" H 7590 7340 50  0001 L BNN "MANUFACTURER"
@@
 AR Path="/60A03F8A/6129E864" Ref="#PWR?"  Part="1"
 AR Path="/60D8C564/6129E864" Ref="#PWR?"  Part="1"
-AR Path="/60CDB738/6129E864" Ref="#PWR0122"  Part="1"
-F 0 "#PWR0122" H 1490 6760 50  0001 C CNN
+AR Path="/60CDB738/6129E864" Ref="#PWR0125"  Part="1"
+F 0 "#PWR0125" H 1490 6760 50  0001 C CNN
 F 1 "GNDREF" V 1495 6882 50  0001 R CNN
 F 2 "" H 1490 7010 50  0001 C CNN
@@
 AR Path="/60A03F8A/612B668B" Ref="#PWR?"  Part="1"
 AR Path="/60D8C564/612B668B" Ref="#PWR?"  Part="1"
-AR Path="/60CDB738/612B668B" Ref="#PWR0120"  Part="1"
-F 0 "#PWR0120" H 1490 5820 50  0001 C CNN
+AR Path="/60CDB738/612B668B" Ref="#PWR0123"  Part="1"
+F 0 "#PWR0123" H 1490 5820 50  0001 C CNN
 F 1 "GNDREF" V 1495 5942 50  0001 R CNN
 F 2 "" H 1490 6070 50  0001 C CNN
@@
 AR Path="/60A03F8A/612C1C2C" Ref="#PWR?"  Part="1"
 AR Path="/60D8C564/612C1C2C" Ref="#PWR?"  Part="1"
-AR Path="/60CDB738/612C1C2C" Ref="#PWR0121"  Part="1"
-F 0 "#PWR0121" H 2670 5820 50  0001 C CNN
+AR Path="/60CDB738/612C1C2C" Ref="#PWR0124"  Part="1"
+F 0 "#PWR0124" H 2670 5820 50  0001 C CNN
 F 1 "GNDREF" V 2675 5942 50  0001 R CNN
 F 2 "" H 2670 6070 50  0001 C CNN
