File: Microcontroller.sch (KiCad schematic (older format))
At the start: 6 parts, among them J13 640456-2, J14 640456-3, J15 640456-3, J16 0022232041, J17 0022232041, U11 STM32H743ZIT6

Commit message: deleted TXS0206 added SN74AVCA406DGGR and corrected schema for it
Connections:
- net ENCODER_A: now also U11.134 (PB4(~JTRST~)); no longer U11.96 (PC6)
- net ENCODER_B: now also U11.135 (PB5); no longer U11.97 (PC7)
- net SDMMC1_CDIR: now reaches U11.140 (PB9)
- net SD_CARD_CS: now reaches U11.117 (PD3)
- net SD_CARD_INS: now reaches U11.118 (PD4)
- new net SDMMC1_D0DIR: U11.96 (PC6)
- new net SDMMC1_D123DIR: U11.97 (PC7)
- no-connect marks 51 -> 46
Changed lines of the file:
@@
 Text Label 1270 3310 0    50   ~ 0
 SWO
-NoConn ~ 1780 3410
-NoConn ~ 1780 3510
-Text HLabel 1270 3610 0    50   BiDi ~ 0
+Text HLabel 1270 3610 0    50   Output ~ 0
 QUADSPI_BK1_NCS
 NoConn ~ 1780 3710
 Text HLabel 1270 3810 0    50   Input ~ 0
 SDMMC1_CKIN
-NoConn ~ 1780 3910
 NoConn ~ 1780 4010
 Text HLabel 1270 4110 0    50   BiDi ~ 0
@@
 Text HLabel 6130 1510 0    50   BiDi ~ 0
 SDMMC1_CMD
-NoConn ~ 6640 1610
-NoConn ~ 6640 1710
 Wire Wire Line
 	6130 1810 6640 1810
@@
 Wire Wire Line
 	3580 1910 4090 1910
-Text HLabel 4090 1910 2    50   Input ~ 0
+Text HLabel 1270 3410 0    50   Input ~ 0
 ENCODER_A
 Wire Wire Line
 	3580 2010 4090 2010
-Text HLabel 4090 2010 2    50   Input ~ 0
+Text HLabel 1270 3510 0    50   Input ~ 0
 ENCODER_B
+Text HLabel 4090 1910 2    50   Output ~ 0
+SDMMC1_D0DIR
+Text HLabel 4090 2010 2    50   Output ~ 0
+SDMMC1_D123DIR
+Text HLabel 1270 3910 0    50   Output ~ 0
+SDMMC1_CDIR
+Wire Wire Line
+	1270 3910 1780 3910
+Text HLabel 6130 1710 0    50   Input ~ 0
+SD_CARD_INS
+Text HLabel 6130 1610 0    50   Output ~ 0
+SD_CARD_CS
+Wire Wire Line
+	6130 1610 6640 1610
+Wire Wire Line
+	6640 1710 6130 1710
+Wire Wire Line
+	1270 3410 1780 3410
+Wire Wire Line
+	1780 3510 1270 3510
 $EndSCHEMATC

Commit message: Footprints for pinheaders changed
Parts:
- J13: footprint digikey-footprints:PinHeader_1x2_P2.54mm_Drill1.02mm -> Connector_PinHeader_2.54mm:PinHeader_1x02_P2.54mm_Vertical
- J14, J15: footprint digikey-footprints:PinHeader_1x3_P2.54_Drill1.1mm -> Connector_PinHeader_2.54mm:PinHeader_1x03_P2.54mm_Vertical
- J16, J17: footprint digikey-footprints:PinHeader_1x4_P2.54mm_Drill1.02mm -> Connector_PinHeader_2.54mm:PinHeader_1x04_P2.54mm_Vertical
Changed lines of the file:
@@
 F 0 "J14" V 1560 5880 50  0000 C CNN
 F 1 "640456-3" V 1120 5910 50  0000 C CNN
-F 2 "digikey-footprints:PinHeader_1x3_P2.54_Drill1.1mm" H 1450 6120 60  0001 L CNN
+F 2 "Connector_PinHeader_2.54mm:PinHeader_1x03_P2.54mm_Vertical" H 1450 6120 60  0001 L CNN
 F 3 "https://www.te.com/commerce/DocumentDelivery/DDEController?Action=srchrtrv&DocNm=640456&DocType=Customer+Drawing&DocLang=English" H 1450 6220 60  0001 L CNN
 F 4 "A19470-ND" H 1450 6320 60  0001 L CNN "Digi-Key_PN"
@@
 F 0 "J16" V 1650 6820 50  0000 C CNN
 F 1 "0022232041" V 1140 6820 50  0000 C CNN
-F 2 "digikey-footprints:PinHeader_1x4_P2.54mm_Drill1.02mm" H 1450 7060 60  0001 L CNN
+F 2 "Connector_PinHeader_2.54mm:PinHeader_1x04_P2.54mm_Vertical" H 1450 7060 60  0001 L CNN
 F 3 "https://www.molex.com/pdm_docs/sd/022232041_sd.pdf" H 1450 7160 60  0001 L CNN
 F 4 "WM4202-ND" H 1450 7260 60  0001 L CNN "Digi-Key_PN"
@@
 F 0 "J15" V 2740 5880 50  0000 C CNN
 F 1 "640456-3" V 2300 5910 50  0000 C CNN
-F 2 "digikey-footprints:PinHeader_1x3_P2.54_Drill1.1mm" H 2630 6120 60  0001 L CNN
+F 2 "Connector_PinHeader_2.54mm:PinHeader_1x03_P2.54mm_Vertical" H 2630 6120 60  0001 L CNN
 F 3 "https://www.te.com/commerce/DocumentDelivery/DDEController?Action=srchrtrv&DocNm=640456&DocType=Customer+Drawing&DocLang=English" H 2630 6220 60  0001 L CNN
 F 4 "A19470-ND" H 2630 6320 60  0001 L CNN "Digi-Key_PN"
@@
 F 0 "J17" V 2830 6820 50  0000 C CNN
 F 1 "0022232041" V 2280 6800 50  0000 C CNN
-F 2 "digikey-footprints:PinHeader_1x4_P2.54mm_Drill1.02mm" H 2630 7060 60  0001 L CNN
+F 2 "Connector_PinHeader_2.54mm:PinHeader_1x04_P2.54mm_Vertical" H 2630 7060 60  0001 L CNN
 F 3 "https://www.molex.com/pdm_docs/sd/022232041_sd.pdf" H 2630 7160 60  0001 L CNN
 F 4 "WM4202-ND" H 2630 7260 60  0001 L CNN "Digi-Key_PN"
@@
 F 0 "J13" V 3460 5660 50  0000 C CNN
 F 1 "640456-2" V 3900 5740 50  0000 C CNN
-F 2 "digikey-footprints:PinHeader_1x2_P2.54mm_Drill1.02mm" H 3780 5920 60  0001 L CNN
+F 2 "Connector_PinHeader_2.54mm:PinHeader_1x02_P2.54mm_Vertical" H 3780 5920 60  0001 L CNN
 F 3 "https://www.te.com/commerce/DocumentDelivery/DDEController?Action=srchrtrv&DocNm=640456&DocType=Customer+Drawing&DocLang=English" H 3780 6020 60  0001 L CNN
 F 4 "A1921-ND" H 3780 6120 60  0001 L CNN "Digi-Key_PN"
