File: U_USB.sch (KiCad schematic (older format))
At the start: 15 parts, among them J1 USB4085-GF-A_REVA, U8 ADUM4160

Commit message: corrected few footprints, correct all resistors and capacitors type for ordering
Parts:
- C2: Type GRM188R7YA105KA12D -> CL10B105KA8NNNC
- L1: value 600R@100MHz [BK2125HS601-T] -> 600R@100MHz; Type (none) -> BK2125HS601-T
- R10, R11, R12, R13: Type (none) -> RC0805FR-0724RL
- R14, R15: value 5,1K -> 5.1K; Type (none) -> RC0805FR-075K1L
- R9: Type (none) -> RC0805FR-0710KL
Changed lines of the file:
@@
 AR Path="/6099558B/60CFFF64" Ref="R14"  Part="1"
 F 0 "R14" H 6190 5090 50  0000 L CNN
-F 1 "5,1K" H 6190 5000 50  0000 L CNN
+F 1 "5.1K" H 6190 5000 50  0000 L CNN
 F 2 "Resistor_SMD:R_0805_2012Metric_Pad1.20x1.40mm_HandSolder" V 6060 5040 50  0001 C CNN
 F 3 "~" H 6130 5040 50  0001 C CNN
+F 4 "RC0805FR-075K1L" H 6130 5040 50  0001 C CNN "Type"
 	1    6130 5040
 	1    0    0    -1
@@
 AR Path="/6099558B/60D0043D" Ref="R15"  Part="1"
 F 0 "R15" H 6480 5090 50  0000 L CNN
-F 1 "5,1K" H 6480 5000 50  0000 L CNN
+F 1 "5.1K" H 6480 5000 50  0000 L CNN
 F 2 "Resistor_SMD:R_0805_2012Metric_Pad1.20x1.40mm_HandSolder" V 6350 5040 50  0001 C CNN
 F 3 "~" H 6420 5040 50  0001 C CNN
+F 4 "RC0805FR-075K1L" H 6420 5040 50  0001 C CNN "Type"
 	1    6420 5040
 	1    0    0    -1
@@
 F 2 "Resistor_SMD:R_0805_2012Metric_Pad1.20x1.40mm_HandSolder" V 4860 3850 50  0001 C CNN
 F 3 "~" H 4930 3850 50  0001 C CNN
+F 4 "RC0805FR-0724RL" V 4930 3850 50  0001 C CNN "Type"
 	1    4930 3850
 	0    1    1    0
@@
 F 2 "Resistor_SMD:R_0805_2012Metric_Pad1.20x1.40mm_HandSolder" V 4860 3950 50  0001 C CNN
 F 3 "~" H 4930 3950 50  0001 C CNN
+F 4 "RC0805FR-0724RL" V 4930 3950 50  0001 C CNN "Type"
 	1    4930 3950
 	0    1    1    0
@@
 F 2 "Capacitor_SMD:C_0603_1608Metric_Pad1.08x0.95mm_HandSolder" H 3598 4730 50  0001 C CNN
 F 3 "https://www.farnell.com/datasheets/2048520.pdf" H 3560 4880 50  0001 C CNN
-F 4 "GRM188R7YA105KA12D" H 3560 4880 50  0001 C CNN "Type"
+F 4 "CL10B105KA8NNNC" H 3560 4880 50  0001 C CNN "Type"
 	1    3560 4880
 	1    0    0    -1
@@
 AR Path="/6099558B/60D586A1" Ref="L1"  Part="1"
 F 0 "L1" H 3792 2906 50  0000 L CNN
-F 1 "600R@100MHz [BK2125HS601-T]" H 3792 2815 50  0000 L CNN
+F 1 "600R@100MHz" H 3792 2815 50  0000 L CNN
 F 2 "Inductor_SMD:L_0805_2012Metric_Pad1.15x1.40mm_HandSolder" H 3740 2860 50  0001 C CNN
 F 3 "https://www.terraelectronica.ru/pdf/show?pdf_file=http%253A%252F%252Fwww.mouser.com%252Fds%252F2%252F396%252Fmlci07_e-9531.pdf" H 3740 2860 50  0001 C CNN
+F 4 "BK2125HS601-T" H 3740 2860 50  0001 C CNN "Type"
 	1    3740 2860
 	1    0    0    -1
@@
 F 2 "Resistor_SMD:R_0805_2012Metric_Pad1.20x1.40mm_HandSolder" V 3020 3850 50  0001 C CNN
 F 3 "~" H 3090 3850 50  0001 C CNN
+F 4 "RC0805FR-0724RL" V 3090 3850 50  0001 C CNN "Type"
 	1    3090 3850
 	0    1    1    0
@@
 F 2 "Resistor_SMD:R_0805_2012Metric_Pad1.20x1.40mm_HandSolder" V 3020 3950 50  0001 C CNN
 F 3 "~" H 3090 3950 50  0001 C CNN
+F 4 "RC0805FR-0724RL" V 3090 3950 50  0001 C CNN "Type"
 	1    3090 3950
 	0    1    1    0
@@
 F 2 "Resistor_SMD:R_0805_2012Metric_Pad1.20x1.40mm_HandSolder" V 3240 3380 50  0001 C CNN
 F 3 "~" H 3310 3380 50  0001 C CNN
+F 4 "RC0805FR-0710KL" H 3310 3380 50  0001 C CNN "Type"
 	1    3310 3380
 	-1   0    0    1

Commit message: ISO1211 power supply apdated. Label USB_GND added
Connections:
- net USB_GND: now reaches C3.2, C4.2, D3.2 (COM), D3.5 (COM), J1.A1 (GND), J1.A12 (GND), J1.B1 (GND), J1.B12 (GND), J1.P1 (SHELL), J1.P2 (SHELL), J1.P3 (SHELL), J1.P4 (SHELL), R14.2, R15.2, U8.2 (GND1), U8.8 (GND1)
Changed lines of the file:
@@
 NoConn ~ 6650 3840
 NoConn ~ 6650 3940
+Text Label 6490 5460 0    50   ~ 0
+USB_GND
 $EndSCHEMATC

Commit message: PCB autorouting attempt
Connections:
- net USB_DP: now reaches D3.3 (TVS2), J1.A6 (DP1), J1.B6 (DP2), R11.1
- net USB_DN: now reaches D3.4 (TVS3), J1.A7 (DN1), J1.B7 (DN2), R13.1
- net USB_VBUS: now reaches C4.1, J1.A4 (VBUS), J1.A9 (VBUS), J1.B4 (VBUS), J1.B9 (VBUS), U8.1 (VBUS1)
Changed lines of the file:
@@
 Text Label 6490 5460 0    50   ~ 0
 USB_GND
+Text Label 5660 3140 0    50   ~ 0
+USB_VBUS
+Text Label 5900 3340 0    50   ~ 0
+USB_DN
+Text Label 5900 3540 0    50   ~ 0
+USB_DP
 $EndSCHEMATC
