File: U_USB.sch (KiCad schematic (older format))
At the start: 15 parts, among them J1 USB4085-GF-A_REVA, U8 ADUM4160

Commit message: PCB layout
Connections:
- net USB_DN renamed USB_D_N
- net USB_DP renamed USB_D_P
Changed lines of the file:
@@
 USB_VBUS
 Text Label 5900 3340 0    50   ~ 0
-USB_DN
+USB_D_N
 Text Label 5900 3540 0    50   ~ 0
-USB_DP
+USB_D_P
 $EndSCHEMATC

Commit message: commit after KiCAD library updates
Parts:
- U8: symbol Interface_USB:ADUM4160 -> Schema_and_PCB-rescue:ADUM4160-Interface_USB
Changed lines of the file:
@@
 	5730 5350 5730 5460
 $Comp
-L Interface_USB:ADUM4160 U8
+L Schema_and_PCB-rescue:ADUM4160-Interface_USB U8
 U 1 1 60CF7C1F
 P 4150 3950
+AR Path="/60CF7C1F" Ref="U8"  Part="1"
+AR Path="/6099558B/60CF7C1F" Ref="U8"  Part="1"
 F 0 "U8" H 3780 4610 50  0000 C CNN
 F 1 "ADUM4160" H 3780 4520 50  0000 C CNN
