File: Buttons.sch (KiCad schematic (older format))
At the start: 24 parts, among them SW1 SW_PUSHBUTTON, SW2 SW_PUSHBUTTON, SW3 SW_PUSHBUTTON, SW4 SW_PUSHBUTTON, SW5 SW_PUSHBUTTON, SW6 SW_PUSHBUTTON

Commit message: PCB layout
Connections:
- net VDD_PER renamed VDD_MCU
Changed lines of the file:
@@
 Wire Wire Line
 	5370 5090 5370 5030
-$Comp
-L SVIELCOM_Library:VDD_PER #PWR?
-U 1 1 60D8F79A
-P 5370 1130
-AR Path="/60D8C564/60D8F79A" Ref="#PWR?"  Part="1"
-AR Path="/60CDBD15/60D8F79A" Ref="#PWR0109"  Part="1"
-F 0 "#PWR0109" H 5370 980 50  0001 C CNN
-F 1 "VDD_PER" H 5385 1303 50  0000 C CNN
-F 2 "" H 5370 1130 50  0001 C CNN
-F 3 "" H 5370 1130 50  0001 C CNN
-	1    5370 1130
-	1    0    0    -1
-$EndComp
 Wire Wire Line
 	5370 1210 5370 1130
@@
 Text Label 3820 4230 0    50   ~ 0
 PG7
+$Comp
+L SVIELCOM_Library:VDD_MCU #PWR?
+U 1 1 60E7C828
+P 5370 1130
+F 0 "#PWR?" H 5370 980 50  0001 C CNN
+F 1 "VDD_MCU" H 5400 1320 50  0000 C CNN
+F 2 "" H 5370 1130 50  0001 C CNN
+F 3 "" H 5370 1130 50  0001 C CNN
+	1    5370 1130
+	1    0    0    -1
+$EndComp
 $EndSCHEMATC

Commit message: PCB before Gerber creating
Changed lines of the file:
@@
 PG3
 Text Label 3820 2910 0    50   ~ 0
+PG7
+Text Label 3820 3350 0    50   ~ 0
+PG6
+Text Label 3820 3790 0    50   ~ 0
+PG5
+Text Label 3820 4230 0    50   ~ 0
 PG4
-Text Label 3820 3350 0    50   ~ 0
-PG5
-Text Label 3820 3790 0    50   ~ 0
-PG6
-Text Label 3820 4230 0    50   ~ 0
-PG7
 $Comp
 L SVIELCOM_Library:VDD_MCU #PWR0107
