File: LAN.sch (KiCad schematic (older format))
At the start: 35 parts, among them J11 Pulse_JXD6-0001NL, J12 OSTTC020162, U30 LAN8742A-CZ-TR, Y3 NX2016SA-25MHz

Commit message: Footprints for pinheaders changed
Parts:
- removed J12: OSTTC020162, digikey-footprints:Term_Block_1x2_P5mm, symbol dk_Terminal-Blocks-Wire-to-Board:OSTTC020162
- added J12: Ground, Connector_PinHeader_2.54mm:PinHeader_1x01_P2.54mm_Vertical, symbol Connector_Generic:Conn_01x01
Connections:
- net GNDS: now also J12.1 (Pin_1)
Changed lines of the file:
@@
 NRST
-$Comp
-L dk_Terminal-Blocks-Wire-to-Board:OSTTC020162 J12
-U 1 1 6119E96E
-P 10110 5930
-F 0 "J12" H 10020 5920 50  0000 R CNN
-F 1 "OSTTC020162" H 10020 6020 50  0000 R CNN
-F 2 "digikey-footprints:Term_Block_1x2_P5mm" H 10310 6130 60  0001 L CNN
-F 3 "http://www.on-shore.com/wp-content/uploads/OSTTCXX0162.pdf" H 10310 6230 60  0001 L CNN
-F 4 "ED2600-ND" H 10310 6330 60  0001 L CNN "Digi-Key_PN"
-F 5 "OSTTC020162" H 10310 6430 60  0001 L CNN "MPN"
-F 6 "Connectors, Interconnects" H 10310 6530 60  0001 L CNN "Category"
-F 7 "Terminal Blocks - Wire to Board" H 10310 6630 60  0001 L CNN "Family"
-F 8 "http://www.on-shore.com/wp-content/uploads/OSTTCXX0162.pdf" H 10310 6730 60  0001 L CNN "DK_Datasheet_Link"
-F 9 "/product-detail/en/on-shore-technology-inc/OSTTC020162/ED2600-ND/614549" H 10310 6830 60  0001 L CNN "DK_Detail_Page"
-F 10 "TERM BLK 2POS SIDE ENTRY 5MM PCB" H 10310 6930 60  0001 L CNN "Description"
-F 11 "On Shore Technology Inc." H 10310 7030 60  0001 L CNN "Manufacturer"
-F 12 "Active" H 10310 7130 60  0001 L CNN "Status"
-	1    10110 5930
-	-1   0    0    1
-$EndComp
 $Comp
 L power:GNDS #PWR0122
@@
 	1    0    0    -1
 $EndComp
-Wire Wire Line
-	10010 6130 10010 6210
-Wire Wire Line
-	10010 6210 10060 6210
-Wire Wire Line
-	10110 6130 10110 6210
-Wire Wire Line
-	10110 6210 10060 6210
-Connection ~ 10060 6210
 $Comp
 L power:PWR_FLAG #FLG013
@@
 	1    0    0    -1
 $EndComp
+Wire Wire Line
+	10060 6170 10060 6210
+$Comp
+L Connector_Generic:Conn_01x01 J12
+U 1 1 60B6A384
+P 10060 5970
+F 0 "J12" V 10030 5880 50  0000 R CNN
+F 1 "Ground" V 9930 5930 50  0000 R CNN
+F 2 "Connector_PinHeader_2.54mm:PinHeader_1x01_P2.54mm_Vertical" H 10060 5970 50  0001 C CNN
+F 3 "~" H 10060 5970 50  0001 C CNN
+	1    10060 5970
+	0    -1   -1   0
+$EndComp
 $EndSCHEMATC

Commit message: PCB drawing
Connections:
- net LAN_PWR: now reaches C85.2, C86.1, C87.1, C88.1, C90.1, C91.1, D15.5, J11.3 (TCT), J11.8 (RCT), L6.2, R91.1, R92.1, R93.1, R94.1, U30.1 (VDD2A), U30.19 (VDD1A)
Changed lines of the file:
@@
 	0    -1   -1   0
 $EndComp
+Text Label 7860 2100 0    50   ~ 0
+LAN_PWR
 $EndSCHEMATC

Commit message: minor changes
Parts:
- R88: footprint Resistor_SMD:R_0805_2012Metric_Pad1.20x1.40mm_HandSolder -> Resistor_SMD:R_0805_2012Metric
Changed lines of the file:
@@
 F 0 "R88" H 2500 2980 50  0000 L CNN
 F 1 "10K" H 2510 2670 50  0000 L CNN
-F 2 "Resistor_SMD:R_0805_2012Metric_Pad1.20x1.40mm_HandSolder" V 2610 2830 50  0001 C CNN
+F 2 "Resistor_SMD:R_0805_2012Metric" V 2610 2830 50  0001 C CNN
 F 3 "~" H 2680 2830 50  0001 C CNN
 F 4 "RC0805FR-0710KL" H 2680 2830 50  0001 C CNN "Type"

Commit message: commit after KiCAD library updates
Parts:
- U30: symbol Схема-и-печатная-плата-rescue:LAN8742A-CZ-TR-Interface_Ethernet -> Schema_and_PCB-rescue:LAN8742A-CZ-TR-Interface_Ethernet-Схема-и-печатная-плата-rescue
Changed lines of the file:
@@
 $EndDescr
 $Comp
-L Схема-и-печатная-плата-rescue:LAN8742A-CZ-TR-Interface_Ethernet U?
+L Schema_and_PCB-rescue:LAN8742A-CZ-TR-Interface_Ethernet-Схема-и-печатная-плата-rescue U?
 U 1 1 6091F45D
 P 3290 3270
