File: Analog_decoupling.sch (KiCad schematic (older format))
At the start: 108 parts, among them J10 22-23-2021, J6 22-23-2021, J8 22-23-2021, U16 LT1129CST-5#PBF, U18 ISO224ADWVR, U19 TLV9001IDBVR, U20 TLV9001IDBVR, U21 ISO224ADWVR, U22 TLV9001IDBVR, U23 TLV9001IDBVR, U25 REF1933AIDDCT, U27 ISO224ADWVR, U28 TLV9001IDBVR, U29 TLV9001IDBVR

Commit message: Analog decoupling annotations and create netlist
Parts:
- renumbered C48 to C1, C58 to C10, C59 to C11, C60 to C12, C62 to C13, C63 to C14, C64 to C15, C65 to C16, C67 to C17, C68 to C18, C70 to C19, C49 to C2, C71 to C20, C72 to C21, C73 to C22, C76 to C23, C77 to C24, C78 to C25, C50 to C3, C51 to C4, C52 to C5, C53 to C6, C55 to C7, C56 to C8, C57 to C9, D6 to D1, D7 to D2, D9 to D3, D10 to D4, D13 to D5, D14 to D6, J6 to J1, J8 to J2, J10 to J3, L3 to L1, L4 to L2, L5 to L3, R24 to R1, R35 to R10, R36 to R11, R37 to R12, R38 to R13, R39 to R14, R41 to R15, R42 to R16, R44 to R17, R45 to R18, R46 to R19, R25 to R2, R47 to R20, R48 to R21, R49 to R22, R50 to R23, R51 to R24, R52 to R25, R53 to R26, R54 to R27, R55 to R28, R58 to R29, R28 to R3, R59 to R30, R62 to R31, R63 to R32, R64 to R33, R65 to R34, R66 to R35, R67 to R36, R68 to R37, R69 to R38, R70 to R39, R29 to R4, R71 to R40, R72 to R41, R73 to R42, R30 to R5, R31 to R6, R32 to R7, R33 to R8, R34 to R9, TP5 to TP1, TP15 to TP10, TP17 to TP11, TP18 to TP12, TP20 to TP13, TP21 to TP14, TP22 to TP15, TP6 to TP2, TP8 to TP3, TP9 to TP4, TP10 to TP5, TP11 to TP6, TP12 to TP7, TP13 to TP8, TP14 to TP9, U16 to U1, U28 to U10, U29 to U11, U18 to U2, U19 to U3, U20 to U4, U21 to U5, U22 to U6, U23 to U7, U25 to U8, U27 to U9

Commit message: Analog decoupling schema completed. Digital_IO completed and clean up
Parts:
- removed C16, C25, C9: 330pF, Capacitor_SMD:C_0603_1608Metric_Pad1.08x0.95mm_HandSolder, symbol Device:C
- added J4: 302-S101, digikey-footprints:PinHeader_2x5_P2.54mm_Drill1.2mm, symbol dk_Rectangular-Connectors-Headers-Male-Pins:302-S101
- added J5: OSTTC020162, digikey-footprints:Term_Block_1x2_P5mm, symbol dk_Terminal-Blocks-Wire-to-Board:OSTTC020162
Connections:
- net labels removed: PF11, PF12, PF13, PF14, PF4, PF5
- wire segments 294 -> 305
Changed lines of the file:
@@
 	0    -1   -1   0
 $EndComp
-$Comp
-L Device:C C9
-U 1 1 60ADF23E
-P 8810 2530
-AR Path="/60ADF23E" Ref="C9"  Part="1"
-AR Path="/60A03F8A/60ADF23E" Ref="C?"  Part="1"
-AR Path="/60D8C564/60ADF23E" Ref="C?"  Part="1"
-F 0 "C9" H 8540 2640 50  0000 L CNN
-F 1 "330pF" H 8450 2560 50  0000 L CNN
-F 2 "Capacitor_SMD:C_0603_1608Metric_Pad1.08x0.95mm_HandSolder" H 8848 2380 50  0001 C CNN
-F 3 "http://www.farnell.com/datasheets/2710676.pdf" H 8810 2530 50  0001 C CNN
-F 4 "GRM188R71H331KA01D" H 8810 2530 50  0001 C CNN "Type"
-	1    8810 2530
-	1    0    0    -1
-$EndComp
 Wire Wire Line
 	8700 2220 8810 2220
 Wire Wire Line
-	8810 2220 8810 2380
-$Comp
-L power:GNDREF #PWR06
-U 1 1 60AE2E2B
-P 8810 2680
-AR Path="/60AE2E2B" Ref="#PWR06"  Part="1"
-AR Path="/60A03F8A/60AE2E2B" Ref="#PWR?"  Part="1"
-AR Path="/60D8C564/60AE2E2B" Ref="#PWR?"  Part="1"
-F 0 "#PWR06" H 8810 2430 50  0001 C CNN
-F 1 "GNDREF" V 8815 2552 50  0001 R CNN
-F 2 "" H 8810 2680 50  0001 C CNN
-F 3 "" H 8810 2680 50  0001 C CNN
-	1    8810 2680
-	1    0    0    -1
-$EndComp
-Wire Wire Line
-	9540 2220 8810 2220
+	9740 2220 8810 2220
 Connection ~ 8810 2220
-Text HLabel 9540 2220 2    50   Output ~ 0
-ADC1_P
 Wire Wire Line
 	7890 3120 7320 3120
 Connection ~ 7320 3120
-Text HLabel 7890 3120 2    50   Output ~ 0
-A_CH1_FAULT
 $Comp
 L Device:L_Core_Ferrite_Coupled L2
@@
 	0    -1   -1   0
 $EndComp
-$Comp
-L Device:C C16
-U 1 1 60B393D6
-P 8860 5590
-AR Path="/60B393D6" Ref="C16"  Part="1"
-AR Path="/60A03F8A/60B393D6" Ref="C?"  Part="1"
-AR Path="/60D8C564/60B393D6" Ref="C?"  Part="1"
-F 0 "C16" H 8590 5700 50  0000 L CNN
-F 1 "330pF" H 8500 5620 50  0000 L CNN
-F 2 "Capacitor_SMD:C_0603_1608Metric_Pad1.08x0.95mm_HandSolder" H 8898 5440 50  0001 C CNN
-F 3 "http://www.farnell.com/datasheets/2710676.pdf" H 8860 5590 50  0001 C CNN
-F 4 "GRM188R71H331KA01D" H 8860 5590 50  0001 C CNN "Type"
-	1    8860 5590
-	1    0    0    -1
-$EndComp
 Wire Wire Line
 	8750 5280 8860 5280
 Wire Wire Line
-	8860 5280 8860 5440
-$Comp
-L power:GNDREF #PWR015
-U 1 1 60B393DE
-P 8860 5740
-AR Path="/60B393DE" Ref="#PWR015"  Part="1"
-AR Path="/60A03F8A/60B393DE" Ref="#PWR?"  Part="1"
-AR Path="/60D8C564/60B393DE" Ref="#PWR?"  Part="1"
-F 0 "#PWR015" H 8860 5490 50  0001 C CNN
-F 1 "GNDREF" V 8865 5612 50  0001 R CNN
-F 2 "" H 8860 5740 50  0001 C CNN
-F 3 "" H 8860 5740 50  0001 C CNN
-	1    8860 5740
-	1    0    0    -1
-$EndComp
-Wire Wire Line
-	9590 5280 8860 5280
+	9800 5280 8860 5280
 Connection ~ 8860 5280
-Text HLabel 9590 5280 2    50   Output ~ 0
-ADC2_P
 Wire Wire Line
 	7940 6180 7370 6180
 Connection ~ 7370 6180
-Text HLabel 7940 6180 2    50   Output ~ 0
-A_CH2_FAULT
 Wire Wire Line
 	5200 4980 6510 4980
@@
 	0    -1   -1   0
 $EndComp
-$Comp
-L Device:C C25
-U 1 1 60BB25B9
-P 8970 9150
-AR Path="/60BB25B9" Ref="C25"  Part="1"
-AR Path="/60A03F8A/60BB25B9" Ref="C?"  Part="1"
-AR Path="/60D8C564/60BB25B9" Ref="C?"  Part="1"
-F 0 "C25" H 8700 9260 50  0000 L CNN
-F 1 "330pF" H 8610 9180 50  0000 L CNN
-F 2 "Capacitor_SMD:C_0603_1608Metric_Pad1.08x0.95mm_HandSolder" H 9008 9000 50  0001 C CNN
-F 3 "http://www.farnell.com/datasheets/2710676.pdf" H 8970 9150 50  0001 C CNN
-F 4 "GRM188R71H331KA01D" H 8970 9150 50  0001 C CNN "Type"
-	1    8970 9150
-	1    0    0    -1
-$EndComp
 Wire Wire Line
 	8860 8840 8970 8840
-Wire Wire Line
-	8970 8840 8970 9000
-$Comp
-L power:GNDREF #PWR028
-U 1 1 60BB25C1
-P 8970 9300
-AR Path="/60BB25C1" Ref="#PWR028"  Part="1"
-AR Path="/60A03F8A/60BB25C1" Ref="#PWR?"  Part="1"
-AR Path="/60D8C564/60BB25C1" Ref="#PWR?"  Part="1"
-F 0 "#PWR028" H 8970 9050 50  0001 C CNN
-F 1 "GNDREF" V 8975 9172 50  0001 R CNN
-F 2 "" H 8970 9300 50  0001 C CNN
-F 3 "" H 8970 9300 50  0001 C CNN
-	1    8970 9300
-	1    0    0    -1
-$EndComp
 Wire Wire Line
 	9700 8840 8970 8840
 Connection ~ 8970 8840
-Text HLabel 9700 8840 2    50   Output ~ 0
-ADC3_P
 Wire Wire Line
 	8050 9740 7480 9740
 Connection ~ 7480 9740
-Text HLabel 8050 9740 2    50   Output ~ 0
-A_CH3_FAULT
 Wire Wire Line
 	5310 8540 6620 8540
@@
 	1    0    0    -1
 $EndComp
-Text Label 9050 2220 0    50   ~ 0
-PF12
-Text Label 9040 5280 0    50   ~ 0
-PF13
-Text Label 9120 8840 0    50   ~ 0
-PF5
-Text Label 7820 9740 0    50   ~ 0
-PF4
-Text Label 7560 3120 0    50   ~ 0
-PF11
-Text Label 7640 6180 0    50   ~ 0
-PF14
+Text Label 9740 2220 2    50   ~ 0
+ADC1_P
+Text Label 9800 5280 2    50   ~ 0
+ADC2_P
+Text Label 9700 8840 2    50   ~ 0
+ADC3_P
+Text Label 8050 9740 2    50   ~ 0
+A_CH3_FAULT
+Text Label 7890 3120 2    50   ~ 0
+A_CH1_FAULT
 $Comp
 L Device:CP C21
@@
 	1    0    0    -1
 $EndComp
+$Comp
+L dk_Rectangular-Connectors-Headers-Male-Pins:302-S101 J4
+U 1 1 60B387F8
+P 13850 6390
+F 0 "J4" H 13890 6840 50  0000 C CNN
+F 1 "302-S101" H 13890 6740 50  0000 C CNN
+F 2 "digikey-footprints:PinHeader_2x5_P2.54mm_Drill1.2mm" H 14050 6590 60  0001 L CNN
+F 3 "http://www.on-shore.com/wp-content/uploads/2018/04/302-SXX1.pdf" V 14050 6690 60  0001 L CNN
+F 4 "ED1543-ND" H 14050 6790 60  0001 L CNN "Digi-Key_PN"
+F 5 "302-S101" H 14050 6890 60  0001 L CNN "MPN"
+F 6 "Connectors, Interconnects" H 14050 6990 60  0001 L CNN "Category"
+F 7 "Rectangular Connectors - Headers, Male Pins" H 14050 7090 60  0001 L CNN "Family"
+F 8 "http://www.on-shore.com/wp-content/uploads/2018/04/302-SXX1.pdf" H 14050 7190 60  0001 L CNN "DK_Datasheet_Link"
+F 9 "/product-detail/en/on-shore-technology-inc/302-S101/ED1543-ND/2178422" H 14050 7290 60  0001 L CNN "DK_Detail_Page"
+F 10 "CONN HEADER VERT 10POS 2.54MM" H 14050 7390 60  0001 L CNN "Description"
+F 11 "On Shore Technology Inc." H 14050 7490 60  0001 L CNN "Manufacturer"
+F 12 "Active" H 14050 7590 60  0001 L CNN "Status"
+	1    13850 6390
+	1    0    0    -1
+$EndComp
+$Comp
+L power:GNDREF #PWR06
+U 1 1 60B3A1E6
+P 13470 6760
+AR Path="/60B3A1E6" Ref="#PWR06"  Part="1"
+AR Path="/60A03F8A/60B3A1E6" Ref="#PWR?"  Part="1"
+AR Path="/60D8C564/60B3A1E6" Ref="#PWR?"  Part="1"
+F 0 "#PWR06" H 13470 6510 50  0001 C CNN
+F 1 "GNDREF" V 13475 6632 50  0001 R CNN
+F 2 "" H 13470 6760 50  0001 C CNN
+F 3 "" H 13470 6760 50  0001 C CNN
+	1    13470 6760
+	1    0    0    -1
+$EndComp
+Wire Wire Line
+	13470 6760 13470 6490
+Wire Wire Line
+	13470 6190 13650 6190
+Wire Wire Line
+	13650 6290 13470 6290
+Connection ~ 13470 6290
+Wire Wire Line
+	13470 6290 13470 6190
+Wire Wire Line
+	13650 6390 13470 6390
+Connection ~ 13470 6390
+Wire Wire Line
+	13470 6390 13470 6290
+Wire Wire Line
+	13650 6490 13470 6490
+Connection ~ 13470 6490
+Wire Wire Line
+	13470 6490 13470 6390
+Wire Wire Line
+	12930 6590 13650 6590
+Wire Wire Line
+	14050 6190 14680 6190
+Wire Wire Line
+	14050 6290 14680 6290
+Wire Wire Line
+	14050 6390 14680 6390
+Wire Wire Line
+	14050 6490 14680 6490
+Wire Wire Line
+	14050 6590 14680 6590
+Text Label 14680 6190 2    50   ~ 0
+ADC1_P
+Text Label 14680 6290 2    50   ~ 0
+ADC2_P
+Text Label 14680 6390 2    50   ~ 0
+ADC3_P
+Text Label 14680 6490 2    50   ~ 0
+A_CH1_FAULT
+Text Label 14680 6590 2    50   ~ 0
+A_CH3_FAULT
+Text Label 12930 6590 0    50   ~ 0
+A_CH2_FAULT
+$Comp
+L dk_Terminal-Blocks-Wire-to-Board:OSTTC020162 J5
+U 1 1 60C63E05
+P 13730 7990
+F 0 "J5" H 13560 8030 50  0000 L CNN
+F 1 "OSTTC020162" H 13500 7880 50  0000 L CNN
+F 2 "digikey-footprints:Term_Block_1x2_P5mm" H 13930 8190 60  0001 L CNN
+F 3 "http://www.on-shore.com/wp-content/uploads/OSTTCXX0162.pdf" H 13930 8290 60  0001 L CNN
+F 4 "ED2600-ND" H 13930 8390 60  0001 L CNN "Digi-Key_PN"
+F 5 "OSTTC020162" H 13930 8490 60  0001 L CNN "MPN"
+F 6 "Connectors, Interconnects" H 13930 8590 60  0001 L CNN "Category"
+F 7 "Terminal Blocks - Wire to Board" H 13930 8690 60  0001 L CNN "Family"
+F 8 "http://www.on-shore.com/wp-content/uploads/OSTTCXX0162.pdf" H 13930 8790 60  0001 L CNN "DK_Datasheet_Link"
+F 9 "/product-detail/en/on-shore-technology-inc/OSTTC020162/ED2600-ND/614549" H 13930 8890 60  0001 L CNN "DK_Detail_Page"
+F 10 "TERM BLK 2POS SIDE ENTRY 5MM PCB" H 13930 8990 60  0001 L CNN "Description"
+F 11 "On Shore Technology Inc." H 13930 9090 60  0001 L CNN "Manufacturer"
+F 12 "Active" H 13930 9190 60  0001 L CNN "Status"
+	1    13730 7990
+	1    0    0    -1
+$EndComp
+$Comp
+L power:GNDREF #PWR0101
+U 1 1 60C64714
+P 13730 7790
+AR Path="/60C64714" Ref="#PWR0101"  Part="1"
+AR Path="/60A03F8A/60C64714" Ref="#PWR?"  Part="1"
+AR Path="/60D8C564/60C64714" Ref="#PWR?"  Part="1"
+F 0 "#PWR0101" H 13730 7540 50  0001 C CNN
+F 1 "GNDREF" V 13735 7662 50  0001 R CNN
+F 2 "" H 13730 7790 50  0001 C CNN
+F 3 "" H 13730 7790 50  0001 C CNN
+	1    13730 7790
+	-1   0    0    1
+$EndComp
+$Comp
+L SVIELCOM_Library:+24V #PWR0102
+U 1 1 60C6601C
+P 13830 7790
+F 0 "#PWR0102" H 13980 7840 50  0001 C CNN
+F 1 "+24V" H 13820 7950 50  0000 C CNN
+F 2 "" H 13830 7790 50  0001 C CNN
+F 3 "" H 13830 7790 50  0001 C CNN
+	1    13830 7790
+	1    0    0    -1
+$EndComp
+$Comp
+L power:PWR_FLAG #FLG0101
+U 1 1 60C67E1D
+P 13830 7790
+F 0 "#FLG0101" H 13830 7865 50  0001 C CNN
+F 1 "PWR_FLAG" V 13800 7940 50  0001 L CNN
+F 2 "" H 13830 7790 50  0001 C CNN
+F 3 "~" H 13830 7790 50  0001 C CNN
+	1    13830 7790
+	0    1    1    0
+$EndComp
+Connection ~ 13830 7790
+Text Label 7940 6180 2    50   ~ 0
+A_CH2_FAULT
 $EndSCHEMATC

Commit message: OA pinout corrected. Mounting holes deleted
Parts:
- removed U10, U11, U3, U4, U6, U7: TLV9001IDBVR, Package_TO_SOT_SMD:SOT-23-5_HandSoldering, symbol Amplifier_Operational:TLV9001IDCK
- added U10, U11, U3, U4, U6, U7: TLV9001IDBVR, Package_TO_SOT_SMD:SOT-23-5, symbol SVIELCOM_Library:TLV9001IDBVR
- R1, R10, R15, R16, R2, R21, R24, R29, R30, R35, R38, R7: footprint Resistor_SMD:R_0603_1608Metric_Pad0.98x0.95mm_HandSolder -> Resistor_SMD:R_0603_1608Metric
- R11, R12, R13, R14, R18, R19, R20, R22, R23, R25, R26, R27, R28, R32, R33, R34, R36, R37, R39, R4, R40, R41, R42, R5, R6, R8, R9: footprint Resistor_SMD:R_0805_2012Metric_Pad1.20x1.40mm_HandSolder -> Resistor_SMD:R_0805_2012Metric

Commit message: ADC1 input changed from IN6 to IN2
Parts:
- U2, U5, U9: symbol Схема-и-печатная-плата-rescue:ISO224ADWVR-Isolator -> Analog_decoupling-rescue:ISO224ADWVR-Isolator-Схема-и-печатная-плата-rescue
Changed lines of the file:
@@
 $EndComp
 $Comp
-L Схема-и-печатная-плата-rescue:ISO224ADWVR-Isolator U2
+L Analog_decoupling-rescue:ISO224ADWVR-Isolator-Схема-и-печатная-плата-rescue U2
 U 1 1 60D90026
 P 3740 1920
@@
 $EndComp
 $Comp
-L Схема-и-печатная-плата-rescue:ISO224ADWVR-Isolator U5
+L Analog_decoupling-rescue:ISO224ADWVR-Isolator-Схема-и-печатная-плата-rescue U5
 U 1 1 60B39259
 P 3790 4980
@@
 $EndComp
 $Comp
-L Схема-и-печатная-плата-rescue:ISO224ADWVR-Isolator U9
+L Analog_decoupling-rescue:ISO224ADWVR-Isolator-Схема-и-печатная-плата-rescue U9
 U 1 1 60BB246B
 P 3900 8540
