File: Microcontroller.kicad_sch (KiCad schematic)
At the start: 6 parts, among them J13 640456-3, J14 640456-3, J15 640456-3, J16 B5B-XH-A_LF__SN_, J17 0022232041, U11 STM32H743ZIT6

Commit message: GPIO port changed for input signals
Connections:
- net A_CH1_FAULT: now also U11.80 (PD11); no longer U11.77 (PD8)
- net A_CH2_FAULT: now also U11.78 (PD9); no longer U11.75 (PB14)
- net A_CH3_FAULT: now also U11.79 (PD10); no longer U11.76 (PB15)
- net SD_CARD_INS: now also U11.114 (PD0); no longer U11.117 (PD3)
