File: Digital_IO_analog_Inputs.kicad_sch (KiCad schematic)
At the start: 52 parts, among them J3 302-S101, J5 OSTTC020162, J7 OSTTC030162, J9 0022232031, Q3 BC817-25LT1G, Q4 BC817-25LT1G, Q5 BC817-25LT1G, Q6 BC817-25LT1G, Q7 BC817-25LT1G, U17 ISO1211DR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

Commit message: All handsolder footprints removed
Parts:
- C48, C49, C50, C52, C54, C61, C66, C69, C74, C75: footprint Capacitor_SMD:C_0603_1608Metric_Pad1.08x0.95mm_HandSolder -> Capacitor_SMD:C_0603_1608Metric
- L3: footprint Inductor_SMD:L_0805_2012Metric_Pad1.15x1.40mm_HandSolder -> Inductor_SMD:L_0805_2012Metric
- R27, R29, R30, R31, R32, R33, R40, R56, R60: footprint Resistor_SMD:R_0805_2012Metric_Pad1.20x1.40mm_HandSolder -> Resistor_SMD:R_0805_2012Metric
Changed lines of the file:
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@@
     (property "Reference" "R40" (id 0) (at 68.072 57.404 90))
     (property "Value" "10K" (id 1) (at 68.326 62.23 90))
-    (property "Footprint" "Resistor_SMD:R_0805_2012Metric_Pad1.20x1.40mm_HandSolder" (id 2) (at 69.088 57.912 90)
+    (property "Footprint" "Resistor_SMD:R_0805_2012Metric" (id 2) (at 69.088 57.912 90)
       (effects (font (size 1.27 1.27)) hide)
     )
@@
       (effects (font (size 1.27 1.27)) (justify left))
     )
-    (property "Footprint" "Capacitor_SMD:C_0603_1608Metric_Pad1.08x0.95mm_HandSolder" (id 2) (at 57.0992 127.254 0)
+    (property "Footprint" "Capacitor_SMD:C_0603_1608Metric" (id 2) (at 57.0992 127.254 0)
       (effects (font (size 1.27 1.27)) hide)
     )
@@
       (effects (font (size 1.27 1.27)) (justify left))
     )
-    (property "Footprint" "Capacitor_SMD:C_0603_1608Metric_Pad1.08x0.95mm_HandSolder" (id 2) (at 63.4492 127.254 0)
+    (property "Footprint" "Capacitor_SMD:C_0603_1608Metric" (id 2) (at 63.4492 127.254 0)
       (effects (font (size 1.27 1.27)) hide)
     )
@@
       (effects (font (size 1.27 1.27)) (justify left))
     )
-    (property "Footprint" "Capacitor_SMD:C_0603_1608Metric_Pad1.08x0.95mm_HandSolder" (id 2) (at 69.7992 127.254 0)
+    (property "Footprint" "Capacitor_SMD:C_0603_1608Metric" (id 2) (at 69.7992 127.254 0)
       (effects (font (size 1.27 1.27)) hide)
     )
@@
       (effects (font (size 1.27 1.27)) (justify left))
     )
-    (property "Footprint" "Capacitor_SMD:C_0603_1608Metric_Pad1.08x0.95mm_HandSolder" (id 2) (at 206.1972 86.36 0)
+    (property "Footprint" "Capacitor_SMD:C_0603_1608Metric" (id 2) (at 206.1972 86.36 0)
       (effects (font (size 1.27 1.27)) hide)
     )
@@
       (effects (font (size 1.27 1.27)) (justify left))
     )
-    (property "Footprint" "Inductor_SMD:L_0805_2012Metric_Pad1.15x1.40mm_HandSolder" (id 2) (at 244.094 56.134 0)
+    (property "Footprint" "Inductor_SMD:L_0805_2012Metric" (id 2) (at 244.094 56.134 0)
       (effects (font (size 1.27 1.27)) hide)
     )
@@
       (effects (font (size 1.27 1.27)) (justify left))
     )
-    (property "Footprint" "Capacitor_SMD:C_0603_1608Metric_Pad1.08x0.95mm_HandSolder" (id 2) (at 249.8852 90.17 0)
+    (property "Footprint" "Capacitor_SMD:C_0603_1608Metric" (id 2) (at 249.8852 90.17 0)
       (effects (font (size 1.27 1.27)) hide)
     )
@@
       (effects (font (size 1.27 1.27)) (justify left))
     )
-    (property "Footprint" "Capacitor_SMD:C_0603_1608Metric_Pad1.08x0.95mm_HandSolder" (id 2) (at 75.3872 83.82 0)
+    (property "Footprint" "Capacitor_SMD:C_0603_1608Metric" (id 2) (at 75.3872 83.82 0)
       (effects (font (size 1.27 1.27)) hide)
     )
@@
     (property "Reference" "R56" (id 0) (at 210.82 104.648 90))
     (property "Value" "560" (id 1) (at 210.82 106.68 90))
-    (property "Footprint" "Resistor_SMD:R_0805_2012Metric_Pad1.20x1.40mm_HandSolder" (id 2) (at 211.328 112.014 90)
+    (property "Footprint" "Resistor_SMD:R_0805_2012Metric" (id 2) (at 211.328 112.014 90)
       (effects (font (size 1.27 1.27)) hide)
     )
@@
       (effects (font (size 1.27 1.27)) (justify left))
     )
-    (property "Footprint" "Capacitor_SMD:C_0603_1608Metric_Pad1.08x0.95mm_HandSolder" (id 2) (at 206.1972 119.126 0)
+    (property "Footprint" "Capacitor_SMD:C_0603_1608Metric" (id 2) (at 206.1972 119.126 0)
       (effects (font (size 1.27 1.27)) hide)
     )
@@
     (property "Reference" "R60" (id 0) (at 210.82 136.906 90))
     (property "Value" "560" (id 1) (at 210.82 138.938 90))
-    (property "Footprint" "Resistor_SMD:R_0805_2012Metric_Pad1.20x1.40mm_HandSolder" (id 2) (at 211.328 144.272 90)
+    (property "Footprint" "Resistor_SMD:R_0805_2012Metric" (id 2) (at 211.328 144.272 90)
       (effects (font (size 1.27 1.27)) hide)
     )
@@
       (effects (font (size 1.27 1.27)) (justify left))
     )
-    (property "Footprint" "Capacitor_SMD:C_0603_1608Metric_Pad1.08x0.95mm_HandSolder" (id 2) (at 206.1972 151.384 0)
+    (property "Footprint" "Capacitor_SMD:C_0603_1608Metric" (id 2) (at 206.1972 151.384 0)
       (effects (font (size 1.27 1.27)) hide)
     )
@@
       (effects (font (size 1.27 1.27)) (justify left))
     )
-    (property "Footprint" "Capacitor_SMD:C_0603_1608Metric_Pad1.08x0.95mm_HandSolder" (id 2) (at 249.8852 122.936 0)
+    (property "Footprint" "Capacitor_SMD:C_0603_1608Metric" (id 2) (at 249.8852 122.936 0)
       (effects (font (size 1.27 1.27)) hide)
     )
@@
       (effects (font (size 1.27 1.27)) (justify left))
     )
-    (property "Footprint" "Capacitor_SMD:C_0603_1608Metric_Pad1.08x0.95mm_HandSolder" (id 2) (at 249.8852 155.194 0)
+    (property "Footprint" "Capacitor_SMD:C_0603_1608Metric" (id 2) (at 249.8852 155.194 0)
       (effects (font (size 1.27 1.27)) hide)
     )
@@
     (property "Reference" "R33" (id 0) (at 100.838 175.768 90))
     (property "Value" "47K" (id 1) (at 101.092 180.594 90))
-    (property "Footprint" "Resistor_SMD:R_0805_2012Metric_Pad1.20x1.40mm_HandSolder" (id 2) (at 101.854 176.276 90)
+    (property "Footprint" "Resistor_SMD:R_0805_2012Metric" (id 2) (at 101.854 176.276 90)
       (effects (font (size 1.27 1.27)) hide)
     )
@@
     (property "Reference" "R27" (id 0) (at 46.228 154.432 0))
     (property "Value" "150" (id 1) (at 46.736 156.718 0))
-    (property "Footprint" "Resistor_SMD:R_0805_2012Metric_Pad1.20x1.40mm_HandSolder" (id 2) (at 41.402 156.464 90)
+    (property "Footprint" "Resistor_SMD:R_0805_2012Metric" (id 2) (at 41.402 156.464 90)
       (effects (font (size 1.27 1.27)) hide)
     )
@@
     (property "Reference" "R30" (id 0) (at 116.332 154.432 0))
     (property "Value" "150" (id 1) (at 116.84 156.718 0))
-    (property "Footprint" "Resistor_SMD:R_0805_2012Metric_Pad1.20x1.40mm_HandSolder" (id 2) (at 111.506 156.464 90)
+    (property "Footprint" "Resistor_SMD:R_0805_2012Metric" (id 2) (at 111.506 156.464 90)
       (effects (font (size 1.27 1.27)) hide)
     )
@@
     (property "Reference" "R29" (id 0) (at 82.042 154.432 0))
     (property "Value" "150" (id 1) (at 82.55 156.718 0))
-    (property "Footprint" "Resistor_SMD:R_0805_2012Metric_Pad1.20x1.40mm_HandSolder" (id 2) (at 77.216 156.464 90)
+    (property "Footprint" "Resistor_SMD:R_0805_2012Metric" (id 2) (at 77.216 156.464 90)
       (effects (font (size 1.27 1.27)) hide)
     )
@@
     (property "Reference" "R31" (id 0) (at 30.734 175.768 90))
     (property "Value" "47K" (id 1) (at 30.988 180.594 90))
-    (property "Footprint" "Resistor_SMD:R_0805_2012Metric_Pad1.20x1.40mm_HandSolder" (id 2) (at 31.75 176.276 90)
+    (property "Footprint" "Resistor_SMD:R_0805_2012Metric" (id 2) (at 31.75 176.276 90)
       (effects (font (size 1.27 1.27)) hide)
     )
@@
     (property "Reference" "R32" (id 0) (at 66.548 175.768 90))
     (property "Value" "47K" (id 1) (at 66.802 180.594 90))
-    (property "Footprint" "Resistor_SMD:R_0805_2012Metric_Pad1.20x1.40mm_HandSolder" (id 2) (at 67.564 176.276 90)
-      (effects (font (size 1.27 1.27)) hide)
-    )
+    (property "Footprint" "Resistor_SMD:R_0805_2012Metric" (id 2) (at 67.564 176.276 90)
+      (effects (font (size 1.27 1.27)) hide)
+    )
