File: Indicator.kicad_sch (KiCad schematic)
At the start: 25 parts, among them Q1 BC817-25LT1G, Q2 BC817-25LT1G, U1 CC56-12SURKWA, U2 CC56-12SURKWA, U3 MAX7219EWG+T, U4 BC56-12SURKWA, U5 SC56-11SRWA, U6 MAX7219EWG+T, U7 CC56-12SURKWA

Commit message: KiCAD6.0 scheema rules check done
Other:
- note added: "PD7"
- note added: "PF2"
- note added: "PF3"
- note added: "PG10"
- note added: "PG11"
- moved on the sheet: U5

Commit message: All handsolder footprints removed
Parts:
- C43, C44: footprint Capacitor_SMD:C_0603_1608Metric_Pad1.08x0.95mm_HandSolder -> Capacitor_SMD:C_0603_1608Metric
- R1, R2, R3, R4, R5, R6, R7, R8: footprint Resistor_SMD:R_0805_2012Metric_Pad1.20x1.40mm_HandSolder -> Resistor_SMD:R_0805_2012Metric
Changed lines of the file:
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@@
     (property "Reference" "R6" (id 0) (at 33.528 47.244 0))
     (property "Value" "16.9K" (id 1) (at 32.512 49.784 0))
-    (property "Footprint" "Resistor_SMD:R_0805_2012Metric_Pad1.20x1.40mm_HandSolder" (id 2) (at 35.052 49.53 90)
+    (property "Footprint" "Resistor_SMD:R_0805_2012Metric" (id 2) (at 35.052 49.53 90)
       (effects (font (size 1.27 1.27)) hide)
     )
@@
     (property "Reference" "R1" (id 0) (at 221.234 25.4 0))
     (property "Value" "100" (id 1) (at 221.742 27.686 0))
-    (property "Footprint" "Resistor_SMD:R_0805_2012Metric_Pad1.20x1.40mm_HandSolder" (id 2) (at 216.408 27.432 90)
+    (property "Footprint" "Resistor_SMD:R_0805_2012Metric" (id 2) (at 216.408 27.432 90)
       (effects (font (size 1.27 1.27)) hide)
     )
@@
     (property "Reference" "R2" (id 0) (at 265.176 25.654 0))
     (property "Value" "100" (id 1) (at 265.43 27.94 0))
-    (property "Footprint" "Resistor_SMD:R_0805_2012Metric_Pad1.20x1.40mm_HandSolder" (id 2) (at 260.35 27.686 90)
+    (property "Footprint" "Resistor_SMD:R_0805_2012Metric" (id 2) (at 260.35 27.686 90)
       (effects (font (size 1.27 1.27)) hide)
     )
@@
     (property "Reference" "R5" (id 0) (at 249.682 46.99 90))
     (property "Value" "47K" (id 1) (at 249.936 51.816 90))
-    (property "Footprint" "Resistor_SMD:R_0805_2012Metric_Pad1.20x1.40mm_HandSolder" (id 2) (at 250.698 47.498 90)
+    (property "Footprint" "Resistor_SMD:R_0805_2012Metric" (id 2) (at 250.698 47.498 90)
       (effects (font (size 1.27 1.27)) hide)
     )
@@
     (property "Reference" "R4" (id 0) (at 205.74 46.736 90))
     (property "Value" "47K" (id 1) (at 205.994 51.562 90))
-    (property "Footprint" "Resistor_SMD:R_0805_2012Metric_Pad1.20x1.40mm_HandSolder" (id 2) (at 206.756 47.244 90)
+    (property "Footprint" "Resistor_SMD:R_0805_2012Metric" (id 2) (at 206.756 47.244 90)
       (effects (font (size 1.27 1.27)) hide)
     )
@@
       (effects (font (size 1.27 1.27)) (justify left))
     )
-    (property "Footprint" "Capacitor_SMD:C_0603_1608Metric_Pad1.08x0.95mm_HandSolder" (id 2) (at 55.3212 45.974 0)
+    (property "Footprint" "Capacitor_SMD:C_0603_1608Metric" (id 2) (at 55.3212 45.974 0)
       (effects (font (size 1.27 1.27)) hide)
     )
@@
       (effects (font (size 1.27 1.27)) (justify left))
     )
-    (property "Footprint" "Capacitor_SMD:C_0603_1608Metric_Pad1.08x0.95mm_HandSolder" (id 2) (at 55.3212 130.048 0)
+    (property "Footprint" "Capacitor_SMD:C_0603_1608Metric" (id 2) (at 55.3212 130.048 0)
       (effects (font (size 1.27 1.27)) hide)
     )
@@
     (property "Reference" "R3" (id 0) (at 39.624 40.894 90))
     (property "Value" "200" (id 1) (at 44.45 40.894 90))
-    (property "Footprint" "Resistor_SMD:R_0805_2012Metric_Pad1.20x1.40mm_HandSolder" (id 2) (at 42.418 41.91 90)
+    (property "Footprint" "Resistor_SMD:R_0805_2012Metric" (id 2) (at 42.418 41.91 90)
       (effects (font (size 1.27 1.27)) hide)
     )
@@
     (property "Reference" "R8" (id 0) (at 39.878 131.572 0))
     (property "Value" "16.9K" (id 1) (at 41.148 133.604 0))
-    (property "Footprint" "Resistor_SMD:R_0805_2012Metric_Pad1.20x1.40mm_HandSolder" (id 2) (at 35.306 133.35 90)
+    (property "Footprint" "Resistor_SMD:R_0805_2012Metric" (id 2) (at 35.306 133.35 90)
       (effects (font (size 1.27 1.27)) hide)
     )
@@
     (property "Reference" "R7" (id 0) (at 39.878 124.714 90))
     (property "Value" "200" (id 1) (at 44.704 124.714 90))
-    (property "Footprint" "Resistor_SMD:R_0805_2012Metric_Pad1.20x1.40mm_HandSolder" (id 2) (at 42.672 125.73 90)
-      (effects (font (size 1.27 1.27)) hide)
-    )
+    (property "Footprint" "Resistor_SMD:R_0805_2012Metric" (id 2) (at 42.672 125.73 90)
+      (effects (font (size 1.27 1.27)) hide)
+    )
