File: LAN.kicad_sch (KiCad schematic)
At the start: 35 parts, among them J11 Pulse_JXD6-0001NL, J12 Ground, U30 LAN8742A-CZ-TR, Y3 NX2016SA-25MHz

Commit message: KiCAD6.0 scheema rules check done
Changed lines of the file:
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@@
+    (pin "1")
+  )
+  (symbol (lib_id "power:PWR_FLAG") (at 139.192 53.34 0) (unit 1)
+    (in_bom yes) (on_board yes)
+    (property "Reference" "#FLG0103" (id 0) (at 139.192 51.435 0)
+      (effects (font (size 1.27 1.27)) hide)
+    )
+    (property "Value" "PWR_FLAG" (id 1) (at 138.938 50.038 90)
+      (effects (font (size 1.27 1.27)) (justify left) hide)
+    )
+    (property "Footprint" "" (id 2) (at 139.192 53.34 0)
+      (effects (font (size 1.27 1.27)) hide)
+    )
+    (property "Datasheet" "~" (id 3) (at 139.192 53.34 0)
+      (effects (font (size 1.27 1.27)) hide)
+    )
     (pin "1")
   )

Commit message: All handsolder footprints removed
Parts:
- R100, R101, R102, R103, R86, R87, R89, R90, R95, R96, R97, R98, R99: footprint Resistor_SMD:R_0805_2012Metric_Pad1.20x1.40mm_HandSolder -> Resistor_SMD:R_0805_2012Metric
Changed lines of the file:
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@@
       (effects (font (size 1.27 1.27)) (justify left))
     )
-    (property "Footprint" "Resistor_SMD:R_0805_2012Metric_Pad1.20x1.40mm_HandSolder" (id 2) (at 255.27 76.2 90)
+    (property "Footprint" "Resistor_SMD:R_0805_2012Metric" (id 2) (at 255.27 76.2 90)
       (effects (font (size 1.27 1.27)) hide)
     )
@@
       (effects (font (size 1.27 1.27)) (justify left))
     )
-    (property "Footprint" "Resistor_SMD:R_0805_2012Metric_Pad1.20x1.40mm_HandSolder" (id 2) (at 247.65 76.2 90)
+    (property "Footprint" "Resistor_SMD:R_0805_2012Metric" (id 2) (at 247.65 76.2 90)
       (effects (font (size 1.27 1.27)) hide)
     )
@@
       (effects (font (size 1.27 1.27)) (justify left))
     )
-    (property "Footprint" "Resistor_SMD:R_0805_2012Metric_Pad1.20x1.40mm_HandSolder" (id 2) (at 263.144 76.2 90)
+    (property "Footprint" "Resistor_SMD:R_0805_2012Metric" (id 2) (at 263.144 76.2 90)
       (effects (font (size 1.27 1.27)) hide)
     )
@@
       (effects (font (size 1.27 1.27)) (justify left))
     )
-    (property "Footprint" "Resistor_SMD:R_0805_2012Metric_Pad1.20x1.40mm_HandSolder" (id 2) (at 159.004 143.256 90)
+    (property "Footprint" "Resistor_SMD:R_0805_2012Metric" (id 2) (at 159.004 143.256 90)
       (effects (font (size 1.27 1.27)) hide)
     )
@@
       (effects (font (size 1.27 1.27)) (justify left))
     )
-    (property "Footprint" "Resistor_SMD:R_0805_2012Metric_Pad1.20x1.40mm_HandSolder" (id 2) (at 83.312 71.882 90)
+    (property "Footprint" "Resistor_SMD:R_0805_2012Metric" (id 2) (at 83.312 71.882 90)
       (effects (font (size 1.27 1.27)) hide)
     )
@@
       (effects (font (size 1.27 1.27)) (justify left))
     )
-    (property "Footprint" "Resistor_SMD:R_0805_2012Metric_Pad1.20x1.40mm_HandSolder" (id 2) (at 38.862 123.698 90)
+    (property "Footprint" "Resistor_SMD:R_0805_2012Metric" (id 2) (at 38.862 123.698 90)
       (effects (font (size 1.27 1.27)) hide)
     )
@@
       (effects (font (size 1.27 1.27)) (justify left))
     )
-    (property "Footprint" "Resistor_SMD:R_0805_2012Metric_Pad1.20x1.40mm_HandSolder" (id 2) (at 76.708 71.882 90)
+    (property "Footprint" "Resistor_SMD:R_0805_2012Metric" (id 2) (at 76.708 71.882 90)
       (effects (font (size 1.27 1.27)) hide)
     )
@@
       (effects (font (size 1.27 1.27)) (justify left))
     )
-    (property "Footprint" "Resistor_SMD:R_0805_2012Metric_Pad1.20x1.40mm_HandSolder" (id 2) (at 38.862 112.268 90)
+    (property "Footprint" "Resistor_SMD:R_0805_2012Metric" (id 2) (at 38.862 112.268 90)
       (effects (font (size 1.27 1.27)) hide)
     )
@@
       (effects (font (size 1.27 1.27)) (justify left))
     )
-    (property "Footprint" "Resistor_SMD:R_0805_2012Metric_Pad1.20x1.40mm_HandSolder" (id 2) (at 47.244 98.044 90)
+    (property "Footprint" "Resistor_SMD:R_0805_2012Metric" (id 2) (at 47.244 98.044 90)
       (effects (font (size 1.27 1.27)) hide)
     )
@@
       (effects (font (size 1.27 1.27)) (justify left))
     )
-    (property "Footprint" "Resistor_SMD:R_0805_2012Metric_Pad1.20x1.40mm_HandSolder" (id 2) (at 38.862 89.408 90)
+    (property "Footprint" "Resistor_SMD:R_0805_2012Metric" (id 2) (at 38.862 89.408 90)
       (effects (font (size 1.27 1.27)) hide)
     )
@@
       (effects (font (size 1.27 1.27)) (justify left))
     )
-    (property "Footprint" "Resistor_SMD:R_0805_2012Metric_Pad1.20x1.40mm_HandSolder" (id 2) (at 38.862 86.868 90)
+    (property "Footprint" "Resistor_SMD:R_0805_2012Metric" (id 2) (at 38.862 86.868 90)
       (effects (font (size 1.27 1.27)) hide)
     )
@@
       (effects (font (size 1.27 1.27)) (justify left))
     )
-    (property "Footprint" "Resistor_SMD:R_0805_2012Metric_Pad1.20x1.40mm_HandSolder" (id 2) (at 62.992 71.882 90)
+    (property "Footprint" "Resistor_SMD:R_0805_2012Metric" (id 2) (at 62.992 71.882 90)
       (effects (font (size 1.27 1.27)) hide)
     )
@@
       (effects (font (size 1.27 1.27)) (justify left))
     )
-    (property "Footprint" "Resistor_SMD:R_0805_2012Metric_Pad1.20x1.40mm_HandSolder" (id 2) (at 55.88 71.882 90)
-      (effects (font (size 1.27 1.27)) hide)
-    )
+    (property "Footprint" "Resistor_SMD:R_0805_2012Metric" (id 2) (at 55.88 71.882 90)
+      (effects (font (size 1.27 1.27)) hide)
+    )
